File: modules/envelope-generator/1-scribble/kiCad/envelope_generator.kicad_sch (KiCad schematic)
At the start: 66 parts, among them J1 PWR, J2 GATE, J3 INV_OUT, J4 OUT, Q1 BC548, SW1 LOOP, U1 TL074, U2 TL074

Commit message: fixes for scribble, added scripts for generating hole for panels
Parts:
- removed C8: 1uF, synth-custom:C_RECT_MKT_1uF, symbol Device:C
- removed D3, D4, D5, D8: 1N4148, Diode_THT:D_DO-35_SOD27_P7.62mm_Horizontal, symbol Diode:1N4148
- removed unit 2 of H1
- removed unit 1 of H1
- removed unit 1 of H2
- removed unit 2 of H2
- removed unit 1 of H3
- removed unit 3 of H3
- removed unit 2 of H3
- removed unit 2 of H4
- removed unit 1 of H4
- removed unit 3 of H4
- removed unit 3 of H5
- removed unit 3 of H6
- removed J2: GATE, synth-custom:Jack_3.5mm_QingPu_WQP-PJ398SM_Vertical_CircularHoles, symbol Synth_Custom:AudioJack2_PJ398SM
- removed J3: INV_OUT, synth-custom:Jack_3.5mm_QingPu_WQP-PJ398SM_Vertical_CircularHoles, symbol Synth_Custom:AudioJack2_PJ398SM
- removed R10, R11, R12, R3, R4, R5, R6, R7, R8, R9: 100K, synth-custom:R_Axial_DIN0207_L6.3mm_D2.5mm_P7.62mm_Horizontal, symbol Device:R
- removed R13: 47K, synth-custom:R_Axial_DIN0207_L6.3mm_D2.5mm_P7.62mm_Horizontal, symbol Device:R
- removed R14: 10K, synth-custom:R_Axial_DIN0207_L6.3mm_D2.5mm_P7.62mm_Horizontal, symbol Device:R
- removed R16: 1K, synth-custom:R_Axial_DIN0207_L6.3mm_D2.5mm_P7.62mm_Horizontal, symbol Device:R
- removed SUSTAIN1: A100K, Potentiometer_THT:Potentiometer_TT_P0915N, symbol Device:R_Potentiometer
- removed TP1: A, symbol Connector:TestPoint
- removed unit 4 of U1
- removed unit 2 of U1
- removed unit 1 of U1
- removed unit 1 of U2
- TP2, TP3: footprint (none) -> TestPoint:TestPoint_Plated_Hole_D2.0mm
Connections:
- net feedback_loop/feedback_input: now reaches H6.2, Q1.2 (B), TP3.1, U2.7
- net feedback_loop/feedback_input: now also U2.6 (-); no longer U2.5 (+)
- net input_sustain/gate_out: now reaches SW1.3 (C)
- net at C7.1, C9_OPT1.1, H6.1: now also U2.5 (+); no longer U2.6 (-)
- net at R18.1, U1.8: now also U1.9 (-); no longer U1.10 (+)
- net at H2.3, TP2.1: now also U1.10 (+); no longer U1.9 (-)
- net feedback_loop/feedback_output: now reaches SW1.1 (A)
- no-connect marks 14 -> 13
Other:
- added sheet feedback_loop (feedback_loop.kicad_sch)
- added sheet input_sustain (input_sustain.kicad_sch)
- added sheet inverted_out (inverted_out.kicad_sch)
- moved on the sheet: ATT1, C7, C9_OPT1, D6, D7, D9, H1C, H2C, H3D, H4D, H5A, H5B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
