File: modules/envelope-generator/1-scribble/kiCad/scribble.kicad_sch (KiCad schematic)
At the start: 44 parts, among them J1 PWR, J4 OUT, Q1 BC548, SW1 LOOP, U1 TL074, U2 TL074

Commit message: vixen & Scribble files
Parts:
- removed H3: TOP_8_SGL, synth-custom:PinHeader_1x04_P2.00mm_Vertical, symbol Synth_Custom:CONN_Header_01x04
- removed H4: BTM_8_SGL, synth-custom:PinSocket_1x04_P2.00mm_Vertical, symbol Synth_Custom:CONN_Socket_01x04
- removed unit 4 of H5
- removed unit 4 of H6
- added unit 2 of H3
- added unit 3 of H3
- added unit 2 of H4
- added unit 3 of H4
- added unit 1 of H5
- added unit 4 of H5
- added unit 4 of H6
- added unit 1 of H6
- added H7: TOP_PWR, synth-custom:PinHeader_1x04_P2.54mm_Vertical, symbol Synth_Custom:CONN_Header_01x04
- added H8: BTM_PWR, synth-custom:PinSocket_1x04_P2.54mm_Vertical, symbol Synth_Custom:CONN_Socket_01x04
- added J4: INV_OUT, synth-custom:Jack_default, symbol Synth_Custom:Jack_default
- added R18: 1K, synth-custom:R_default, symbol Device:R
- added TP5, TP6, TP7, TP8, TP9: C, Connector_Pin:Pin_D1.0mm_L10.0mm, symbol Connector:TestPoint
- D1, D2: footprint Diode_THT:D_DO-41_SOD81_P10.16mm_Horizontal -> synth-custom:D_PWR_default
- D3: renamed from D6; footprint Diode_THT:D_DO-35_SOD27_P7.62mm_Horizontal -> synth-custom:D_default
- D4: renamed from D7; footprint Diode_THT:D_DO-35_SOD27_P7.62mm_Horizontal -> synth-custom:D_default
- H100: renamed from H7; footprint MountingHole:MountingHole_2.5mm -> MountingHole:MountingHole_3.2mm_M3
- H102: renamed from H8; footprint MountingHole:MountingHole_2.5mm -> MountingHole:MountingHole_3.2mm_M3
- H103: renamed from H9; footprint MountingHole:MountingHole_2.5mm -> MountingHole:MountingHole_3.2mm_M3
- H104: renamed from H10; footprint MountingHole:MountingHole_2.5mm -> MountingHole:MountingHole_3.2mm_M3
- H105: renamed from H11; footprint MountingHole:MountingHole_2.5mm -> MountingHole:MountingHole_3.2mm_M3
- H106: renamed from H12; footprint MountingHole:MountingHole_2.5mm -> MountingHole:MountingHole_3.2mm_M3
- H107: renamed from H13; footprint MountingHole:MountingHole_2.5mm -> MountingHole:MountingHole_3.2mm_M3
- H108: renamed from H14; footprint MountingHole:MountingHole_2.5mm -> MountingHole:MountingHole_3.2mm_M3
- H3: renamed from H2; value ~ -> BTM_SW; footprint synth-custom:PinSocket_1x04_P2.00mm_Vertical -> synth-custom:PinSocket_1x04_P2.54mm_Vertical
- H4: renamed from H1; value ~ -> TOP_SW; footprint synth-custom:PinHeader_1x04_P2.00mm_Vertical -> synth-custom:PinHeader_1x04_P2.54mm_Vertical
- H5: renamed from H6; value BTM_8_SGL -> BTM_OUT; footprint synth-custom:PinSocket_1x04_P2.00mm_Vertical -> synth-custom:PinSocket_1x04_P2.54mm_Vertical
- H6: renamed from H5; value BTM_8_SGL -> TOP_OUT; footprint synth-custom:PinHeader_1x04_P2.00mm_Vertical -> synth-custom:PinHeader_1x04_P2.54mm_Vertical
- J1: symbol Synth_Custom:Conn_02x08_PWR_Eurorack -> Synth_Custom:CONN_02x08_PWR_Eurorack
- J2: renamed from J4; footprint synth-custom:Jack_3.5mm_QingPu_WQP-PJ398SM_Vertical_CircularHoles -> synth-custom:Jack_default; symbol Synth_Custom:AudioJack2_PJ398SM -> Synth_Custom:Jack_default
- Q1: footprint Package_TO_SOT_THT:TO-92_Inline -> Package_TO_SOT_THT:TO-92_HandSolder
- R1: renamed from R18; footprint synth-custom:R_Axial_DIN0207_L6.3mm_D2.5mm_P7.62mm_Horizontal -> synth-custom:R_default
- R2: renamed from R1; footprint synth-custom:R_Axial_DIN0207_L6.3mm_D2.5mm_P7.62mm_Horizontal -> synth-custom:R_default
- R3: renamed from R2; footprint synth-custom:R_Axial_DIN0207_L6.3mm_D2.5mm_P7.62mm_Horizontal -> synth-custom:R_default
- R4: renamed from R17; footprint synth-custom:R_Axial_DIN0207_L6.3mm_D2.5mm_P7.62mm_Horizontal -> synth-custom:R_default
- R5: renamed from R15; footprint synth-custom:R_Axial_DIN0207_L6.3mm_D2.5mm_P7.62mm_Horizontal -> synth-custom:R_default
- SW1: footprint synth-custom:SPDT_Toggle -> synth-custom:SW_default
- TP1: renamed from TP2; footprint TestPoint:TestPoint_Plated_Hole_D2.0mm -> Connector_Pin:Pin_D1.0mm_L10.0mm
- TP2: renamed from TP3; footprint TestPoint:TestPoint_Plated_Hole_D2.0mm -> Connector_Pin:Pin_D1.0mm_L10.0mm
- renumbered C9 to C1, C10 to C2, C5 to C3, C6 to C4, C1 to C5, C2 to C6, C3 to C7, C4 to C8, C7 to C9, D9 to D5, U2 to U1, U1 to U2
Connections:
- net +12V: now also TP5.1
- net -12V: now also TP7.1
- net GNDREF: now also H7.1, H7.2, H7.3, H7.4, H8.1, H8.2, H8.3, H8.4, J4.S, TP6.1
- net feedback_loop/feedback_input: now also H5.3, U2.1, U2.2 (-); no longer H5.2, U2.6 (-), U2.7
- net feedback_loop/feedback_output: now also H3.3; no longer SW1.1 (A)
- net at ATT1.2, ATT1.3, SUS/REL1.2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: now also H6.2; no longer H6.1
- net at R5.2: now also H6.3; no longer H6.2
- net at D3.2 (A), D4.1 (K): now also H4.2, TP9.1
- net at C9.1, C9_OPT1.1: now also H5.2, U2.3 (+), TP8.1; no longer H5.1, U2.5 (+)
- net at R1.2: now also H3.2
- net at TP1.1, U1.10 (+): now also H3.1; no longer H3.3
- net at R4.2: now also H6.1
- net input_sustain/gate_in: now reaches J1.15 (GATE)
- net input_sustain/gate_in: now also J1.16 (GATE)
- net at SW1.2 (B): now also H4.1; no longer H4.3
- net at Q1.3 (E): now also H5.1
- new net: J4.T, R18.2
- new net: H6.4, R18.1
- new net: H4.3, SW1.1 (A)
- new net inverted_out/inv_output: H5.4
- no-connect marks 13 -> 12
Other:
- sheet input_sustain ports: added gate_in; removed none
- sheet inverted_out ports: added inv_output; removed none
- note added: "2"
- note added: "21.04.2024"
- note added: "Maybe this requires a diode & resistor to pull down?"
- note added: "Scribble"
- note added: "Sribble"
- moved on the sheet: C5, C7, D1, H3D, H4D, H5C, H6C, J2, R2, R5

Commit message: sensei models, scribble fixes
Parts:
- added TP10: INV_OUT, Connector_Pin:Pin_D1.0mm_L10.0mm, symbol Connector:TestPoint
- ATT1, SUS/REL1: footprint Potentiometer_THT:Potentiometer_TT_P0915N -> Synth:Potentiometer_TT_P0915N; symbol Device:R_Potentiometer -> synth:R_Potentiometer (P0915N)
- C9, C9_OPT1: footprint synth-custom:C_RECT_MKT_1uF -> Synth:C_RECT_MKT_1uF; symbol Device:C -> synth:C_1uF (MKS)
- D1, D2: footprint synth-custom:D_PWR_default -> Synth:D_DO-41_SOD81_P10.16mm_Horizontal; symbol Diode:1N5819 -> synth:D_Schottky (1N5819)
- D3, D4: footprint synth-custom:D_default -> Synth:D_DO-35_SOD27_P7.62mm_Horizontal; symbol Diode:1N4148 -> synth:D_Signal (1N4148)
- H3, H5, H8: footprint synth-custom:PinSocket_1x04_P2.54mm_Vertical -> Synth:PinSocket_1x04_P2.54mm_Vertical; symbol Synth_Custom:CONN_Socket_01x04 -> synth:PinSocket_01x04
- H4, H6, H7: footprint synth-custom:PinHeader_1x04_P2.54mm_Vertical -> Synth:PinHeader_1x04_P2.54mm_Vertical; symbol Synth_Custom:CONN_Header_01x04 -> synth:PinHeader_01x04
- J1: footprint synth-custom:CONN_02x08_PWR -> Synth:IDC-Header_2x08_P2.54mm_Vertical; symbol Synth_Custom:CONN_02x08_PWR_Eurorack -> synth:Conn_02x08_EuroRack_Power
- J2, J4: footprint synth-custom:Jack_default -> Synth:Jack_3.5mm_QingPu_WQP-PJ398SM_Vertical_CircularHoles; symbol Synth_Custom:Jack_default -> synth:AudioJack_Mono_3.5mm
- R1, R18, R2, R3, R4, R5: footprint synth-custom:R_default -> Synth:R_Default (DIN0207); symbol Device:R -> synth:R_Default
- SW1: footprint synth-custom:SW_default -> Synth:SW_default; symbol Synth_Custom:SW_SPDT -> synth:SW_SPDT
- TP1: value B -> TRG_INPUT
- TP2: value C -> OUT
- TP8: value C -> CAP_OUT
- TP9: value C -> CAP_IN
Connections:
- net +12V: now also R2.1; no longer R2.2
- net -12V: now also R3.1; no longer R3.2
- net inverted_out/inv_output: now also TP10.1
- net at R5.1: now also H6.3 (Pin_3); no longer J2.T
- net at R5.2: now also J2.T; no longer H6.3
- net at D2.2 (A): now also R3.2; no longer R3.1
- net at D5.2 (A): now also R4.2; no longer R4.1
- net at J4.T: now also R18.1; no longer R18.2
- net at D1.1 (K): now also R2.2; no longer R2.1
- net at U1.8, U1.9 (-): now also R1.2; no longer R1.1
- net at H3.2 (Pin_2): now also R1.1; no longer R1.2
- net at H6.1 (Pin_1): now also R4.1; no longer R4.2
- net at H6.4 (Pin_4): now also R18.2; no longer R18.1
Other:
- moved on the sheet: ATT1, C1, C2, C3, C4, C5, C6, C7, C8, C9, C9_OPT1, D1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

Commit message: cleaning up the main readme, update for 3340-vco
Parts:
- added J5: Conn_01x03, Connector_PinHeader_2.54mm:PinHeader_1x03_P2.54mm_Vertical, symbol Connector_Generic:Conn_01x03
Connections:
- net input_sustain/gate_in: now also J5.2 (Pin_2); no longer J1.15 (GATE), J1.16 (GATE)
- new net: J1.15 (GATE), J1.16 (GATE), J5.3 (Pin_3)
- no-connect marks 12 -> 13
Other:
- note removed: "Maybe this requires a diode & resistor to pull down?"
Changed lines of the file:
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@@
 	)
 	(no_connect
+		(at 95.25 226.06)
+	)
+	(no_connect
 		(at 388.62 226.06)
 	)
@@
 	(wire
 		(pts
-			(xy 21.59 93.98) (xy 21.59 229.87)
+			(xy 21.59 93.98) (xy 21.59 228.6)
 		)
 		(stroke
@@
 	(wire
 		(pts
+			(xy 100.33 233.68) (xy 157.48 233.68)
+		)
+		(stroke
+			(width 0)
+			(type default)
+		)
+	)
+	(wire
+		(pts
 			(xy 125.73 275.59) (xy 139.7 275.59)
 		)
@@
 	(wire
 		(pts
-			(xy 21.59 229.87) (xy 157.48 229.87)
+			(xy 21.59 228.6) (xy 97.79 228.6)
 		)
 		(stroke
@@
 	(wire
 		(pts
+			(xy 100.33 226.06) (xy 100.33 233.68)
+		)
+		(stroke
+			(width 0)
+			(type default)
+		)
+	)
+	(wire
+		(pts
 			(xy 349.25 95.25) (xy 351.79 95.25)
 		)
@@
 	(wire
 		(pts
+			(xy 97.79 228.6) (xy 97.79 226.06)
+		)
+		(stroke
+			(width 0)
+			(type default)
+		)
+	)
+	(wire
+		(pts
 			(xy 283.21 273.05) (xy 286.385 273.05)
 		)
@@
 	(wire
 		(pts
-			(xy 157.48 229.87) (xy 157.48 246.38)
+			(xy 157.48 233.68) (xy 157.48 246.38)
 		)
 		(stroke
@@
 		)
 	)
-	(text "Maybe this requires a diode & resistor to pull down?"
-		(exclude_from_sim no)
-		(at 125.095 228.6 0)
-		(effects
-			(font
-				(size 1.27 1.27)
-			)
-			(justify left bottom)
-		)
-	)
 	(text "Scribble"
 		(exclude_from_sim no)
@@
 					(unit 1)
 				)
+			)
+		)
+	)
+	(symbol
+		(lib_id "Connector_Generic:Conn_01x03")
+		(at 97.79 220.98 90)
+		(unit 1)
+		(exclude_from_sim no)
+		(in_bom yes)
+		(on_board yes)
+		(dnp no)
+		(fields_autoplaced yes)
+		(property "Reference" "J5"
+			(at 102.87 219.7099 90)
+			(effects
+				(font
+					(size 1.27 1.27)
+				)
+				(justify right)
+			)
+		)
+		(property "Value" "Conn_01x03"
+			(at 102.87 222.2499 90)
+			(effects
+				(font
+					(size 1.27 1.27)
+				)
+				(justify right)
+			)
+		)
+		(property "Footprint" "Connector_PinHeader_2.54mm:PinHeader_1x03_P2.54mm_Vertical"
+			(at 97.79 220.98 0)
+			(effects
+				(font
+					(size 1.27 1.27)
+				)
+				(hide yes)
+			)
+		)
+		(property "Datasheet" "~"
+			(at 97.79 220.98 0)
+			(effects
+				(font
+					(size 1.27 1.27)
+				)
+				(hide yes)
+			)
+		)
+		(property "Description" "Generic connector, single row, 01x03, script generated (kicad-library-utils/schlib/autogen/connector/)"
+			(at 97.79 220.98 0)
+			(effects
+				(font
+					(size 1.27 1.27)
+				)
+				(hide yes)
+			)
+		)
+		(pin "2"
+		)
+		(pin "1"
+		)
+		(pin "3"
+		)
+		(instances
+			(project "scribble"
+				(path "/ffcc7acb-943e-4c85-833d-d9691a289ebb"
+					(reference "J5")
+					(unit 1)
+				)

Commit message: update to BOM and add panels
Parts:
- C1, C2, C3, C4: footprint Capacitor_THT:CP_Radial_D4.0mm_P2.00mm -> Capacitor_THT:C_Disc_D5.0mm_W2.5mm_P5.00mm; symbol Device:C_Polarized -> Device:C
- H100, H102, H103, H104, H105, H106, H107, H108, TP1, TP10, TP2, TP5, TP6, TP7, TP8, TP9: now left out of the parts list
- H3: value BTM_SW -> PinSocket_1x04
- H4: value TOP_SW -> PinHeader_1x04
- H5: value BTM_OUT -> PinSocket_1x04
- H6: value TOP_OUT -> PinHeader_1x04
- H7: value TOP_PWR -> PinHeader_1x04
- H8: value BTM_PWR -> PinSocket_1x04
- J5: value Conn_01x03 -> PinHeader_1x03
- R1: value 100 -> 100R
- R2, R3: value 10 -> 10R
- R4: value 470 -> 470R
Changed lines of the file:
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@@
 		(unit 1)
 		(exclude_from_sim no)
-		(in_bom yes)
+		(in_bom no)
 		(on_board yes)
 		(dnp no)
@@
 		(unit 1)
 		(exclude_from_sim no)
-		(in_bom yes)
+		(in_bom no)
 		(on_board yes)
 		(dnp no)
@@
 		(unit 1)
 		(exclude_from_sim no)
-		(in_bom yes)
+		(in_bom no)
 		(on_board yes)
 		(dnp no)
@@
 			)
 		)
-		(property "Value" "BTM_OUT"
+		(property "Value" "PinSocket_1x04"
 			(at 245.11 95.25 0)
 			(effects
@@
 	)
 	(symbol
-		(lib_id "Device:C_Polarized")
+		(lib_id "Device:C")
 		(at 125.73 271.78 0)
 		(unit 1)
@@
 		(fields_autoplaced yes)
 		(property "Reference" "C4"
-			(at 129.54 269.621 0)
+			(at 129.54 270.5099 0)
 			(effects
 				(font
@@
 		)
 		(property "Value" "0.1uF"
-			(at 129.54 272.161 0)
+			(at 129.54 273.0499 0)
 			(effects
 				(font
@@
 			)
 		)
-		(property "Footprint" "Capacitor_THT:CP_Radial_D4.0mm_P2.00mm"
+		(property "Footprint" "Capacitor_THT:C_Disc_D5.0mm_W2.5mm_P5.00mm"
 			(at 126.6952 275.59 0)
 			(effects
@@
 			)
 		)
-		(property "Description" "Polarized capacitor"
+		(property "Description" "Unpolarized capacitor"
 			(at 125.73 271.78 0)
 			(effects
@@
 			)
 		)
-		(property "Value" "BTM_OUT"
+		(property "Value" "PinSocket_1x04"
 			(at 339.09 92.71 0)
 			(effects
@@
 			)
 		)
-		(property "Value" "TOP_PWR"
+		(property "Value" "PinHeader_1x04"
 			(at 266.065 266.7 0)
 			(effects
@@
 			)
 		)
-		(property "Value" "TOP_SW"
+		(property "Value" "PinHeader_1x04"
 			(at 175.895 99.06 0)
 			(effects
@@
 			)
 		)
-		(property "Value" "BTM_PWR"
+		(property "Value" "PinSocket_1x04"
 			(at 278.13 271.78 0)
 			(effects
@@
 		(unit 1)
 		(exclude_from_sim no)
-		(in_bom yes)
+		(in_bom no)
 		(on_board yes)
 		(dnp no)
@@
 			)
 		)
-		(property "Value" "10"
+		(property "Value" "10R"
 			(at 198.12 278.765 90)
 			(effects
@@
 			)
 		)
-		(property "Value" "TOP_OUT"
+		(property "Value" "PinHeader_1x04"
 			(at 241.3 90.17 0)
 			(effects
@@
 	)
 	(symbol
-		(lib_id "Device:C_Polarized")
+		(lib_id "Device:C")
 		(at 82.55 254 0)
 		(unit 1)
@@
 		(fields_autoplaced yes)
 		(property "Reference" "C1"
-			(at 86.36 251.841 0)
+			(at 86.36 252.7299 0)
 			(effects
 				(font
@@
 		)
 		(property "Value" "0.1uF"
-			(at 86.36 254.381 0)
+			(at 86.36 255.2699 0)
 			(effects
 				(font
@@
 			)
 		)
-		(property "Footprint" "Capacitor_THT:CP_Radial_D4.0mm_P2.00mm"
+		(property "Footprint" "Capacitor_THT:C_Disc_D5.0mm_W2.5mm_P5.00mm"
 			(at 83.5152 257.81 0)
 			(effects
@@
 			)
 		)
-		(property "Description" "Polarized capacitor"
+		(property "Description" "Unpolarized capacitor"
 			(at 82.55 254 0)
 			(effects
@@
 			)
 		)
-		(property "Value" "BTM_SW"
+		(property "Value" "PinSocket_1x04"
 			(at 170.18 91.44 0)
 			(effects
@@
 			)
 		)
-		(property "Value" "BTM_PWR"
+		(property "Value" "PinSocket_1x04"
 			(at 278.13 275.59 0)
 			(effects
@@
 			)
 		)
-		(property "Value" "470"
+		(property "Value" "470R"
 			(at 334.01 62.23 90)
 			(effects
@@
 		(unit 1)
 		(exclude_from_sim no)
-		(in_bom yes)
+		(in_bom no)
 		(on_board yes)
 		(dnp no)
@@
 	)
 	(symbol
-		(lib_id "Device:C_Polarized")
+		(lib_id "Device:C")
 		(at 125.73 254 0)
 		(unit 1)
@@
 		(fields_autoplaced yes)
 		(property "Reference" "C3"
-			(at 129.54 251.841 0)
+			(at 129.54 252.7299 0)
 			(effects
 				(font
@@
 		)
 		(property "Value" "0.1uF"
-			(at 129.54 254.381 0)
+			(at 129.54 255.2699 0)
 			(effects
 				(font
@@
 			)
 		)
-		(property "Footprint" "Capacitor_THT:CP_Radial_D4.0mm_P2.00mm"
+		(property "Footprint" "Capacitor_THT:C_Disc_D5.0mm_W2.5mm_P5.00mm"
 			(at 126.6952 257.81 0)
 			(effects
@@
 			)
 		)
-		(property "Description" "Polarized capacitor"
+		(property "Description" "Unpolarized capacitor"
 			(at 125.73 254 0)
 			(effects
@@
 			)
 		)
-		(property "Value" "BTM_SW"
+		(property "Value" "PinSocket_1x04"
 			(at 102.87 113.665 0)
 			(effects
@@
 			)
 		)
-		(property "Value" "TOP_PWR"
+		(property "Value" "PinHeader_1x04"
 			(at 266.065 270.51 0)
 			(effects
@@
 			)
 		)
-		(property "Value" "BTM_SW"
+		(property "Value" "PinSocket_1x04"
 			(at 124.46 99.06 0)
 			(effects
@@
 		(unit 1)
 		(exclude_from_sim no)
-		(in_bom yes)
+		(in_bom no)
 		(on_board yes)
 		(dnp no)
@@
 			)
 		)
-		(property "Value" "BTM_OUT"
+		(property "Value" "PinSocket_1x04"
 			(at 316.23 62.23 0)
 			(effects
@@
 		(unit 1)
 		(exclude_from_sim no)
-		(in_bom yes)
+		(in_bom no)
 		(on_board yes)
 		(dnp no)
@@
 		(unit 1)
 		(exclude_from_sim no)
-		(in_bom yes)
+		(in_bom no)
 		(on_board yes)
 		(dnp no)
@@
 	)
 	(symbol
-		(lib_id "Device:C_Polarized")
+		(lib_id "Device:C")
 		(at 82.55 271.78 0)
 		(unit 1)
@@
 		(fields_autoplaced yes)
 		(property "Reference" "C2"
-			(at 86.36 269.621 0)
+			(at 86.36 270.5099 0)
 			(effects
 				(font
@@
 		)
 		(property "Value" "0.1uF"
-			(at 86.36 272.161 0)
+			(at 86.36 273.0499 0)
 			(effects
 				(font
@@
 			)
 		)
-		(property "Footprint" "Capacitor_THT:CP_Radial_D4.0mm_P2.00mm"
+		(property "Footprint" "Capacitor_THT:C_Disc_D5.0mm_W2.5mm_P5.00mm"
 			(at 83.5152 275.59 0)
 			(effects
@@
 			)
 		)
-		(property "Description" "Polarized capacitor"
+		(property "Description" "Unpolarized capacitor"
 			(at 82.55 271.78 0)
 			(effects
@@
 			)
 		)
-		(property "Value" "TOP_SW"
+		(property "Value" "PinHeader_1x04"
 			(at 111.125 109.855 0)
 			(effects
@@
 		(unit 1)
 		(exclude_from_sim no)
-		(in_bom yes)
+		(in_bom no)
 		(on_board yes)
 		(dnp no)
@@
 			)
 		)
-		(property "Value" "TOP_SW"
+		(property "Value" "PinHeader_1x04"
 			(at 120.65 85.09 0)
 			(effects
@@
 			)
 		)
-		(property "Value" "Conn_01x03"
+		(property "Value" "PinHeader_1x03"
 			(at 102.87 222.2499 90)
 			(effects
@@
 			)
 		)
-		(property "Value" "TOP_PWR"
+		(property "Value" "PinHeader_1x04"
 			(at 266.065 274.32 0)
 			(effects
@@
 		(unit 1)
 		(exclude_from_sim no)
-		(in_bom yes)
+		(in_bom no)
 		(on_board yes)
 		(dnp no)
@@
 			)
 		)
-		(property "Value" "BTM_PWR"
+		(property "Value" "PinSocket_1x04"
 			(at 278.13 279.4 0)
 			(effects
@@
 			)
 		)
-		(property "Value" "BTM_SW"
+		(property "Value" "PinSocket_1x04"
 			(at 278.13 261.62 0)
 			(effects
@@
 			)
 		)
-		(property "Value" "100"
+		(property "Value" "100R"
 			(at 157.48 90.17 90)
 			(effects
@@
 			)
 		)
-		(property "Value" "BTM_OUT"
+		(property "Value" "PinSocket_1x04"
 			(at 351.155 123.19 0)
 			(effects
@@
 			)
 		)
-		(property "Value" "BTM_PWR"
+		(property "Value" "PinSocket_1x04"
 			(at 278.13 267.97 0)
 			(effects
@@
 			)
 		)
-		(property "Value" "TOP_OUT"
+		(property "Value" "PinHeader_1x04"
 			(at 344.17 97.79 0)
 			(effects
@@
 		(unit 1)
 		(exclude_from_sim no)
-		(in_bom yes)
+		(in_bom no)
 		(on_board yes)
 		(dnp no)
@@
 		(unit 1)
 		(exclude_from_sim no)
-		(in_bom yes)
+		(in_bom no)
 		(on_board yes)
 		(dnp no)
@@
 		(unit 1)
 		(exclude_from_sim no)
-		(in_bom yes)
+		(in_bom no)
 		(on_board yes)
 		(dnp no)
@@
 			)
 		)
-		(property "Value" "TOP_OUT"
+		(property "Value" "PinHeader_1x04"
 			(at 356.235 128.27 0)
 			(effects
@@
 		(unit 1)
 		(exclude_from_sim no)
-		(in_bom yes)
+		(in_bom no)
 		(on_board yes)
 		(dnp no)
@@
 			)
 		)
-		(property "Value" "TOP_SW"
+		(property "Value" "PinHeader_1x04"
 			(at 266.065 256.54 0)
 			(effects
@@
 			)
 		)
-		(property "Value" "TOP_OUT"
+		(property "Value" "PinHeader_1x04"
 			(at 320.04 67.31 0)
 			(effects
@@
 		(unit 1)
 		(exclude_from_sim no)
-		(in_bom yes)
+		(in_bom no)
 		(on_board yes)
 		(dnp no)
@@
 		(fields_autoplaced yes)
 		(property "Reference" "R2"
-			(at 198.12 243.205 90)
+			(at 198.12 243.84 90)
 			(effects
 				(font
@@
 			)
 		)
-		(property "Value" "10"
-			(at 198.12 245.745 90)
+		(property "Value" "10R"
+			(at 198.12 246.38 90)
 			(effects
 				(font
@@
 			)
 		)
-		(property "Value" "TOP_PWR"
+		(property "Value" "PinHeader_1x04"
 			(at 266.065 262.89 0)
 			(effects
@@
 		(unit 1)
 		(exclude_from_sim no)
-		(in_bom yes)
+		(in_bom no)
 		(on_board yes)
 		(dnp no)

Commit message: finish all panels, update build status, add ibom and small fixes
Connections:
- net GNDREF: now also U2.12 (+), U2.9 (-)
- net at U2.13 (-): now also U2.14
- net at U2.10 (+): now also U2.8
- no-connect marks 13 -> 7
Other:
- moved on the sheet: U2D
