File: modules/active-mixers/1-distored-daisy/kiCad/active_mixer.kicad_sch (KiCad schematic)
At the start: 72 parts, among them J1 INPUT_1, J2 INPUT_2, J3 INPUT_3, J4 INPUT_4, J5 OUTPUT, J6 OUTPUT, Q1 BC547, Q2 BC547, Q3 BC547, Q4 BC547, Q5 BC547, U1 TL074

Commit message: comments on schematic
Other:
- note added: "Might be better to have this as a TrimPot"
Changed lines of the file:
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@@
     (fill (type none))
+  )
+  (text "Might be better to have this as a TrimPot" (at 259.08 147.32 0)
+    (effects (font (size 1.27 1.27)) (justify left bottom))
   )
   (symbol (lib_id "Transistor_BJT:BC547") (at 104.14 93.98 90) (unit 1)
