File: modules/active-mixers/1-distored-daisy/kiCad/distorted_daisy.kicad_sch (KiCad schematic)
At the start: 79 parts, among them J1 INPUT_1, J2 INPUT_2, J3 INPUT_3, J4 INPUT_4, J5 OUTPUT, J6 INV_OUT, Q1 BC547, Q2 BC547, Q3 BC547, Q4 BC547, Q5 BC547, U1 TL074

Commit message: cleaning up the main readme, update for 3340-vco
Parts:
- D3: value LED_IN_1 -> RED_IN_1_20mA
- D4: value LED_IN_2 -> RED_IN_2_20mA
- D5: value LED_IN_3 -> RED_IN_3_20mA
- D6: value LED_IN_4 -> RED_IN_4_20mA
- D7: value LED_OUT -> YELLOW_OUT_20mA
- J6: value INV_OUT -> DIST_OUT
- R12, R19, R3, R6, R9: value 1K -> 680R
Other:
- note added: "I think this R is too much here"
Changed lines of the file:
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@@
 		)
 	)
+	(text "I think this R is too much here"
+		(exclude_from_sim no)
+		(at 107.442 153.67 0)
+		(effects
+			(font
+				(size 1.27 1.27)
+			)
+		)
+	)
+	(text "I think this R is too much here"
+		(exclude_from_sim no)
+		(at 109.728 99.06 0)
+		(effects
+			(font
+				(size 1.27 1.27)
+			)
+		)
+	)
+	(text "I think this R is too much here"
+		(exclude_from_sim no)
+		(at 372.11 31.75 0)
+		(effects
+			(font
+				(size 1.27 1.27)
+			)
+		)
+	)
+	(text "I think this R is too much here"
+		(exclude_from_sim no)
+		(at 107.442 204.724 0)
+		(effects
+			(font
+				(size 1.27 1.27)
+			)
+		)
+	)
+	(text "I think this R is too much here"
+		(exclude_from_sim no)
+		(at 107.442 46.99 0)
+		(effects
+			(font
+				(size 1.27 1.27)
+			)
+		)
+	)
 	(symbol
 		(lib_id "Transistor_BJT:BC547")
@@
 			)
 		)
-		(property "Value" "1K"
+		(property "Value" "680R"
 			(at 66.04 86.36 90)
 			(effects
@@
 			)
 		)
-		(property "Value" "1K"
+		(property "Value" "680R"
 			(at 64.77 34.29 90)
 			(effects
@@
 			)
 		)
-		(property "Value" "LED_OUT"
+		(property "Value" "YELLOW_OUT_20mA"
 			(at 336.8675 17.78 0)
 			(effects
@@
 			)
 		)
-		(property "Value" "1K"
+		(property "Value" "680R"
 			(at 63.5 193.04 90)
 			(effects
@@
 			)
 		)
-		(property "Value" "1K"
+		(property "Value" "680R"
 			(at 63.5 140.97 90)
 			(effects
@@
 			)
 		)
-		(property "Value" "INV_OUT"
+		(property "Value" "DIST_OUT"
 			(at 393.7 110.5534 0)
 			(effects
@@
 			)
 		)
-		(property "Value" "LED_IN_1"
+		(property "Value" "RED_IN_1_20mA"
 			(at 76.5175 33.02 0)
 			(effects
@@
 		(fields_autoplaced yes)
 		(property "Reference" "R19"
-			(at 325.12 17.145 90)
+			(at 325.12 16.51 90)
 			(effects
 				(font
@@
 			)
 		)
-		(property "Value" "1K"
-			(at 325.12 19.685 90)
+		(property "Value" "680R"
+			(at 325.12 19.05 90)
 			(effects
 				(font
@@
 			)
 		)
-		(property "Value" "LED_IN_2"
+		(property "Value" "RED_IN_2_20mA"
 			(at 77.7875 85.09 0)
 			(effects
@@
 			)
 		)
-		(property "Value" "LED_IN_4"
+		(property "Value" "RED_IN_4_20mA"
 			(at 75.2475 191.77 0)
 			(effects
@@
 			)
 		)
-		(property "Value" "LED_IN_3"
+		(property "Value" "RED_IN_3_20mA"
 			(at 75.2475 139.7 0)
 			(effects

Commit message: finish all panels, update build status, add ibom and small fixes
Parts:
- H10, H11, H12, H13, H5, H6, H7, H8, TP1, TP10, TP11, TP2, TP3, TP4, TP5, TP6, TP7, TP8, TP9: now left out of the parts list
- R1, R2: value 10 -> 10R
Connections:
- net GNDREF: now also U1.12 (+)
- net at U1.13 (-): now also U1.14
- no-connect marks 9 -> 6
Other:
- note removed: "I think this R is too much here"
Changed lines of the file:
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@@
 	)
 	(no_connect
-		(at 267.97 247.65)
-	)
-	(no_connect
 		(at 41.91 215.9)
 	)
@@
 	)
 	(no_connect
-		(at 283.21 250.19)
-	)
-	(no_connect
 		(at 52.07 109.22)
 	)
@@
 		(at 384.81 106.68)
 	)
-	(no_connect
-		(at 267.97 252.73)
-	)
 	(wire
 		(pts
@@
 	(wire
 		(pts
+			(xy 267.97 252.73) (xy 267.97 256.54)
+		)
+		(stroke
+			(width 0)
+			(type default)
+		)
+	)
+	(wire
+		(pts
 			(xy 328.93 43.18) (xy 328.93 59.69)
 		)
@@
 	(wire
 		(pts
+			(xy 283.21 256.54) (xy 283.21 250.19)
+		)
+		(stroke
+			(width 0)
+			(type default)
+		)
+	)
+	(wire
+		(pts
 			(xy 306.07 77.47) (xy 306.07 62.23)
 		)
@@
 	(wire
 		(pts
+			(xy 267.97 256.54) (xy 283.21 256.54)
+		)
+		(stroke
+			(width 0)
+			(type default)
+		)
+	)
+	(wire
+		(pts
 			(xy 314.96 77.47) (xy 306.07 77.47)
 		)
@@
 	(wire
 		(pts
+			(xy 262.89 247.65) (xy 267.97 247.65)
+		)
+		(stroke
+			(width 0)
+			(type default)
+		)
+	)
+	(wire
+		(pts
 			(xy 347.98 109.22) (xy 347.98 121.92)
 		)
@@
 		)
 	)
-	(text "I think this R is too much here"
-		(exclude_from_sim no)
-		(at 107.442 153.67 0)
-		(effects
-			(font
-				(size 1.27 1.27)
-			)
-		)
-	)
-	(text "I think this R is too much here"
-		(exclude_from_sim no)
-		(at 109.728 99.06 0)
-		(effects
-			(font
-				(size 1.27 1.27)
-			)
-		)
-	)
-	(text "I think this R is too much here"
-		(exclude_from_sim no)
-		(at 372.11 31.75 0)
-		(effects
-			(font
-				(size 1.27 1.27)
-			)
-		)
-	)
-	(text "I think this R is too much here"
-		(exclude_from_sim no)
-		(at 107.442 204.724 0)
-		(effects
-			(font
-				(size 1.27 1.27)
-			)
-		)
-	)
-	(text "I think this R is too much here"
-		(exclude_from_sim no)
-		(at 107.442 46.99 0)
-		(effects
-			(font
-				(size 1.27 1.27)
-			)
-		)
-	)
 	(symbol
 		(lib_id "Transistor_BJT:BC547")
@@
 		(unit 1)
 		(exclude_from_sim no)
-		(in_bom yes)
+		(in_bom no)
 		(on_board yes)
 		(dnp no)
@@
 		(unit 1)
 		(exclude_from_sim no)
-		(in_bom yes)
+		(in_bom no)
 		(on_board yes)
 		(dnp no)
@@
 		(unit 1)
 		(exclude_from_sim no)
-		(in_bom yes)
+		(in_bom no)
 		(on_board yes)
 		(dnp no)
@@
 	)
 	(symbol
+		(lib_id "power:GNDREF")
+		(at 262.89 247.65 270)
+		(unit 1)
+		(exclude_from_sim no)
+		(in_bom yes)
+		(on_board yes)
+		(dnp no)
+		(fields_autoplaced yes)
+		(property "Reference" "#PWR037"
+			(at 256.54 247.65 0)
+			(effects
+				(font
+					(size 1.27 1.27)
+				)
+				(hide yes)
+			)
+		)
+		(property "Value" "GNDREF"
+			(at 259.08 247.6499 90)
+			(effects
+				(font
+					(size 1.27 1.27)
+				)
+				(justify right)
+			)
+		)
+		(property "Footprint" ""
+			(at 262.89 247.65 0)
+			(effects
+				(font
+					(size 1.27 1.27)
+				)
+				(hide yes)
+			)
+		)
+		(property "Datasheet" ""
+			(at 262.89 247.65 0)
+			(effects
+				(font
+					(size 1.27 1.27)
+				)
+				(hide yes)
+			)
+		)
+		(property "Description" "Power symbol creates a global label with name \"GNDREF\" , reference supply ground"
+			(at 262.89 247.65 0)
+			(effects
+				(font
+					(size 1.27 1.27)
+				)
+				(hide yes)
+			)
+		)
+		(pin "1"
+		)
+		(instances
+			(project "distorted_daisy"
+				(path "/ffcc7acb-943e-4c85-833d-d9691a289ebb"
+					(reference "#PWR037")
+					(unit 1)
+				)
+			)
+		)
+	)
+	(symbol
 		(lib_id "synth:R_Default")
 		(at 102.87 158.75 180)
@@
 		(unit 1)
 		(exclude_from_sim no)
-		(in_bom yes)
+		(in_bom no)
 		(on_board yes)
 		(dnp no)
@@
 		(unit 1)
 		(exclude_from_sim no)
-		(in_bom yes)
+		(in_bom no)
 		(on_board yes)
 		(dnp no)
@@
 			)
 		)
-		(property "Value" "10"
+		(property "Value" "10R"
 			(at 198.12 278.13 90)
 			(effects
@@
 		(unit 1)
 		(exclude_from_sim no)
-		(in_bom yes)
+		(in_bom no)
 		(on_board yes)
 		(dnp no)
@@
 		(unit 1)
 		(exclude_from_sim no)
-		(in_bom yes)
+		(in_bom no)
 		(on_board yes)
 		(dnp no)
@@
 		(unit 1)
 		(exclude_from_sim no)
-		(in_bom yes)
+		(in_bom no)
 		(on_board yes)
 		(dnp no)
@@
 		(unit 1)
 		(exclude_from_sim no)
-		(in_bom yes)
+		(in_bom no)
 		(on_board yes)
 		(dnp no)
@@
 		(unit 1)
 		(exclude_from_sim no)
-		(in_bom yes)
+		(in_bom no)
 		(on_board yes)
 		(dnp no)
@@
 		(unit 1)
 		(exclude_from_sim no)
-		(in_bom yes)
+		(in_bom no)
 		(on_board yes)
 		(dnp no)
@@
 		(unit 1)
 		(exclude_from_sim no)
-		(in_bom yes)
+		(in_bom no)
 		(on_board yes)
 		(dnp no)
@@
 		(unit 1)
 		(exclude_from_sim no)
-		(in_bom yes)
+		(in_bom no)
 		(on_board yes)
 		(dnp no)
@@
 		(unit 1)
 		(exclude_from_sim no)
-		(in_bom yes)
+		(in_bom no)
 		(on_board yes)
 		(dnp no)
@@
 		(unit 1)
 		(exclude_from_sim no)
-		(in_bom yes)
+		(in_bom no)
 		(on_board yes)
 		(dnp no)
@@
 		(unit 1)
 		(exclude_from_sim no)
-		(in_bom yes)
+		(in_bom no)
 		(on_board yes)
 		(dnp no)
@@
 		(unit 1)
 		(exclude_from_sim no)
-		(in_bom yes)
+		(in_bom no)
 		(on_board yes)
 		(dnp no)
@@
 			)
 		)
-		(property "Value" "10"
+		(property "Value" "10R"
 			(at 198.12 250.19 90)
 			(effects
@@
 		(unit 1)
 		(exclude_from_sim no)
-		(in_bom yes)
+		(in_bom no)
 		(on_board yes)
 		(dnp no)
@@
 		(unit 1)
 		(exclude_from_sim no)
-		(in_bom yes)
+		(in_bom no)
 		(on_board yes)
 		(dnp no)
