File: modules/utility/5-passive-mult/kiCad/passive-mult.kicad_sch (KiCad schematic)
At the start: 8 parts, among them J1 INPUT, J2 INPUT, J3 OUTPUT, J4 OUTPUT, J5 OUTPUT, J6 OUTPUT, J7 OUTPUT, J8 OUTPUT

Commit message: final versions of PCB for modules
Other:
- note added: "1"
- note added: "Lennart Querter"
- note added: "Passive Multiple"
- note added: "Passive Multiple REV.1"
- moved on the sheet: J1, J2, J3, J4, J5, J6, J7, J8
