File: modules/filters/1-3320/kiCad/3320.kicad_sch (KiCad schematic)
At the start: 52 parts, among them U2 TL072

Commit message: final versions of PCB for modules
Parts:
- removed CUT_OFF_CTRL_1: B100K, Synth:Potentiometer_TT_P0915N, symbol synth:R_Potentiometer (P0915N)
- removed CUT_OFF_CV_IN_1: INPUT, Synth:Jack_3.5mm_QingPu_WQP-PJ398SM_Vertical_CircularHoles, symbol synth:AudioJack_Mono_3.5mm
- removed R20: 51K, Synth:R_Default (DIN0207), symbol synth:R_Default
- removed R21, R22: 100K, Synth:R_Default (DIN0207), symbol synth:R_Default
- added C14: 1uF, Capacitor_THT:CP_Radial_D4.0mm_P2.00mm, symbol Device:C_Polarized
- added C15, C7, C8: 0.1uF, Capacitor_THT:C_Rect_L4.6mm_W2.0mm_P2.50mm_MKS02_FKP02, symbol Device:C
- added FREQ_CTRL_1: B100K, Synth:Potentiometer_TT_P0915N, symbol synth:R_Potentiometer (P0915N)
- added FREQ_CV_IN_1: INPUT, Synth:Jack_3.5mm_QingPu_WQP-PJ398SM_Vertical_CircularHoles, symbol synth:AudioJack_Mono_3.5mm
- added FREQ_CV_IN_LVL_1, OUT_LVL_1, RES_CV_IN_LVL_1: B100K, Synth:Potentiometer_Alpha_RD901F-40-00D_Single_Vertical_CircularHoles, symbol synth:R_Potentiometer (Alpha_9mm)
- added H10, H11, H12, H13, H14, H15, H8, H9: MountingHole, MountingHole:MountingHole_3.2mm_M3, symbol Mechanical:MountingHole
- added H2, H4: PinHeader_01x04, Synth:PinHeader_1x04_P2.54mm_Vertical, symbol synth:PinHeader_01x04
- added H3, H6: PinSocket_01x04, Synth:PinSocket_1x04_P2.54mm_Vertical, symbol synth:PinSocket_01x04
- added H5: PinHeader_01x04, Synth:PinSocket_1x02_P2.54mm_Vertical, symbol synth:PinSocket_01x02
- added H7: PinSocket_01x04, Synth:PinHeader_1x02_P2.54mm_Vertical, symbol synth:PinHeader_01x02
- added R10, R30, R6: 100K, Synth:R_Default (DIN0207), symbol synth:R_Default
- added R11, R29, R9: 68K, Synth:R_Default (DIN0207), symbol synth:R_Default
- added R12: 150K, Synth:R_Default (DIN0207), symbol synth:R_Default
- added R13: 100k, Synth:R_Default (DIN0207), symbol synth:R_Default
- added R14, R15: 1K8, Synth:R_Default (DIN0207), symbol synth:R_Default
- added R16: 91K, Synth:R_Default (DIN0207), symbol synth:R_Default
- added R31: 330K, Synth:R_Default (DIN0207), symbol synth:R_Default
- added R32: 51K, Synth:R_Default (DIN0207), symbol synth:R_Default
- added R33: 3K3, Synth:R_Default (DIN0207), symbol synth:R_Default
- added RV1, RV2, RV3: 50K, Synth:Potentiometer_Bourns_3296W_Vertical, symbol synth:R_Potentiometer_Trim (Bourns)
- added TP1: RES_IN, Connector_Pin:Pin_D1.0mm_L10.0mm, symbol Connector:TestPoint
- added TP10: OUT, Connector_Pin:Pin_D1.0mm_L10.0mm, symbol Connector:TestPoint
- added TP2: F_IN, Connector_Pin:Pin_D1.0mm_L10.0mm, symbol Connector:TestPoint
- added TP3: FREQ_CTRL, Connector_Pin:Pin_D1.0mm_L10.0mm, symbol Connector:TestPoint
- added TP4: RES_CTRL, Connector_Pin:Pin_D1.0mm_L10.0mm, symbol Connector:TestPoint
- added TP5: POLE_1, Connector_Pin:Pin_D1.0mm_L10.0mm, symbol Connector:TestPoint
- added TP6: POLE_2, Connector_Pin:Pin_D1.0mm_L10.0mm, symbol Connector:TestPoint
- added TP7: POLE_3, Connector_Pin:Pin_D1.0mm_L10.0mm, symbol Connector:TestPoint
- added TP8: POLE_4, Connector_Pin:Pin_D1.0mm_L10.0mm, symbol Connector:TestPoint
- added TP9: V_RES, Connector_Pin:Pin_D1.0mm_L10.0mm, symbol Connector:TestPoint
- added unit 2 of U1
- added unit 3 of U1
- added unit 4 of U2
- added unit 2 of U2
- added unit 3 of U2
- IN_LVL_1, IN_LVL_2: footprint Synth:Potentiometer_TT_P0915N -> Synth:Potentiometer_Alpha_RD901F-40-00D_Single_Vertical_CircularHoles; symbol synth:R_Potentiometer (P0915N) -> synth:R_Potentiometer (Alpha_9mm)
- R5: value 1K8 -> 100K
- R7: renamed from R3; value 91K -> 100K
- R8: renamed from R4; value 91K -> 100K
- U2: value TL072 -> TL074; footprint Package_DIP:DIP-8_W7.62mm_Socket_LongPads -> Package_DIP:DIP-14_W7.62mm_Socket_LongPads; symbol Amplifier_Operational:TL072 -> Amplifier_Operational:TL074
- renumbered C4 to C10, C7 to C11, C8 to C12, C9 to C13, C5 to C3, C6 to C4, C10 to C5, C11 to C6, C3 to C9, OUTPUT_1 to OUT_1, R8 to R17, R9 to R18, R10 to R19, R11 to R20, R12 to R21, R13 to R22, R14 to R23, R15 to R24, R16 to R25, R17 to R26, R18 to R27, R19 to R28, R6 to R3, R23 to R34, R7 to R4, TP1 to TP11, TP2 to TP12, TP3 to TP13, U2 to U1, U1 to U3
Connections:
- net +12V: now also U2.4 (V+), C15.2, C7.1, H4.1 (Pin_1), H6.1 (Pin_1), U1.8 (V+); no longer U2.8 (V+)
- net -12V: now also U2.11 (V-), C8.2, FREQ_CTRL_1.3, H4.4 (Pin_4), H6.4 (Pin_4), U1.4 (V-); no longer U2.4 (V-)
- net GNDREF: now also C15.1, C7.2, C8.1, FREQ_CTRL_1.1, FREQ_CV_IN_1.S, FREQ_CV_IN_LVL_1.3, H2.4 (Pin_4), H3.4 (Pin_4), H4.2 (Pin_2), H4.3 (Pin_3), H5.2 (Pin_2), H6.2 (Pin_2), H6.3 (Pin_3), H7.2 (Pin_2), OUT_LVL_1.1, R14.2, R29.1, R30.1, R33.2, RES_CV_IN_LVL_1.3, RV3.2, RV3.3, U1.5 (+), U2.10 (+), U2.5 (+); no longer R5.2
- net at R7.1, R8.1: now also H2.1 (Pin_1); no longer R17.2, U3.1 (INPUT_A)
- net at RES_CV_IN_1.T: now also RES_CV_IN_LVL_1.1
- net at R23.1, R24.2, U3.15 (OUT_C): now also TP7.1
- net at U3.9 (RES_CTRL): now also R12.1, R15.1, TP4.1
- net at RES_CTRL_1.2: now also R2.2
- net at R1.1, R2.1: now also H2.3 (Pin_3); no longer R5.1, U3.12 (FREQ_CTRL)
- net at U1.1: now also R10.2, R9.2; no longer U1.2 (-)
- net at R20.1, R21.2, U3.6 (OUT_B): now also TP6.1
- net at C13.1, R26.1, U3.10 (OUT_D): now also TP8.1
- net at R17.1, R18.2, U3.7 (OUT_A): now also TP5.1
- net at U3.8 (V_RES): now also R32.2, R33.1, TP9.1
- net at C13.2: now also U2.3 (+), R29.2; no longer U2.5 (+)
- net at R1.2: now also RES_CV_IN_LVL_1.2
- new net: OUT_LVL_1.2, R34.1
- new net: H7.1 (Pin_1), OUT_LVL_1.3
- new net: C14.1, H5.1 (Pin_1), R31.1, TP10.1, U2.1
- new net: H3.1 (Pin_1), U2.12 (+)
- new net: R16.2, TP2.1, U2.13 (-), U2.14
- new net: R11.1, RV2.1
- new net: R11.2, R13.1, U2.8
- new net: H3.2 (Pin_2), RV2.2, RV2.3, U2.9 (-)
- new net: R30.2, R31.2, U2.2 (-)
- new net: FREQ_CTRL_1.2, R6.2
- new net: H2.2 (Pin_2), R5.1, R6.1
- new net: R12.2, U1.7
- new net: R15.2, RV3.1
- new net: H3.3 (Pin_3), RV1.2, RV1.3, TP1.1, U1.2 (-)
- new net: U2.6 (-), U2.7
- new net: R16.1, R17.2, U3.1 (INPUT_A)
- new net: R13.2, R14.1, TP3.1, U3.12 (FREQ_CTRL)
- new net: FREQ_CV_IN_1.T, FREQ_CV_IN_LVL_1.1
- new net: FREQ_CV_IN_LVL_1.2, R5.2
- new net: R9.1, RV1.1
- new net: C14.2, R32.1
- new net: R10.1, U1.6 (-)
Other:
- note added: "-100mV to +350mV"
- note added: "3320 Filter (Low-Pass)"
- note added: "Max Res Amount"
- moved on the sheet: AUDIO_IN_1, AUDIO_IN_2, C1, C10, C11, C12, C13, C2, C3, C4, C5, C6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

Commit message: 7555 readme
Parts:
- H5: value PinHeader_01x04 -> PinSocket_1x02
- H7: value PinSocket_01x04 -> PinHeader_1x02
- TP1, TP10, TP11, TP12, TP13, TP2, TP3, TP4, TP5, TP6, TP7, TP8, TP9: now left out of the parts list
- U3: value ~ -> CEM3320
Other:
- note added: "WRONG WAY AROUND!!"
Changed lines of the file:
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@@
 		)
 	)
+	(text "WRONG WAY AROUND!!"
+		(exclude_from_sim no)
+		(at 33.528 253.238 0)
+		(effects
+			(font
+				(size 1.27 1.27)
+			)
+		)
+	)
 	(text "Lennart Querter"
 		(exclude_from_sim no)
@@
 		(at 232.41 80.01 0)
 		(unit 1)
-		(exclude_from_sim no)
-		(in_bom yes)
+		(exclude_from_sim yes)
+		(in_bom no)
 		(on_board yes)
 		(dnp no)
@@
 		(at 339.09 93.98 0)
 		(unit 1)
-		(exclude_from_sim no)
-		(in_bom yes)
+		(exclude_from_sim yes)
+		(in_bom no)
 		(on_board yes)
 		(dnp no)
@@
 			)
 		)
-		(property "Value" "PinHeader_01x04"
+		(property "Value" "PinSocket_1x02"
 			(at 354.33 95.2499 0)
 			(effects
@@
 		(at 283.21 116.84 180)
 		(unit 1)
-		(exclude_from_sim no)
-		(in_bom yes)
+		(exclude_from_sim yes)
+		(in_bom no)
 		(on_board yes)
 		(dnp no)
@@
 		(at 217.17 80.01 0)
 		(unit 1)
-		(exclude_from_sim no)
-		(in_bom yes)
+		(exclude_from_sim yes)
+		(in_bom no)
 		(on_board yes)
 		(dnp no)
@@
 		(at 397.51 231.14 90)
 		(unit 1)
-		(exclude_from_sim no)
-		(in_bom yes)
+		(exclude_from_sim yes)
+		(in_bom no)
 		(on_board yes)
 		(dnp no)
@@
 		(at 198.12 175.26 270)
 		(unit 1)
-		(exclude_from_sim no)
-		(in_bom yes)
+		(exclude_from_sim yes)
+		(in_bom no)
 		(on_board yes)
 		(dnp no)
@@
 		(at 247.65 80.01 0)
 		(unit 1)
-		(exclude_from_sim no)
-		(in_bom yes)
+		(exclude_from_sim yes)
+		(in_bom no)
 		(on_board yes)
 		(dnp no)
@@
 		(at 266.7 80.01 0)
 		(unit 1)
-		(exclude_from_sim no)
-		(in_bom yes)
+		(exclude_from_sim yes)
+		(in_bom no)
 		(on_board yes)
 		(dnp no)
@@
 			)
 		)
-		(property "Value" "~"
+		(property "Value" "CEM3320"
 			(at 274.32 113.6965 0)
 			(effects
@@
 			)
 		)
-		(property "Value" "PinSocket_01x04"
+		(property "Value" "PinHeader_1x02"
 			(at 353.06 92.7101 0)
 			(effects
@@
 		(at 397.51 246.38 90)
 		(unit 1)
-		(exclude_from_sim no)
-		(in_bom yes)
+		(exclude_from_sim yes)
+		(in_bom no)
 		(on_board yes)
 		(dnp no)
@@
 		(at 92.71 180.34 180)
 		(unit 1)
-		(exclude_from_sim no)
-		(in_bom yes)
+		(exclude_from_sim yes)
+		(in_bom no)
 		(on_board yes)
 		(dnp no)
@@
 			)
 		)
-		(property "Value" "PinSocket_01x04"
+		(property "Value" "PinHeader_1x02"
 			(at 367.03 241.3001 0)
 			(effects
@@
 		(at 397.51 238.76 90)
 		(unit 1)
-		(exclude_from_sim no)
-		(in_bom yes)
+		(exclude_from_sim yes)
+		(in_bom no)
 		(on_board yes)
 		(dnp no)
@@
 		(at 185.42 116.84 0)
 		(unit 1)
-		(exclude_from_sim no)
-		(in_bom yes)
+		(exclude_from_sim yes)
+		(in_bom no)
 		(on_board yes)
 		(dnp no)
@@
 		(at 162.56 91.44 0)
 		(unit 1)
-		(exclude_from_sim no)
-		(in_bom yes)
+		(exclude_from_sim yes)
+		(in_bom no)
 		(on_board yes)
 		(dnp no)
@@
 			)
 		)
-		(property "Value" "PinHeader_01x04"
+		(property "Value" "PinSocket_1x02"
 			(at 368.3 243.8399 0)
 			(effects
