File: helpers/stm32_templates/stm32_template.kicad_sch (KiCad schematic)
At the start: 23 parts, among them J1 BOOT_RUN, J2 Conn_01x04, J3 Conn_01x16, J4 Conn_01x16, J5 Conn_01x16, U1 STM32F411RETx, Y1 20MHZ

Commit message: debugging and rework for ricochet, midas, wolkje. Added IBOM for drums and other modules.
Other:
- note added: "TODO: THIS SHOULD PULL UP TO 3.3V"
Changed lines of the file:
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@@
+		)
+	)
+	(text "TODO: THIS SHOULD PULL UP TO 3.3V"
+		(exclude_from_sim no)
+		(at 93.726 46.228 0)
+		(effects
+			(font
+				(size 1.27 1.27)
+			)
 		)
 	)
