File: modules/utility/1-midi-2-cv/kiCad/buffered_mcp4728.kicad_sch (KiCad schematic)
At the start: 21 parts, among them U3 MCP4728, U4 TL074

Commit message: finish up PCB finals for run-2, continue on C code for midas/sequencer
Parts:
- U4: footprint Package_SO:SOIC-14_3.9x8.7mm_P1.27mm -> Synth:SOIC-14
Changed lines of the file:
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@@
 	(wire
 		(pts
-			(xy 125.73 167.64) (xy 135.89 167.64)
+			(xy 132.08 167.64) (xy 135.89 167.64)
 		)
 		(stroke
@@
 	(wire
 		(pts
-			(xy 128.27 92.71) (xy 135.89 92.71)
+			(xy 132.08 92.71) (xy 135.89 92.71)
 		)
 		(stroke
@@
 	(wire
 		(pts
-			(xy 128.27 40.64) (xy 134.62 40.64)
+			(xy 132.08 40.64) (xy 134.62 40.64)
 		)
 		(stroke
@@
 	(wire
 		(pts
-			(xy 128.27 132.08) (xy 135.89 132.08)
+			(xy 132.08 132.08) (xy 135.89 132.08)
 		)
 		(stroke
@@
 	(symbol
 		(lib_id "power:GNDREF")
-		(at 128.27 40.64 270)
+		(at 132.08 40.64 0)
 		(unit 1)
 		(exclude_from_sim no)
@@
 		(fields_autoplaced yes)
 		(property "Reference" "#PWR013"
-			(at 121.92 40.64 0)
+			(at 132.08 46.99 0)
 			(effects
 				(font
@@
 		)
 		(property "Value" "GNDREF"
-			(at 127 36.83 90)
+			(at 128.27 41.91 90)
 			(effects
 				(font
 					(size 1.27 1.27)
 				)
+				(hide yes)
 			)
 		)
 		(property "Footprint" ""
-			(at 128.27 40.64 0)
+			(at 132.08 40.64 0)
 			(effects
 				(font
@@
 		)
 		(property "Datasheet" ""
-			(at 128.27 40.64 0)
+			(at 132.08 40.64 0)
 			(effects
 				(font
@@
 		)
 		(property "Description" "Power symbol creates a global label with name \"GNDREF\" , reference supply ground"
-			(at 128.27 40.64 0)
+			(at 132.08 40.64 0)
 			(effects
 				(font
@@
 				)
 				(justify left)
+				(hide yes)
 			)
 		)
@@
 	(symbol
 		(lib_id "power:GNDREF")
-		(at 204.47 158.75 270)
+		(at 204.47 158.75 0)
 		(unit 1)
 		(exclude_from_sim no)
@@
 		(fields_autoplaced yes)
 		(property "Reference" "#PWR019"
-			(at 198.12 158.75 0)
+			(at 204.47 165.1 0)
 			(effects
 				(font
@@
 		)
 		(property "Value" "GNDREF"
-			(at 200.66 158.7499 90)
+			(at 204.4699 162.56 90)
 			(effects
 				(font
@@
 				)
 				(justify right)
+				(hide yes)
 			)
 		)
@@
 				)
 				(justify right)
+				(hide yes)
 			)
 		)
@@
 	(symbol
 		(lib_id "power:GNDREF")
-		(at 204.47 83.82 270)
+		(at 204.47 83.82 0)
 		(unit 1)
 		(exclude_from_sim no)
@@
 		(fields_autoplaced yes)
 		(property "Reference" "#PWR017"
-			(at 198.12 83.82 0)
+			(at 204.47 90.17 0)
 			(effects
 				(font
@@
 		)
 		(property "Value" "GNDREF"
-			(at 200.66 83.8199 90)
+			(at 204.4699 87.63 90)
 			(effects
 				(font
@@
 				)
 				(justify right)
+				(hide yes)
 			)
 		)
@@
 			)
 		)
-		(property "Footprint" "Package_SO:SOIC-14_3.9x8.7mm_P1.27mm"
+		(property "Footprint" "Synth:SOIC-14"
 			(at 152.4 78.74 0)
 			(effects
@@
 			)
 		)
-		(property "Footprint" "Package_SO:SOIC-14_3.9x8.7mm_P1.27mm"
+		(property "Footprint" "Synth:SOIC-14"
 			(at 152.4 153.67 0)
 			(effects
@@
 	(symbol
 		(lib_id "power:GNDREF")
-		(at 205.74 31.75 270)
+		(at 205.74 31.75 0)
 		(unit 1)
 		(exclude_from_sim no)
@@
 		(fields_autoplaced yes)
 		(property "Reference" "#PWR020"
-			(at 199.39 31.75 0)
+			(at 205.74 38.1 0)
 			(effects
 				(font
@@
 		)
 		(property "Value" "GNDREF"
-			(at 201.93 31.7499 90)
+			(at 205.7399 35.56 90)
 			(effects
 				(font
@@
 				)
 				(justify right)
+				(hide yes)
 			)
 		)
@@
 	(symbol
 		(lib_id "power:GNDREF")
-		(at 204.47 123.19 270)
+		(at 204.47 123.19 0)
 		(unit 1)
 		(exclude_from_sim no)
@@
 		(fields_autoplaced yes)
 		(property "Reference" "#PWR018"
-			(at 198.12 123.19 0)
+			(at 204.47 129.54 0)
 			(effects
 				(font
@@
 		)
 		(property "Value" "GNDREF"
-			(at 200.66 123.1899 90)
+			(at 204.4699 127 90)
 			(effects
 				(font
@@
 				)
 				(justify right)
+				(hide yes)
 			)
 		)
@@
 			)
 		)
-		(property "Footprint" "Package_SO:SOIC-14_3.9x8.7mm_P1.27mm"
+		(property "Footprint" "Synth:SOIC-14"
 			(at 152.4 26.67 0)
 			(effects
@@
 	(symbol
 		(lib_id "power:GNDREF")
-		(at 128.27 132.08 270)
+		(at 132.08 132.08 0)
 		(unit 1)
 		(exclude_from_sim no)
@@
 		(fields_autoplaced yes)
 		(property "Reference" "#PWR015"
-			(at 121.92 132.08 0)
+			(at 132.08 138.43 0)
 			(effects
 				(font
@@
 		)
 		(property "Value" "GNDREF"
-			(at 127 128.27 90)
+			(at 128.27 133.35 90)
 			(effects
 				(font
 					(size 1.27 1.27)
 				)
+				(hide yes)
 			)
 		)
 		(property "Footprint" ""
-			(at 128.27 132.08 0)
+			(at 132.08 132.08 0)
 			(effects
 				(font
@@
 		)
 		(property "Datasheet" ""
-			(at 128.27 132.08 0)
+			(at 132.08 132.08 0)
 			(effects
 				(font
@@
 		)
 		(property "Description" "Power symbol creates a global label with name \"GNDREF\" , reference supply ground"
-			(at 128.27 132.08 0)
+			(at 132.08 132.08 0)
 			(effects
 				(font
@@
 	(symbol
 		(lib_id "power:GNDREF")
-		(at 128.27 92.71 270)
+		(at 132.08 92.71 0)
 		(unit 1)
 		(exclude_from_sim no)
@@
 		(fields_autoplaced yes)
 		(property "Reference" "#PWR014"
-			(at 121.92 92.71 0)
+			(at 132.08 99.06 0)
 			(effects
 				(font
@@
 		)
 		(property "Value" "GNDREF"
-			(at 127 88.9 90)
+			(at 128.27 93.98 90)
 			(effects
 				(font
 					(size 1.27 1.27)
 				)
+				(hide yes)
 			)
 		)
 		(property "Footprint" ""
-			(at 128.27 92.71 0)
+			(at 132.08 92.71 0)
 			(effects
 				(font
@@
 		)
 		(property "Datasheet" ""
-			(at 128.27 92.71 0)
+			(at 132.08 92.71 0)
 			(effects
 				(font
@@
 		)
 		(property "Description" "Power symbol creates a global label with name \"GNDREF\" , reference supply ground"
-			(at 128.27 92.71 0)
+			(at 132.08 92.71 0)
 			(effects
 				(font
@@
 	(symbol
 		(lib_id "power:GNDREF")
-		(at 125.73 167.64 270)
+		(at 132.08 167.64 0)
 		(unit 1)
 		(exclude_from_sim no)
@@
 		(fields_autoplaced yes)
 		(property "Reference" "#PWR016"
-			(at 119.38 167.64 0)
+			(at 132.08 173.99 0)
 			(effects
 				(font
@@
 		)
 		(property "Value" "GNDREF"
-			(at 124.46 163.83 90)
+			(at 128.27 168.91 90)
 			(effects
 				(font
 					(size 1.27 1.27)
 				)
+				(hide yes)
 			)
 		)
 		(property "Footprint" ""
-			(at 125.73 167.64 0)
+			(at 132.08 167.64 0)
 			(effects
 				(font
@@
 		)
 		(property "Datasheet" ""
-			(at 125.73 167.64 0)
+			(at 132.08 167.64 0)
 			(effects
 				(font
@@
 		)
 		(property "Description" "Power symbol creates a global label with name \"GNDREF\" , reference supply ground"
-			(at 125.73 167.64 0)
+			(at 132.08 167.64 0)
 			(effects
 				(font
@@
 			)
 		)
-		(property "Footprint" "Package_SO:SOIC-14_3.9x8.7mm_P1.27mm"
+		(property "Footprint" "Synth:SOIC-14"
 			(at 152.4 118.11 0)
 			(effects

Commit message: debugging and rework for ricochet, midas, wolkje. Added IBOM for drums and other modules.
Parts:
- removed H3: PinSocket_01x04, Synth:PinSocket_1x04_P2.54mm_Vertical, symbol synth:PinSocket_01x04
- removed H4: PinHeader_01x04, Synth:PinHeader_1x04_P2.54mm_Vertical, symbol synth:PinHeader_01x04
- renumbered R5 to R10, R9 to R11, R13 to R12, R6 to R13, R10 to R14, R14 to R3, R3 to R4, R7 to R5, R11 to R6, R4 to R7, R12 to R9, U4 to U2
Connections:
- net GNDREF: now also U3.4 (~{LDAC})
- net at R6.1: now also R8.2, U2.14
- net at R11.2, U2.1: now also R9.1
- net at R14.2, U2.7: now also R12.1
- net at R5.2, U2.8: now also R3.1
- net +5V renamed +3.3V
- no-connect marks 6 -> 5
