File: modules/utility/1-midi-2-cv/kiCad/midi-2-cv.kicad_pcb (KiCad board)
At the start: 2 copper layers, 181 x 111 mm, 40 parts, among them J1 PWR, J2 INPUT, J3 OUTPUT, U1 TL074

Commit message: midi2cv project reset
Parts:
- removed the C5 at (160.0, 103.0)
- removed the C5 at (60.0, 103.0)
- removed the C6 at (74.0, 98.0)
- removed the C6 at (174.0, 98.0)
- removed H1 (x2): TOP_4_SGL, Synth:PinHeader_1x04_P2.54mm_Vertical
- removed H2 (x2): BTM_4_SGL, Synth:PinSocket_1x04_P2.54mm_Vertical
- removed H3 (x2): TOP_8_SGL, Synth:PinHeader_1x08_P2.54mm_Vertical
- removed H4 (x2): BTM_8_SGL, Synth:PinSocket_1x08_P2.54mm_Vertical
- removed H5 (x2): TOP_8_PWR, Synth:PinHeader_1x08_P2.54mm_Vertical
- removed H6 (x2): BTM_8_PWR, Synth:PinSocket_1x08_P2.54mm_Vertical
- removed H7: Conn_02x05_PWR_Eurorack, Synth:IDC-Header_2x05_P2.54mm_Vertical
- removed the J2 at (200.0, 149.0)
- removed the J2 at (100.0, 149.0)
- removed J3 (x2): OUTPUT, Synth:Jack_3.5mm_QingPu_WQP-PJ398SM_Vertical_CircularHoles
- removed the U1 at (63.2, 95.4)
- removed the U1 at (163.2, 95.4)
- added ADC_1: ADC_4, Connector_Pin:Pin_D1.3mm_L11.0mm, F.Cu at (-42.5, 62.7)
- added ADC_2: ADC_1, Connector_Pin:Pin_D1.3mm_L11.0mm, F.Cu at (-42.5, 67.3)
- added ADC_3: ADC_2, Connector_Pin:Pin_D1.3mm_L11.0mm, F.Cu at (-42.5, 72.0)
- added ADC_4: ADC_3, Connector_Pin:Pin_D1.3mm_L11.0mm, F.Cu at (-42.5, 76.7)
- added C11: 0.1uF, Capacitor_THT:C_Disc_D5.0mm_W2.5mm_P5.00mm, F.Cu at (-28.3, 128.7)
- added C12: 0.1uF, Capacitor_THT:C_Disc_D5.0mm_W2.5mm_P5.00mm, F.Cu at (-28.3, 132.7)
- added C13: 0.1uF, Capacitor_THT:C_Disc_D5.0mm_W2.5mm_P5.00mm, F.Cu at (-28.3, 136.8)
- added C14: 0.1uF, Capacitor_THT:C_Disc_D5.0mm_W2.5mm_P5.00mm, F.Cu at (-28.3, 140.8)
- added C5: 0.1uF, Capacitor_THT:C_Disc_D5.0mm_W2.5mm_P5.00mm, F.Cu at (-28.3, 104.3)
- added C6: 0.1uF, Capacitor_THT:C_Disc_D5.0mm_W2.5mm_P5.00mm, F.Cu at (-28.3, 108.4)
- added CLK_OUT_1: OUTPUT, Synth:Jack_3.5mm_QingPu_WQP-PJ398SM_Vertical_CircularHoles, F.Cu at (111.5, 153.7)
- added CV_OUT_1: CV_OUT_1, Synth:Jack_3.5mm_QingPu_WQP-PJ398SM_Vertical_CircularHoles, F.Cu at (112.3, 59.0)
- added CV_OUT_2: CV_OUT_2, Synth:Jack_3.5mm_QingPu_WQP-PJ398SM_Vertical_CircularHoles, F.Cu at (113.0, 88.6)
- added CV_OUT_3: CV_OUT_3, Synth:Jack_3.5mm_QingPu_WQP-PJ398SM_Vertical_CircularHoles, F.Cu at (113.0, 103.5)
- added CV_OUT_4: CV_OUT_4, Synth:Jack_3.5mm_QingPu_WQP-PJ398SM_Vertical_CircularHoles, F.Cu at (113.4, 134.0)
- added D5: RED_OUT_20mA, Synth:LED_D5.0mm (center Aligned), F.Cu at (-18.6, 96.5)
- added D6: RED_OUT_20mA, Synth:LED_D5.0mm (center Aligned), F.Cu at (-11.1, 96.5)
- added D7: RED_OUT_20mA, Synth:LED_D5.0mm (center Aligned), F.Cu at (-3.63, 96.5)
- added GATE_1: GATE_2, Synth:Jack_3.5mm_QingPu_WQP-PJ398SM_Vertical_CircularHoles, F.Cu at (102.4, 88.5)
- added GATE_2: GATE_1, Synth:Jack_3.5mm_QingPu_WQP-PJ398SM_Vertical_CircularHoles, F.Cu at (102.3, 59.0)
- added GATE_3: GATE_3, Synth:Jack_3.5mm_QingPu_WQP-PJ398SM_Vertical_CircularHoles, F.Cu at (102.5, 103.5)
- added GATE_4: GATE_4, Synth:Jack_3.5mm_QingPu_WQP-PJ398SM_Vertical_CircularHoles, F.Cu at (102.3, 133.8)
- added J2: PWR, Synth:IDC-Header_2x08_P2.54mm_Vertical, F.Cu at (61.7, 57.7)
- added MOD_1: MOD_1, Synth:Jack_3.5mm_QingPu_WQP-PJ398SM_Vertical_CircularHoles, F.Cu at (122.8, 73.7)
- added MOD_2: MOD_2, Synth:Jack_3.5mm_QingPu_WQP-PJ398SM_Vertical_CircularHoles, F.Cu at (102.3, 73.7)
- added MOD_3: MOD_3, Synth:Jack_3.5mm_QingPu_WQP-PJ398SM_Vertical_CircularHoles, F.Cu at (123.9, 119.2)
- added MOD_4: MOD_4, Synth:Jack_3.5mm_QingPu_WQP-PJ398SM_Vertical_CircularHoles, F.Cu at (102.6, 118.4)
- added PWM_GEN_1: PWM_GEN_1, Connector_Pin:Pin_D1.3mm_L11.0mm, F.Cu at (-42.5, 81.3)
- added Q1: BC548, Package_TO_SOT_THT:TO-92_Inline, F.Cu at (12.0, 63.6)
- added Q2: BC548, Package_TO_SOT_THT:TO-92_Inline, F.Cu at (12.0, 69.4)
- added Q3: BC548, Package_TO_SOT_THT:TO-92_Inline, F.Cu at (12.0, 75.2)
- added Q4: BC548, Package_TO_SOT_THT:TO-92_Inline, F.Cu at (12.0, 81.0)
- added R10: 1K, Synth:R_Default (DIN0207), F.Cu at (-56.5, 98.8)
- added R11: 1K, Synth:R_Default (DIN0207), F.Cu at (-56.5, 102.9)
- added R12: 1K, Synth:R_Default (DIN0207), F.Cu at (-56.5, 107.0)
- added R13: 1K, Synth:R_Default (DIN0207), F.Cu at (-56.5, 111.0)
- added R14: 1K, Synth:R_Default (DIN0207), F.Cu at (-56.5, 115.0)
- added R15: 1K, Synth:R_Default (DIN0207), F.Cu at (-56.5, 119.1)
- added R16: 1K, Synth:R_Default (DIN0207), F.Cu at (-56.5, 123.2)
- added R17: 1K, Synth:R_Default (DIN0207), F.Cu at (-56.5, 127.2)
- added R18: 10K [1%], Synth:R_Default (DIN0207), F.Cu at (20.2, 62.4)
- added R19: 10K [1%], Synth:R_Default (DIN0207), F.Cu at (20.2, 66.5)
- added R20: 10K [1%], Synth:R_Default (DIN0207), F.Cu at (20.2, 70.5)
- added R21: 10K [1%], Synth:R_Default (DIN0207), F.Cu at (20.2, 74.5)
- added R22: 47K [1%], Synth:R_Default (DIN0207), F.Cu at (20.2, 78.6)
- added R23: 47K [1%], Synth:R_Default (DIN0207), F.Cu at (20.2, 82.7)
- added R24: 47K [1%], Synth:R_Default (DIN0207), F.Cu at (20.2, 86.7)
- added R25: 47K [1%], Synth:R_Default (DIN0207), F.Cu at (20.2, 90.8)
- added R26: 10K [1%], Synth:R_Default (DIN0207), F.Cu at (0.79, 104.3)
- added R27: 10K [1%], Synth:R_Default (DIN0207), F.Cu at (0.79, 108.4)
- added R28: 10K [1%], Synth:R_Default (DIN0207), F.Cu at (0.79, 112.5)
- added R29: 10K [1%], Synth:R_Default (DIN0207), F.Cu at (0.79, 116.5)
- added R30: 47K [1%], Synth:R_Default (DIN0207), F.Cu at (0.79, 120.5)
- added R31: 47K [1%], Synth:R_Default (DIN0207), F.Cu at (0.79, 124.6)
- added R32: 47K [1%], Synth:R_Default (DIN0207), F.Cu at (0.79, 128.7)
- added R33: 47K [1%], Synth:R_Default (DIN0207), F.Cu at (0.79, 132.7)
- added R34: 10K [1%], Synth:R_Default (DIN0207), F.Cu at (24.6, 104.3)
- added R35: 10K [1%], Synth:R_Default (DIN0207), F.Cu at (24.6, 108.4)
- added R36: 10K [1%], Synth:R_Default (DIN0207), F.Cu at (24.6, 112.5)
- added R37: 10K [1%], Synth:R_Default (DIN0207), F.Cu at (24.6, 116.5)
- added R38: 47K [1%], Synth:R_Default (DIN0207), F.Cu at (24.6, 120.5)
- added R39: 47K [1%], Synth:R_Default (DIN0207), F.Cu at (24.6, 124.6)
- added R40: 47K [1%], Synth:R_Default (DIN0207), F.Cu at (24.6, 128.7)
- added R41: 47K [1%], Synth:R_Default (DIN0207), F.Cu at (24.6, 132.7)
- added R42: 10, Synth:R_Default (DIN0207), F.Cu at (-20.1, 128.6)
- added R43: 10, Synth:R_Default (DIN0207), F.Cu at (-20.1, 132.6)
- added R44: 68K, Synth:R_Default (DIN0207), F.Cu at (-28.3, 62.4)
- added R45: 68K, Synth:R_Default (DIN0207), F.Cu at (-28.3, 66.5)
- added R46: 100K, Synth:R_Default (DIN0207), F.Cu at (-28.3, 70.5)
- added R47: 100K, Synth:R_Default (DIN0207), F.Cu at (-28.3, 74.5)
- added R48: 470R, Synth:R_Default (DIN0207), F.Cu at (-28.3, 78.6)
- added R49: 470R, Synth:R_Default (DIN0207), F.Cu at (-28.3, 82.7)
- added R5: 1K, Synth:R_Default (DIN0207), F.Cu at (-56.5, 78.6)
- added R50: 22K, Synth:R_Default (DIN0207), F.Cu at (-28.3, 86.7)
- added R51: 22K, Synth:R_Default (DIN0207), F.Cu at (-28.3, 90.8)
- added R52: 1K, Synth:R_Default (DIN0207), F.Cu at (-15.0, 62.4)
- added R53: 1K, Synth:R_Default (DIN0207), F.Cu at (-15.0, 66.5)
- added R54: 100K, Synth:R_Default (DIN0207), F.Cu at (-15.0, 70.5)
- added R55: 100K, Synth:R_Default (DIN0207), F.Cu at (-15.0, 74.5)
- added R56: 68K, Synth:R_Default (DIN0207), F.Cu at (-15.0, 78.6)
- added R57: 68K, Synth:R_Default (DIN0207), F.Cu at (-15.0, 82.7)
- added R58: 100K, Synth:R_Default (DIN0207), F.Cu at (-15.0, 86.7)
- added R59: 100K, Synth:R_Default (DIN0207), F.Cu at (-15.0, 90.8)
- added R6: 1K, Synth:R_Default (DIN0207), F.Cu at (-56.5, 82.7)
- added R60: 470R, Synth:R_Default (DIN0207), F.Cu at (-1.65, 62.4)
- added R61: 470R, Synth:R_Default (DIN0207), F.Cu at (-1.65, 66.5)
- added R62: 22K, Synth:R_Default (DIN0207), F.Cu at (-1.65, 70.5)
- added R63: 22K, Synth:R_Default (DIN0207), F.Cu at (-1.65, 74.5)
- added R64: 1K, Synth:R_Default (DIN0207), F.Cu at (-1.65, 78.6)
- added R65: 1K, Synth:R_Default (DIN0207), F.Cu at (-1.65, 82.7)
- added R66: 100K, Synth:R_Default (DIN0207), F.Cu at (-1.65, 86.7)
- added R67: 100K, Synth:R_Default (DIN0207), F.Cu at (-1.65, 90.8)
- added R7: 22K, Synth:R_Default (DIN0207), F.Cu at (-56.5, 86.7)
- added R8: 68K, Synth:R_Default (DIN0207), F.Cu at (-56.5, 90.8)
- added R9: 1K, Synth:R_Default (DIN0207), F.Cu at (-56.5, 94.8)
- added U1: 6N135, Package_DIP:DIP-8_W7.62mm, F.Cu at (148.0, 85.9)
- added U10: TL074, Package_SO:SOIC-14_3.9x8.7mm_P1.27mm, F.Cu at (-9.52, 107.6)
- added U2: STM32F401CCUx, stm32:YAAJ_BlackPill_1, B.Cu at (62.6, 151.5)
- added U3: TL074, Package_SO:SOIC-14_3.9x8.7mm_P1.27mm, F.Cu at (-40.6, 114.9)
- added U4: MCP4728, Package_SO:MSOP-10_3x3mm_P0.5mm, F.Cu at (35.6, 73.1)
- added U5: TL074, Package_SO:SOIC-14_3.9x8.7mm_P1.27mm, F.Cu at (55.4, 94.9)
- added U6: MCP4728, Package_SO:MSOP-10_3x3mm_P0.5mm, F.Cu at (16.2, 115.0)
- added U7: TL074, Package_SO:SOIC-14_3.9x8.7mm_P1.27mm, F.Cu at (16.7, 107.6)
- added U8: MCP4728, Package_SO:MSOP-10_3x3mm_P0.5mm, F.Cu at (40.0, 115.0)
- added U9: TL074, Package_SO:SOIC-14_3.9x8.7mm_P1.27mm, F.Cu at (40.5, 107.6)
- added VEL_1: VEL_1, Synth:Jack_3.5mm_QingPu_WQP-PJ398SM_Vertical_CircularHoles, F.Cu at (122.6, 58.9)
- added VEL_2: VEL_2, Synth:Jack_3.5mm_QingPu_WQP-PJ398SM_Vertical_CircularHoles, F.Cu at (123.3, 88.4)
- added VEL_3: VEL_3, Synth:Jack_3.5mm_QingPu_WQP-PJ398SM_Vertical_CircularHoles, F.Cu at (123.4, 103.7)
- added VEL_4: VEL_4, Synth:Jack_3.5mm_QingPu_WQP-PJ398SM_Vertical_CircularHoles, F.Cu at (123.8, 133.7)
- C1, C2, C3, C4: moved to F.Cu
- C10, C9: footprint Capacitor_THT:CP_Radial_D4.0mm_P2.00mm -> Capacitor_THT:C_Disc_D5.0mm_W2.5mm_P5.00mm; moved to F.Cu
- C7, C8: value 47uF -> 0.1uF; footprint Capacitor_THT:CP_Radial_D6.3mm_P2.50mm -> Capacitor_THT:C_Disc_D5.0mm_W2.5mm_P5.00mm; moved to F.Cu
- D1: value 1N5819 -> 1N4148; footprint Synth:D_DO-41_SOD81_P10.16mm_Horizontal -> Synth:D_DO-35_SOD27_P7.62mm_Horizontal
- D4: value 1N5819 -> RED_OUT_20mA; footprint Synth:D_DO-41_SOD81_P10.16mm_Horizontal -> Synth:LED_D5.0mm (center Aligned)
- J1: value PWR -> DIN-5_180degree; footprint Synth:IDC-Header_2x08_P2.54mm_Vertical -> Connector_Audio:Jack_XLR-6.35mm_Neutrik_NCJ5FI-V_Vertical; moved to F.Cu
- R1: value 10 -> 220R
- R2: value 10 -> 10K
- R3, R4: value 10 -> 1K
- moved R3 218.6 mm to (-56.5, 70.5)
- moved R4 218.0 mm to (-56.5, 74.5)
- moved C9 207.3 mm to (-28.3, 120.5), turned to 0 degrees
- moved C10 206.5 mm to (-28.3, 124.6), turned to 0 degrees
- moved D3 204.9 mm to (-19.8, 124.4), turned to 0 degrees
- moved C7 199.4 mm to (-28.3, 112.5), turned to 0 degrees
- moved C8 198.6 mm to (-28.3, 116.5), turned to 0 degrees
- moved D4 189.0 mm to (-26.1, 96.5)
- moved D1 127.9 mm to (-43.2, 107.8), turned to 0 degrees
- moved R2 118.4 mm to (-56.5, 66.5)
- moved R1 118.2 mm to (-56.5, 62.4)
- moved C3 103.6 mm to (-6.59, 129.3), turned to 0 degrees
- moved C4 102.6 mm to (-6.59, 134.8), turned to 0 degrees
- moved J1 100.2 mm to (153.7, 64.0)
- moved C2 95.6 mm to (-18.9, 114.1), turned to 0 degrees
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Connections:
- J1 pad 1: Net-(D2-K) -> unconnected-(J1-Pad1)
- J1 pad 2: Net-(D2-K) -> GNDREF
- J1 pad 3: GNDREF -> unconnected-(J1-Pad3)
- R1 pad 1: +12V -> Net-(J1-Pad4)
- R2 pad 1: -12V -> +3.3V
- R2 pad 2: Net-(D2-A) -> Net-(U2-PA10)
- R3 pad 1: +12V -> Net-(CV_OUT_1-PadT)
- R3 pad 2: Net-(D3-K) -> /buffered_mcp4728/OUT_1
- R4 pad 1: -12V -> Net-(CV_OUT_2-PadT)
- R4 pad 2: Net-(D4-A) -> /buffered_mcp4728/OUT_2
Routing:
- net -12V: track 60.2 -> 0.00 mm
- net +12V: track 52.7 -> 0.00 mm
- net Net-(D1-A): track 16.3 -> 0.00 mm
- net Net-(D4-K): track 14.3 -> 0.00 mm
- net Net-(D3-A): track 9.45 -> 0.00 mm
- net Net-(D2-K): track 8.46 -> 0.00 mm
- net Net-(D3-K): track 3.37 -> 0.00 mm
- net Net-(D1-K): track 3.37 -> 0.00 mm
- net Net-(D4-A): track 3.35 -> 0.00 mm
- net Net-(D2-A): track 3.26 -> 0.00 mm
Other:
- board size 181 x 111 mm -> 81 x 111 mm

Commit message: add panels, redo gerbers for distorted daisy
Parts:
- removed ADC_1: ADC_4, Connector_Pin:Pin_D1.3mm_L11.0mm
- removed ADC_2: ADC_1, Connector_Pin:Pin_D1.3mm_L11.0mm
- removed ADC_3: ADC_2, Connector_Pin:Pin_D1.3mm_L11.0mm
- removed ADC_4: ADC_3, Connector_Pin:Pin_D1.3mm_L11.0mm
- removed C7, C8: 0.1uF, Capacitor_THT:C_Disc_D5.0mm_W2.5mm_P5.00mm
- removed CLK_OUT_1: OUTPUT, Synth:Jack_3.5mm_QingPu_WQP-PJ398SM_Vertical_CircularHoles
- removed J1: DIN-5_180degree, Connector_Audio:Jack_XLR-6.35mm_Neutrik_NCJ5FI-V_Vertical
- removed PWM_GEN_1: PWM_GEN_1, Connector_Pin:Pin_D1.3mm_L11.0mm
- removed R65: 1K, Synth:R_Default (DIN0207)
- removed R66, R67: 100K, Synth:R_Default (DIN0207)
- removed U10: TL074, Package_SO:SOIC-14_3.9x8.7mm_P1.27mm
- added C15: 0.1uF, Capacitor_THT:C_Disc_D5.0mm_W2.5mm_P5.00mm, F.Cu at (-68.5, 155.1)
- added C16: 0.1uF, Capacitor_THT:C_Disc_D5.0mm_W2.5mm_P5.00mm, F.Cu at (-68.5, 159.2)
- added H1: Conn_02x05_PWR_Eurorack, Synth:IDC-Header_2x05_P2.54mm_Vertical, F.Cu at (54.9, 58.5)
- added U11: MCP4728, Package_SO:MSOP-10_3x3mm_P0.5mm, F.Cu at (-100.6, 31.2)
- C1: value 47uF -> 0.1uF; footprint Capacitor_THT:CP_Radial_D6.3mm_P2.50mm -> Capacitor_THT:CP_Radial_D4.0mm_P2.00mm
- C3: value 0.1uF -> 47uF; footprint Capacitor_THT:CP_Radial_D4.0mm_P2.00mm -> Capacitor_THT:CP_Radial_D6.3mm_P2.50mm
- C5, C6: footprint Capacitor_THT:C_Disc_D5.0mm_W2.5mm_P5.00mm -> Capacitor_THT:CP_Radial_D4.0mm_P2.00mm
- CV_OUT_1: value CV_OUT_1 -> CV_OUT_2
- CV_OUT_2: value CV_OUT_2 -> CV_OUT_3
- CV_OUT_3: value CV_OUT_3 -> CV_OUT_4
- CV_OUT_4: value CV_OUT_4 -> CV_OUT_1
- J2: value PWR -> DIN-6; footprint Synth:IDC-Header_2x08_P2.54mm_Vertical -> Synth:MIDI_DIN5-SD-60BV
- MOD_1: value MOD_1 -> MOD_2
- MOD_2: value MOD_2 -> MOD_3
- MOD_3: value MOD_3 -> MOD_4
- MOD_4: value MOD_4 -> MOD_1
- R10, R9: value 1K -> 47K [1%]
- R15, R16, R17, R3, R4, R5, R6: value 1K -> 10K [1%]
- R19, R20, R21, R34, R35, R36: value 10K [1%] -> 47K [1%]
- R23, R24, R25, R38, R39, R40: value 47K [1%] -> 1K
- R26, R37: value 10K [1%] -> 1K
- R27, R28: value 10K [1%] -> 10
- R30, R31, R32: value 47K [1%] -> 10K [1%]
- R41: value 47K [1%] -> 68K
- R42: value 10 -> 68K
- R43: value 10 -> 100K
- R44, R56: value 68K -> 100K
- R45, R57: value 68K -> 470R
- R46, R58: value 100K -> 470R
- R47, R59: value 100K -> 22K
- R48, R60: value 470R -> 22K
- R49, R61: value 470R -> 1K
- R50, R62: value 22K -> 1K
- R51, R63: value 22K -> 100K
- R52, R64: value 1K -> 100K
- R53: value 1K -> 68K
- R54: value 100K -> 68K
- R7: value 22K -> 47K [1%]
- R8: value 68K -> 47K [1%]
- U2: value STM32F401CCUx -> YAAJ_WeAct_BlackPill_Part_Like; footprint stm32:YAAJ_BlackPill_1 -> stm32:YAAJ_WeAct_BlackPill_SWD_2
- U3, U5: value TL074 -> MCP4728; footprint Package_SO:SOIC-14_3.9x8.7mm_P1.27mm -> Package_SO:MSOP-10_3x3mm_P0.5mm
- U4, U6, U8: value MCP4728 -> TL074; footprint Package_SO:MSOP-10_3x3mm_P0.5mm -> Package_SO:SOIC-14_3.9x8.7mm_P1.27mm
- U7: value TL074 -> L7805; footprint Package_SO:SOIC-14_3.9x8.7mm_P1.27mm -> Package_TO_SOT_THT:TO-220-3_Horizontal_TabDown
- VEL_1: value VEL_1 -> VEL_2
- VEL_2: value VEL_2 -> VEL_3
- VEL_3: value VEL_3 -> VEL_4
- VEL_4: value VEL_4 -> VEL_1
- moved D4 181.4 mm to (153.1, 124.7), turned to 90 degrees
- moved D5 172.6 mm to (153.1, 114.0), turned to 90 degrees
- moved D6 164.3 mm to (153.1, 103.0), turned to 90 degrees
- moved U8 159.9 mm to (-100.5, 38.5)
- moved R34 156.4 mm to (-116.0, 35.7)
- moved R35 156.4 mm to (-116.0, 39.8)
- moved R36 156.4 mm to (-116.0, 43.8)
- moved R37 156.4 mm to (-116.0, 47.9)
- moved R38 156.4 mm to (-116.0, 51.9)
- moved R39 156.4 mm to (-116.0, 56.0)
- moved R40 156.4 mm to (-116.0, 60.0)
- moved U5 156.0 mm to (-100.6, 92.2)
- moved D7 155.7 mm to (152.0, 92.0), turned to 90 degrees
- moved J2 155.2 mm to (186.5, 150.0), turned to 0 degrees
- moved R29 154.4 mm to (-116.0, 15.4)
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Connections:
- C2 pad 1: GNDREF -> +12V
- C2 pad 2: -12V -> GNDREF
- C3 pad 1: +12V -> GNDREF
- C3 pad 2: GNDREF -> -12V
- C4 pad 1: GNDREF -> +5V
- C4 pad 2: -12V -> GNDREF
- J2 pad 1: Net-(D3-K) -> unconnected-(J2-Pad1)
- J2 pad 2: Net-(D3-K) -> Net-(J2-Pad2)
- J2 pad 4: GNDREF -> Net-(D1-A)
- J2 pad 5: GNDREF -> unconnected-(J2-Pad5)
- J2 pad 6: GNDREF -> unconnected-(J2-Pad6)
- R1 pad 1: Net-(J1-Pad4) -> Net-(J2-Pad2)
- R10 pad 2: /buffered_mcp4729/OUT_1 -> Net-(U4D--)
- R11 pad 1: Net-(R11-Pad1) -> Net-(CV_OUT_1-PadT)
- R11 pad 2: /buffered_mcp4729/OUT_2 -> Net-(R11-Pad2)
- R12 pad 1: Net-(R12-Pad1) -> Net-(CV_OUT_2-PadT)
- R12 pad 2: /buffered_mcp4729/OUT_4 -> Net-(R12-Pad2)
- R13 pad 1: Net-(R13-Pad1) -> Net-(CV_OUT_3-PadT)
- R13 pad 2: /buffered_mcp4729/OUT_3 -> Net-(R10-Pad1)
- R14 pad 1: Net-(MOD_1-PadT) -> Net-(CV_OUT_4-PadT)
- R14 pad 2: /buffered_mcp4730/OUT_1 -> Net-(R14-Pad2)
- R15 pad 1: Net-(MOD_2-PadT) -> Net-(U6A--)
- R15 pad 2: /buffered_mcp4730/OUT_2 -> GNDREF
- R16 pad 1: Net-(MOD_3-PadT) -> Net-(U6B--)
- R16 pad 2: /buffered_mcp4730/OUT_4 -> GNDREF
- R17 pad 1: Net-(MOD_4-PadT) -> Net-(U6C--)
- R17 pad 2: /buffered_mcp4730/OUT_3 -> GNDREF
- R18 pad 1: Net-(U5A--) -> Net-(U6D--)
- R19 pad 1: Net-(U5B--) -> Net-(R19-Pad1)
- R19 pad 2: GNDREF -> Net-(U6A--)
- R20 pad 1: Net-(U5C--) -> Net-(R20-Pad1)
- R20 pad 2: GNDREF -> Net-(U6B--)
- R21 pad 1: Net-(U5D--) -> Net-(R21-Pad1)
- R21 pad 2: GNDREF -> Net-(U6C--)
- R22 pad 1: /buffered_mcp4728/OUT_1 -> Net-(R22-Pad1)
- R22 pad 2: Net-(U5A--) -> Net-(U6D--)
- R23 pad 1: /buffered_mcp4728/OUT_2 -> Net-(R23-Pad1)
- R23 pad 2: Net-(U5B--) -> Net-(R20-Pad1)
- R24 pad 1: /buffered_mcp4728/OUT_3 -> Net-(R24-Pad1)
- R24 pad 2: Net-(U5C--) -> Net-(R21-Pad1)
- R25 pad 1: /buffered_mcp4728/OUT_4 -> Net-(R25-Pad1)
- R25 pad 2: Net-(U5D--) -> Net-(R22-Pad1)
- R26 pad 1: Net-(U7A--) -> Net-(R26-Pad1)
- R26 pad 2: GNDREF -> Net-(R19-Pad1)
- R27 pad 1: Net-(U7B--) -> +12V
- R27 pad 2: GNDREF -> Net-(D2-K)
- R28 pad 1: Net-(U7C--) -> -12V
- R28 pad 2: GNDREF -> Net-(D3-A)
- R29 pad 1: Net-(U7D--) -> Net-(U8A--)
- R3 pad 1: Net-(CV_OUT_1-PadT) -> Net-(U4A--)
- R3 pad 2: /buffered_mcp4728/OUT_1 -> GNDREF
- R30 pad 1: /buffered_mcp4729/OUT_1 -> Net-(U8B--)
- R30 pad 2: Net-(U7A--) -> GNDREF
- R31 pad 1: /buffered_mcp4729/OUT_2 -> Net-(U8C--)
- R31 pad 2: Net-(U7B--) -> GNDREF
- R32 pad 1: /buffered_mcp4729/OUT_3 -> Net-(U8D--)
- R32 pad 2: Net-(U7C--) -> GNDREF
- R33 pad 1: /buffered_mcp4729/OUT_4 -> Net-(R33-Pad1)
- R33 pad 2: Net-(U7D--) -> Net-(U8A--)
- R34 pad 1: Net-(U9A--) -> Net-(R34-Pad1)
- R34 pad 2: GNDREF -> Net-(U8B--)
- R35 pad 1: Net-(U9B--) -> Net-(R35-Pad1)
- R35 pad 2: GNDREF -> Net-(U8C--)
- R36 pad 1: Net-(U9C--) -> Net-(R36-Pad1)
- R36 pad 2: GNDREF -> Net-(U8D--)
- R37 pad 1: Net-(U9D--) -> Net-(MOD_1-PadT)
- R37 pad 2: GNDREF -> Net-(R34-Pad1)
- R38 pad 1: /buffered_mcp4730/OUT_1 -> Net-(MOD_2-PadT)
- R38 pad 2: Net-(U9A--) -> Net-(R35-Pad1)
- R39 pad 1: /buffered_mcp4730/OUT_2 -> Net-(MOD_3-PadT)
- R39 pad 2: Net-(U9B--) -> Net-(R36-Pad1)
- R4 pad 1: Net-(CV_OUT_2-PadT) -> Net-(U4B--)
- R4 pad 2: /buffered_mcp4728/OUT_2 -> GNDREF
- R40 pad 1: /buffered_mcp4730/OUT_3 -> Net-(MOD_4-PadT)
- R40 pad 2: Net-(U9C--) -> Net-(R33-Pad1)
- R41 pad 1: /buffered_mcp4730/OUT_4 -> Net-(U9B--)
- R41 pad 2: Net-(U9D--) -> GNDREF
- R42 pad 1: +12V -> Net-(U9A--)
- R42 pad 2: Net-(D2-K) -> GNDREF
- R43 pad 1: -12V -> Net-(R43-Pad1)
- R43 pad 2: Net-(D3-A) -> Net-(U9B--)
- R44 pad 1: Net-(U10B--) -> Net-(R44-Pad1)
- R44 pad 2: GNDREF -> Net-(U9A--)
- R45 pad 1: Net-(U10A--) -> Net-(D4-K)
- R46 pad 1: Net-(R46-Pad1) -> Net-(D5-K)
- R46 pad 2: Net-(U10B--) -> GNDREF
- R47 pad 1: Net-(R47-Pad1) -> Net-(Q1-B)
- R47 pad 2: Net-(U10A--) -> Net-(R43-Pad1)
- R48 pad 1: Net-(D4-K) -> Net-(Q2-B)
- R48 pad 2: GNDREF -> Net-(R44-Pad1)
- R49 pad 1: Net-(D5-K) -> Net-(GATE_1-PadT)
- R49 pad 2: GNDREF -> Net-(R43-Pad1)
- R5 pad 1: Net-(CV_OUT_3-PadT) -> Net-(U4C--)
- R5 pad 2: /buffered_mcp4728/OUT_4 -> GNDREF
- R50 pad 1: Net-(Q1-B) -> Net-(GATE_2-PadT)
- R50 pad 2: Net-(R46-Pad1) -> Net-(R44-Pad1)
- R51 pad 1: Net-(Q2-B) -> +3.3V
- R51 pad 2: Net-(R47-Pad1) -> /gate_out/GATE_2_CALLBACK
- R52 pad 1: Net-(GATE_1-PadT) -> +3.3V
- R52 pad 2: Net-(R46-Pad1) -> /gate_out/GATE_1_CALLBACK
- R53 pad 1: Net-(GATE_2-PadT) -> Net-(U9D--)
- R53 pad 2: Net-(R47-Pad1) -> GNDREF
- R54 pad 1: +3.3V -> Net-(U9C--)
- R54 pad 2: /gate_out/GATE_2_CALLBACK -> GNDREF
- R55 pad 1: +3.3V -> Net-(R55-Pad1)
- R55 pad 2: /gate_out/GATE_1_CALLBACK -> Net-(U9C--)
- R56 pad 1: Net-(U10D--) -> Net-(R56-Pad1)
- R56 pad 2: GNDREF -> Net-(U9D--)
- R57 pad 1: Net-(U10C--) -> Net-(D6-K)
- R58 pad 1: Net-(R58-Pad1) -> Net-(D7-K)
- R58 pad 2: Net-(U10C--) -> GNDREF
- R59 pad 1: Net-(R59-Pad1) -> Net-(Q3-B)
- R59 pad 2: Net-(U10D--) -> Net-(R55-Pad1)
- R6 pad 1: Net-(CV_OUT_4-PadT) -> Net-(U4D--)
- R6 pad 2: /buffered_mcp4728/OUT_3 -> GNDREF
- R60 pad 1: Net-(D6-K) -> Net-(Q4-B)
- R60 pad 2: GNDREF -> Net-(R56-Pad1)
- R61 pad 1: Net-(D7-K) -> Net-(GATE_3-PadT)
- R61 pad 2: GNDREF -> Net-(R55-Pad1)
- R62 pad 1: Net-(Q3-B) -> Net-(GATE_4-PadT)
- R62 pad 2: Net-(R58-Pad1) -> Net-(R56-Pad1)
- R63 pad 1: Net-(Q4-B) -> +3.3V
- R63 pad 2: Net-(R59-Pad1) -> /gate_out/GATE_3_CALLBACK
- R64 pad 1: Net-(GATE_3-PadT) -> +3.3V
- R64 pad 2: Net-(R58-Pad1) -> /gate_out/GATE_4_CALLBACK
- R7 pad 1: GNDREF -> Net-(R14-Pad2)
- R7 pad 2: Net-(U3A--) -> Net-(U4A--)
- R8 pad 1: Net-(U3A--) -> Net-(R11-Pad2)
- R8 pad 2: +12V -> Net-(U4B--)
- R9 pad 1: Net-(CLK_OUT_1-PadT) -> Net-(R12-Pad2)
- R9 pad 2: Net-(R9-Pad2) -> Net-(U4C--)
- U2 pad 1: unconnected-(U2-VBAT-Pad1) -> /gate_out/GATE_IN_1
- U2 pad 10: /gate_out/GATE_1_CALLBACK -> unconnected-(U2-PA15-Pad10)
- U2 pad 11: /gate_out/GATE_2_CALLBACK -> /mcp4728_vel-out/SDA
- U2 pad 12: /gate_out/GATE_3_CALLBACK -> /mcp4728_mod-out/SDA
- U2 pad 13: /gate_out/GATE_4_CALLBACK -> unconnected-(U2-PB5-Pad13)
- U2 pad 14: Net-(U2-PA4) -> /mcp4728_cv-out/SCL
- U2 pad 15: Net-(U2-PA5) -> /mcp4728_cv-out/SDA
- U2 pad 16: Net-(U2-PA6) -> /mcp4728_mod-out/SCL
- U2 pad 17: Net-(U2-PA7) -> unconnected-(U2-PB9-Pad17)
- U2 pad 18: Net-(U2-PB0) -> +5V
- U2 pad 19: unconnected-(U2-PB1-Pad19) -> GNDREF
- U2 pad 2: unconnected-(U2-PC13-Pad2) -> /gate_out/GATE_IN_2
- U2 pad 20: unconnected-(U2-PB2-Pad20) -> +3.3V
- U2 pad 21: /buffered_mcp4729/SCL -> unconnected-(U2-VBat-Pad21)
- U2 pad 23: GNDREF -> unconnected-(U2-PC14-Pad23)
- U2 pad 24: +3.3V -> unconnected-(U2-PC15-Pad24)
- U2 pad 25: /gate_out/GATE_IN_1 -> unconnected-(U2-RES-Pad25)
- U2 pad 26: /gate_out/GATE_IN_2 -> /gate_out/GATE_1_CALLBACK
- U2 pad 27: /gate_out/GATE_IN_3 -> /gate_out/GATE_2_CALLBACK
- U2 pad 28: /gate_out/GATE_IN_4 -> /gate_out/GATE_3_CALLBACK
- U2 pad 29: /buffered_mcp4730/SCL -> /gate_out/GATE_4_CALLBACK
- U2 pad 3: unconnected-(U2-PC14-Pad3) -> /gate_out/GATE_IN_3
- U2 pad 30: Net-(U2-PA9) -> unconnected-(U2-PA4-Pad30)
- U2 pad 31: Net-(U2-PA10) -> unconnected-(U2-PA5-Pad31)
- U2 pad 4: unconnected-(U2-PC15-Pad4) -> /gate_out/GATE_IN_4
- U2 pad 7: unconnected-(U2-NRST-Pad7) -> Net-(U2-PA10)
- U2 pad 8: GNDREF -> unconnected-(U2-PA11-Pad8)
- U3 pad 1: Net-(R9-Pad2) -> +5V
- U3 pad 10: (no net) -> GNDREF
- U3 pad 2: Net-(U3A--) -> /mcp4728_cv-out/SCL
- U3 pad 3: Net-(U2-PA7) -> /mcp4728_cv-out/SDA
- U3 pad 4: +12V -> unconnected-(U3-~{LDAC}-Pad4)
- U3 pad 5: (no net) -> unconnected-(U3-RDY/~{BSY}-Pad5)
- U3 pad 6: (no net) -> Net-(U3-VOUTA)
- U3 pad 7: (no net) -> Net-(U3-VOUTB)
- U3 pad 8: (no net) -> Net-(U3-VOUTC)
- U3 pad 9: (no net) -> Net-(U3-VOUTD)
- U4 pad 1: +5V -> Net-(R14-Pad2)
- U4 pad 10: GNDREF -> Net-(U3-VOUTC)
- U4 pad 2: /buffered_mcp4728/SCL -> Net-(U4A--)
- U4 pad 3: /buffered_mcp4728/SDA -> Net-(U3-VOUTA)
- U4 pad 4: unconnected-(U4-~{LDAC}-Pad4) -> +12V
- U4 pad 5: unconnected-(U4-RDY/~{BSY}-Pad5) -> Net-(U3-VOUTB)
- U4 pad 6: Net-(U4-VOUTA) -> Net-(U4B--)
- U4 pad 7: Net-(U4-VOUTB) -> Net-(R11-Pad2)
- U4 pad 8: Net-(U4-VOUTC) -> Net-(R12-Pad2)
- U4 pad 9: Net-(U4-VOUTD) -> Net-(U4C--)
- U5 pad 1: /buffered_mcp4728/OUT_1 -> +5V
- U5 pad 10: Net-(U4-VOUTC) -> GNDREF
- U5 pad 2: Net-(U5A--) -> /mcp4728_vel-out/SCL
- U5 pad 3: Net-(U4-VOUTA) -> /mcp4728_vel-out/SDA
- U5 pad 4: +12V -> unconnected-(U5-~{LDAC}-Pad4)
- U5 pad 5: Net-(U4-VOUTB) -> unconnected-(U5-RDY/~{BSY}-Pad5)
- U5 pad 6: Net-(U5B--) -> Net-(U5-VOUTA)
- U5 pad 7: /buffered_mcp4728/OUT_2 -> Net-(U5-VOUTB)
- U5 pad 8: /buffered_mcp4728/OUT_3 -> Net-(U5-VOUTC)
- U5 pad 9: Net-(U5C--) -> Net-(U5-VOUTD)
- U6 pad 1: +5V -> Net-(R19-Pad1)
- U6 pad 10: GNDREF -> Net-(U5-VOUTC)
- U6 pad 2: /buffered_mcp4729/SCL -> Net-(U6A--)
- U6 pad 3: /buffered_mcp4729/SDA -> Net-(U5-VOUTA)
- U6 pad 4: unconnected-(U6-~{LDAC}-Pad4) -> +12V
- U6 pad 5: unconnected-(U6-RDY/~{BSY}-Pad5) -> Net-(U5-VOUTB)
- U6 pad 6: Net-(U6-VOUTA) -> Net-(U6B--)
- U6 pad 7: Net-(U6-VOUTB) -> Net-(R20-Pad1)
- U6 pad 8: Net-(U6-VOUTC) -> Net-(R21-Pad1)
- U6 pad 9: Net-(U6-VOUTD) -> Net-(U6C--)
- U7 pad 1: /buffered_mcp4729/OUT_1 -> +12V
- U7 pad 2: Net-(U7A--) -> GNDREF
- U7 pad 3: Net-(U6-VOUTA) -> +5V
- U8 pad 1: +5V -> Net-(R33-Pad1)
- U8 pad 10: GNDREF -> Net-(U11-VOUTC)
- U8 pad 2: /buffered_mcp4730/SCL -> Net-(U8A--)
- U8 pad 3: /buffered_mcp4730/SDA -> Net-(U11-VOUTA)
- U8 pad 4: unconnected-(U8-~{LDAC}-Pad4) -> +12V
- U8 pad 5: unconnected-(U8-RDY/~{BSY}-Pad5) -> Net-(U11-VOUTB)
- U8 pad 6: Net-(U8-VOUTA) -> Net-(U8B--)
- U8 pad 7: Net-(U8-VOUTB) -> Net-(R34-Pad1)
- U8 pad 8: Net-(U8-VOUTC) -> Net-(R35-Pad1)
- U8 pad 9: Net-(U8-VOUTD) -> Net-(U8C--)
- U9 pad 1: /buffered_mcp4730/OUT_1 -> Net-(R44-Pad1)
- U9 pad 10: Net-(U8-VOUTC) -> /gate_out/GATE_IN_3
- U9 pad 12: Net-(U8-VOUTD) -> /gate_out/GATE_IN_4
- U9 pad 14: /buffered_mcp4730/OUT_4 -> Net-(R56-Pad1)
- U9 pad 3: Net-(U8-VOUTA) -> /gate_out/GATE_IN_1
- U9 pad 5: Net-(U8-VOUTB) -> /gate_out/GATE_IN_2
- U9 pad 7: /buffered_mcp4730/OUT_2 -> Net-(R43-Pad1)
- U9 pad 8: /buffered_mcp4730/OUT_3 -> Net-(R55-Pad1)
- VEL_1 pad T: Net-(R10-Pad1) -> Net-(R23-Pad1)
- VEL_2 pad T: Net-(R11-Pad1) -> Net-(R24-Pad1)
- VEL_3 pad T: Net-(R12-Pad1) -> Net-(R25-Pad1)
- VEL_4 pad T: Net-(R13-Pad1) -> Net-(R26-Pad1)
Other:
- board size 81 x 111 mm -> 181 x 110 mm

Commit message: dd some more modules, update src for midi-2-cv
Parts:
- removed J2: DIN-6, Synth:MIDI_DIN5-SD-60BV
- removed U11: MCP4728, Package_SO:MSOP-10_3x3mm_P0.5mm
- added C17: 0.1uF, Capacitor_SMD:C_0805_2012Metric_Pad1.18x1.45mm_HandSolder, F.Cu at (82.7, 77.8)
- added C7: 0.1uF, Capacitor_THT:CP_Radial_D4.0mm_P2.00mm, B.Cu at (70.0, 57.5)
- added C8: 0.1uF, Capacitor_THT:CP_Radial_D4.0mm_P2.00mm, B.Cu at (70.0, 62.5)
- added G***: LOGO, Synth:lenimal_logo_full, F.Cu at (138.8, 139.0)
- added G***: LOGO, Synth:lenimal_logo_full, F.Cu at (55.7, 158.7)
- added G***: LOGO, Synth:lenimal_logo_full, B.Cu at (55.6, 158.7)
- added G***: LOGO, Synth:lenimal_logo_full, B.Cu at (138.6, 139.0)
- added H10: PinSocket_01x04, Synth:PinSocket_1x04_P2.54mm_Vertical, F.Cu at (79.0, 96.0)
- added H11: PinHeader_01x04, Synth:PinHeader_1x04_P2.54mm_Vertical, B.Cu at (130.0, 96.0)
- added H12: PinHeader_01x04, Synth:PinHeader_1x04_P2.54mm_Vertical, F.Cu at (64.0, 84.0)
- added H13: PinSocket_01x04, Synth:PinSocket_1x04_P2.54mm_Vertical, B.Cu at (115.0, 84.0)
- added H14: PinSocket_01x04, Synth:PinSocket_1x04_P2.54mm_Vertical, F.Cu at (73.0, 136.0)
- added H15: PinHeader_01x04, Synth:PinHeader_1x04_P2.54mm_Vertical, B.Cu at (124.0, 136.0)
- added H16: PinHeader_01x02, Synth:PinHeader_1x02_P2.54mm_Vertical, B.Cu at (117.0, 153.0)
- added H17: PinSocket_01x02, Synth:PinSocket_1x02_P2.54mm_Vertical, F.Cu at (66.0, 153.0)
- added H2: PinSocket_01x02, Synth:PinSocket_1x02_P2.54mm_Vertical, F.Cu at (66.0, 157.0)
- added H3: PinSocket_01x04, Synth:PinSocket_1x04_P2.54mm_Vertical, F.Cu at (66.0, 116.0)
- added H4: PinHeader_01x04, Synth:PinHeader_1x04_P2.54mm_Vertical, B.Cu at (117.0, 116.0)
- added H5: PinSocket_01x04, Synth:PinSocket_1x04_P2.54mm_Vertical, F.Cu at (90.0, 76.0)
- added H6: PinHeader_01x04, Synth:PinHeader_1x04_P2.54mm_Vertical, B.Cu at (141.0, 76.0)
- added H7: Conn_02x05_PWR_Eurorack, Synth:IDC-Header_2x05_P2.54mm_Vertical, B.Cu at (54.0, 66.0)
- added H8: PinSocket_01x04, Synth:PinSocket_1x04_P2.54mm_Vertical, B.Cu at (140.9, 52.5)
- added H9: PinHeader_01x04, Synth:PinHeader_1x04_P2.54mm_Vertical, F.Cu at (89.9, 52.5)
- added J1: DIN-6, Synth:MIDI_DIN5-SD-60BV, F.Cu at (142.0, 151.0)
- added R65: 6K8, Resistor_SMD:R_0805_2012Metric_Pad1.20x1.40mm_HandSolder, F.Cu at (60.5, 138.4)
- added R66: 6K8, Resistor_SMD:R_0805_2012Metric_Pad1.20x1.40mm_HandSolder, F.Cu at (59.9, 114.0)
- added R67: 6K8, Resistor_SMD:R_0805_2012Metric_Pad1.20x1.40mm_HandSolder, F.Cu at (59.6, 143.6)
- added R68: 6K8, Resistor_SMD:R_0805_2012Metric_Pad1.20x1.40mm_HandSolder, F.Cu at (59.6, 151.0)
- added RV1: 20K, Potentiometer_THT:Potentiometer_Piher_PT-6-V_Vertical, B.Cu at (57.4, 137.0)
- added RV2: 20K, Potentiometer_THT:Potentiometer_Piher_PT-6-V_Vertical, B.Cu at (52.7, 118.2)
- added RV3: 20K, Potentiometer_THT:Potentiometer_Piher_PT-6-V_Vertical, B.Cu at (57.4, 144.4)
- added RV4: 20K, Potentiometer_THT:Potentiometer_Piher_PT-6-V_Vertical, B.Cu at (57.4, 151.8)
- added SW1: ON-OFF-ON, Synth:SW_default, F.Cu at (107.0, 149.8)
- added TP1: GND, Connector_Pin:Pin_D1.0mm_L10.0mm, F.Cu at (75.3, 60.0)
- added TP10: GATE_1_OUT, Connector_Pin:Pin_D1.0mm_L10.0mm, B.Cu at (62.8, 76.2)
- added TP11: CV_2_OUT, Connector_Pin:Pin_D1.0mm_L10.0mm, B.Cu at (74.7, 119.8)
- added TP12: CV_1_OUT, Connector_Pin:Pin_D1.0mm_L10.0mm, B.Cu at (62.5, 118.6)
- added TP13: CV_3_OUT, Connector_Pin:Pin_D1.0mm_L10.0mm, B.Cu at (53.0, 122.8)
- added TP14: CV_4_OUT, Connector_Pin:Pin_D1.0mm_L10.0mm, B.Cu at (53.0, 128.9)
- added TP2: +12V, Connector_Pin:Pin_D1.0mm_L10.0mm, F.Cu at (75.3, 56.8)
- added TP3: -12V, Connector_Pin:Pin_D1.0mm_L10.0mm, F.Cu at (75.3, 63.3)
- added TP4: +5V, Connector_Pin:Pin_D1.0mm_L10.0mm, B.Cu at (76.3, 102.6)
- added TP5: +3.3V, Connector_Pin:Pin_D1.0mm_L10.0mm, B.Cu at (67.0, 148.5)
- added TP6: MIDI_IN, Connector_Pin:Pin_D1.0mm_L10.0mm, B.Cu at (73.0, 156.2)
- added TP7: GATE_3_OUT, Connector_Pin:Pin_D1.0mm_L10.0mm, B.Cu at (53.1, 99.6)
- added TP8: GATE_4_OUT, Connector_Pin:Pin_D1.0mm_L10.0mm, B.Cu at (60.6, 99.5)
- added TP9: GATE_2_OUT, Connector_Pin:Pin_D1.0mm_L10.0mm, B.Cu at (53.1, 75.7)
- added U10: MCP4728, Package_SO:MSOP-10_3x3mm_P0.5mm, F.Cu at (78.9, 80.0)
- C1: footprint Capacitor_THT:CP_Radial_D4.0mm_P2.00mm -> Capacitor_SMD:C_0805_2012Metric_Pad1.18x1.45mm_HandSolder
- C10, C11, C12, C13, C14, C15, C16, C9: footprint Capacitor_THT:C_Disc_D5.0mm_W2.5mm_P5.00mm -> Capacitor_SMD:C_0805_2012Metric_Pad1.18x1.45mm_HandSolder
- C2: value 47uF -> 0.1uF; footprint Capacitor_THT:CP_Radial_D6.3mm_P2.50mm -> Capacitor_SMD:C_0805_2012Metric_Pad1.18x1.45mm_HandSolder
- C3: value 47uF -> 0.1uF; footprint Capacitor_THT:CP_Radial_D6.3mm_P2.50mm -> Capacitor_THT:CP_Radial_D4.0mm_P2.00mm; moved to B.Cu
- C4, C5: value 0.1uF -> 47uF; footprint Capacitor_THT:CP_Radial_D4.0mm_P2.00mm -> Capacitor_THT:CP_Radial_D6.3mm_P2.50mm; moved to B.Cu
- C6: moved to B.Cu
- CV_OUT_1: value CV_OUT_2 -> CV_OUT_1
- CV_OUT_2: value CV_OUT_3 -> CV_OUT_2
- CV_OUT_3: value CV_OUT_4 -> CV_OUT_3
- CV_OUT_4: value CV_OUT_1 -> CV_OUT_4
- D1: footprint Synth:D_DO-35_SOD27_P7.62mm_Horizontal -> Diode_SMD:D_SOD-123
- D2, D3: footprint Synth:D_DO-41_SOD81_P10.16mm_Horizontal -> Diode_SMD:D_SOD-123; moved to B.Cu
- D4, D5, D6, D7: footprint Synth:LED_D5.0mm (center Aligned) -> Synth:LED_D3.0mm
- GATE_1: value GATE_2 -> GATE_1
- GATE_2: value GATE_1 -> GATE_2
- H1: value Conn_02x05_PWR_Eurorack -> PinHeader_01x02; footprint Synth:IDC-Header_2x05_P2.54mm_Vertical -> Synth:PinHeader_1x02_P2.54mm_Vertical; moved to B.Cu
- MOD_1: value MOD_2 -> MOD_1
- MOD_2: value MOD_3 -> MOD_2
- MOD_3: value MOD_4 -> MOD_3
- MOD_4: value MOD_1 -> MOD_4
- Q1, Q2, Q3, Q4: value BC548 -> BC848; footprint Package_TO_SOT_THT:TO-92_Inline -> Package_TO_SOT_SMD:SOT-23; moved to B.Cu
- R1, R15, R16, R17, R18, R19, R2, R20, R21, R22, R29, R30, R31, R32, R33, R34, R35, R36, R41, R42, R43, R44, R45, R46, R51, R52, R53, R54, R55, R56, R57, R58, R63, R64: footprint Synth:R_Default (DIN0207) -> Resistor_SMD:R_0805_2012Metric_Pad1.20x1.40mm_HandSolder
- R10, R7, R8, R9: value 47K [1%] -> 47K [0.1%]; footprint Synth:R_Default (DIN0207) -> Resistor_SMD:R_0805_2012Metric_Pad1.20x1.40mm_HandSolder
- R11, R12, R13, R14, R23, R24, R25, R26, R37, R38, R39, R40, R47, R48, R49, R50, R59, R60, R61, R62: footprint Synth:R_Default (DIN0207) -> Resistor_SMD:R_0805_2012Metric_Pad1.20x1.40mm_HandSolder; moved to B.Cu
- R27, R28: value 10 -> 10R; footprint Synth:R_Default (DIN0207) -> Resistor_SMD:R_0805_2012Metric_Pad1.20x1.40mm_HandSolder; moved to B.Cu
- R3, R4, R5, R6: value 10K [1%] -> 10K [0.1%]; footprint Synth:R_Default (DIN0207) -> Resistor_SMD:R_0805_2012Metric_Pad1.20x1.40mm_HandSolder
- U2: footprint stm32:YAAJ_WeAct_BlackPill_SWD_2 -> stm32:YAAJ_WeAct_BlackPill_2
- U7: footprint Package_TO_SOT_THT:TO-220-3_Horizontal_TabDown -> Package_TO_SOT_SMD:SOT-89-3_Handsoldering
- VEL_1: value VEL_2 -> VEL_1
- VEL_2: value VEL_3 -> VEL_2
- VEL_3: value VEL_4 -> VEL_3
- VEL_4: value VEL_1 -> VEL_4
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Connections:
- C1 pad 1: +12V -> GNDREF
- C1 pad 2: GNDREF -> +5V
- C2 pad 1: +12V -> GNDREF
- C2 pad 2: GNDREF -> +5V
- C3 pad 1: GNDREF -> +12V
- C3 pad 2: -12V -> GNDREF
- C4 pad 1: +5V -> +12V
- C5 pad 1: +12V -> GNDREF
- C5 pad 2: GNDREF -> -12V
- C6 pad 1: GNDREF -> +5V
- C6 pad 2: -12V -> GNDREF
- GATE_1 pad TN: /gate_out/GATE_2_CALLBACK -> Net-(H15A-Pin_1)
- GATE_2 pad TN: /gate_out/GATE_1_CALLBACK -> Net-(H15B-Pin_2)
- GATE_3 pad TN: /gate_out/GATE_3_CALLBACK -> Net-(H15C-Pin_3)
- GATE_4 pad TN: /gate_out/GATE_4_CALLBACK -> Net-(H15D-Pin_4)
- H1 pad 1: Net-(D3-K) -> +3.3V
- H1 pad 2: Net-(D3-K) -> Net-(H1B-Pin_2)
- Q1 pad 1: Net-(D4-A) -> Net-(Q1-B)
- Q1 pad 2: Net-(Q1-B) -> +12V
- Q1 pad 3: +12V -> Net-(D4-A)
- Q2 pad 1: Net-(D5-A) -> Net-(Q2-B)
- Q2 pad 2: Net-(Q2-B) -> +12V
- Q2 pad 3: +12V -> Net-(D5-A)
- Q3 pad 1: Net-(D6-A) -> Net-(Q3-B)
- Q3 pad 2: Net-(Q3-B) -> +12V
- Q3 pad 3: +12V -> Net-(D6-A)
- Q4 pad 1: Net-(D7-A) -> Net-(Q4-B)
- Q4 pad 2: Net-(Q4-B) -> +12V
- Q4 pad 3: +12V -> Net-(D7-A)
- R1 pad 1: Net-(J2-Pad2) -> Net-(D1-K)
- R1 pad 2: Net-(D1-K) -> Net-(J1-Pad2)
- R10 pad 1: Net-(R10-Pad1) -> Net-(U4D--)
- R10 pad 2: Net-(U4D--) -> Net-(H3D-Pin_4)
- R11 pad 1: Net-(CV_OUT_1-PadT) -> Net-(H4B-Pin_2)
- R11 pad 2: Net-(R11-Pad2) -> Net-(CV_OUT_2-PadT)
- R12 pad 1: Net-(CV_OUT_2-PadT) -> Net-(H4C-Pin_3)
- R12 pad 2: Net-(R12-Pad2) -> Net-(CV_OUT_3-PadT)
- R13 pad 1: Net-(CV_OUT_3-PadT) -> Net-(H4D-Pin_4)
- R13 pad 2: Net-(R10-Pad1) -> Net-(CV_OUT_4-PadT)
- R14 pad 1: Net-(CV_OUT_4-PadT) -> Net-(H4A-Pin_1)
- R14 pad 2: Net-(R14-Pad2) -> Net-(CV_OUT_1-PadT)
- R15 pad 1: Net-(U6A--) -> GNDREF
- R15 pad 2: GNDREF -> Net-(U6A--)
- R16 pad 1: Net-(U6B--) -> GNDREF
- R16 pad 2: GNDREF -> Net-(U6B--)
- R17 pad 1: Net-(U6C--) -> GNDREF
- R17 pad 2: GNDREF -> Net-(U6C--)
- R18 pad 1: Net-(U6D--) -> GNDREF
- R18 pad 2: GNDREF -> Net-(U6D--)
- R19 pad 1: Net-(R19-Pad1) -> Net-(U6A--)
- R19 pad 2: Net-(U6A--) -> Net-(H5A-Pin_1)
- R2 pad 1: +3.3V -> Net-(H1B-Pin_2)
- R2 pad 2: Net-(U2-PA10) -> +3.3V
- R20 pad 1: Net-(R20-Pad1) -> Net-(U6B--)
- R20 pad 2: Net-(U6B--) -> Net-(H5B-Pin_2)
- R21 pad 1: Net-(R21-Pad1) -> Net-(U6C--)
- R21 pad 2: Net-(U6C--) -> Net-(H5C-Pin_3)
- R22 pad 1: Net-(R22-Pad1) -> Net-(U6D--)
- R22 pad 2: Net-(U6D--) -> Net-(H5D-Pin_4)
- R23 pad 1: Net-(R23-Pad1) -> Net-(H6B-Pin_2)
- R23 pad 2: Net-(R20-Pad1) -> Net-(MOD_2-PadT)
- R24 pad 1: Net-(R24-Pad1) -> Net-(H6C-Pin_3)
- R24 pad 2: Net-(R21-Pad1) -> Net-(MOD_3-PadT)
- R25 pad 1: Net-(R25-Pad1) -> Net-(H6D-Pin_4)
- R25 pad 2: Net-(R22-Pad1) -> Net-(MOD_4-PadT)
- R26 pad 1: Net-(R26-Pad1) -> Net-(H6A-Pin_1)
- R26 pad 2: Net-(R19-Pad1) -> Net-(MOD_1-PadT)
- R27 pad 1: +12V -> Net-(D2-K)
- R27 pad 2: Net-(D2-K) -> +12V
- R28 pad 1: -12V -> Net-(D3-A)
- R28 pad 2: Net-(D3-A) -> -12V
- R29 pad 1: Net-(U8A--) -> GNDREF
- R29 pad 2: GNDREF -> Net-(U8A--)
- R3 pad 1: Net-(U4A--) -> GNDREF
- R3 pad 2: GNDREF -> Net-(U4A--)
- R30 pad 1: Net-(U8B--) -> GNDREF
- R30 pad 2: GNDREF -> Net-(U8B--)
- R31 pad 1: Net-(U8C--) -> GNDREF
- R31 pad 2: GNDREF -> Net-(U8C--)
- R32 pad 1: Net-(U8D--) -> GNDREF
- R32 pad 2: GNDREF -> Net-(U8D--)
- R33 pad 1: Net-(R33-Pad1) -> Net-(U8A--)
- R33 pad 2: Net-(U8A--) -> Net-(H10A-Pin_1)
- R34 pad 1: Net-(R34-Pad1) -> Net-(U8B--)
- R34 pad 2: Net-(U8B--) -> Net-(H10B-Pin_2)
- R35 pad 1: Net-(R35-Pad1) -> Net-(U8C--)
- R35 pad 2: Net-(U8C--) -> Net-(H10C-Pin_3)
- R36 pad 1: Net-(R36-Pad1) -> Net-(U8D--)
- R36 pad 2: Net-(U8D--) -> Net-(H10D-Pin_4)
- R37 pad 1: Net-(MOD_1-PadT) -> Net-(H11B-Pin_2)
- R37 pad 2: Net-(R34-Pad1) -> Net-(R37-Pad2)
- R38 pad 1: Net-(MOD_2-PadT) -> Net-(H11C-Pin_3)
- R38 pad 2: Net-(R35-Pad1) -> Net-(R38-Pad2)
- R39 pad 1: Net-(MOD_3-PadT) -> Net-(H11D-Pin_4)
- R39 pad 2: Net-(R36-Pad1) -> Net-(R39-Pad2)
- R4 pad 1: Net-(U4B--) -> GNDREF
- R4 pad 2: GNDREF -> Net-(U4B--)
- R40 pad 1: Net-(MOD_4-PadT) -> Net-(H11A-Pin_1)
- R40 pad 2: Net-(R33-Pad1) -> Net-(R40-Pad2)
- R41 pad 1: Net-(U9B--) -> GNDREF
- R41 pad 2: GNDREF -> Net-(U9A--)
- R42 pad 1: Net-(U9A--) -> GNDREF
- R42 pad 2: GNDREF -> Net-(U9B--)
- R43 pad 1: Net-(R43-Pad1) -> Net-(U9A--)
- R43 pad 2: Net-(U9B--) -> Net-(H12A-Pin_1)
- R44 pad 1: Net-(R44-Pad1) -> Net-(U9B--)
- R44 pad 2: Net-(U9A--) -> Net-(H12B-Pin_2)
- R45 pad 1: Net-(D4-K) -> GNDREF
- R45 pad 2: GNDREF -> Net-(D4-K)
- R46 pad 1: Net-(D5-K) -> GNDREF
- R46 pad 2: GNDREF -> Net-(D5-K)
- R47 pad 1: Net-(Q1-B) -> Net-(H13A-Pin_1)
- R47 pad 2: Net-(R43-Pad1) -> Net-(Q1-B)
- R48 pad 1: Net-(Q2-B) -> Net-(H13B-Pin_2)
- R48 pad 2: Net-(R44-Pad1) -> Net-(Q2-B)
- R49 pad 1: Net-(GATE_1-PadT) -> Net-(H13A-Pin_1)
- R49 pad 2: Net-(R43-Pad1) -> Net-(GATE_1-PadT)
- R5 pad 1: Net-(U4C--) -> GNDREF
- R5 pad 2: GNDREF -> Net-(U4C--)
- R50 pad 1: Net-(GATE_2-PadT) -> Net-(H13B-Pin_2)
- R50 pad 2: Net-(R44-Pad1) -> Net-(GATE_2-PadT)
- R51 pad 1: +3.3V -> /gate_out/GATE_1_CALLBACK
- R51 pad 2: /gate_out/GATE_2_CALLBACK -> +3.3V
- R52 pad 1: +3.3V -> /gate_out/GATE_2_CALLBACK
- R52 pad 2: /gate_out/GATE_1_CALLBACK -> +3.3V
- R53 pad 1: Net-(U9D--) -> GNDREF
- R53 pad 2: GNDREF -> Net-(U9C--)
- R54 pad 1: Net-(U9C--) -> GNDREF
- R54 pad 2: GNDREF -> Net-(U9D--)
- R55 pad 1: Net-(R55-Pad1) -> Net-(U9C--)
- R55 pad 2: Net-(U9C--) -> Net-(H12C-Pin_3)
- R56 pad 1: Net-(R56-Pad1) -> Net-(U9D--)
- R56 pad 2: Net-(U9D--) -> Net-(H12D-Pin_4)
- R57 pad 1: Net-(D6-K) -> GNDREF
- R57 pad 2: GNDREF -> Net-(D6-K)
- R58 pad 1: Net-(D7-K) -> GNDREF
- R58 pad 2: GNDREF -> Net-(D7-K)
- R59 pad 1: Net-(Q3-B) -> Net-(H13C-Pin_3)
- R59 pad 2: Net-(R55-Pad1) -> Net-(Q3-B)
- R6 pad 1: Net-(U4D--) -> GNDREF
- R6 pad 2: GNDREF -> Net-(U4D--)
- R60 pad 1: Net-(Q4-B) -> Net-(H13D-Pin_4)
- R60 pad 2: Net-(R56-Pad1) -> Net-(Q4-B)
- R61 pad 1: Net-(GATE_3-PadT) -> Net-(H13C-Pin_3)
- R61 pad 2: Net-(R55-Pad1) -> Net-(GATE_3-PadT)
- R62 pad 1: Net-(GATE_4-PadT) -> Net-(H13D-Pin_4)
- R62 pad 2: Net-(R56-Pad1) -> Net-(GATE_4-PadT)
- R63 pad 1: +3.3V -> /gate_out/GATE_3_CALLBACK
- R63 pad 2: /gate_out/GATE_3_CALLBACK -> +3.3V
- R64 pad 1: +3.3V -> /gate_out/GATE_4_CALLBACK
- R64 pad 2: /gate_out/GATE_4_CALLBACK -> +3.3V
- R7 pad 1: Net-(R14-Pad2) -> Net-(U4A--)
- R7 pad 2: Net-(U4A--) -> Net-(H3A-Pin_1)
- R8 pad 1: Net-(R11-Pad2) -> Net-(U4B--)
- R8 pad 2: Net-(U4B--) -> Net-(H3B-Pin_2)
- R9 pad 1: Net-(R12-Pad2) -> Net-(U4C--)
- R9 pad 2: Net-(U4C--) -> Net-(H3C-Pin_3)
- U1 pad 6: Net-(U2-PA10) -> Net-(H1B-Pin_2)
- U2 pad 11: /mcp4728_vel-out/SDA -> /mcp4728_velocity-out/SDA
- U2 pad 12: /mcp4728_mod-out/SDA -> /mcp4728_mod-wheel-out/SDA
- U2 pad 16: /mcp4728_mod-out/SCL -> /mcp4728_mod-wheel-out/SCL
- U2 pad 23: unconnected-(U2-PC14-Pad23) -> Net-(H17A-Pin_1)
- U2 pad 24: unconnected-(U2-PC15-Pad24) -> Net-(H17B-Pin_2)
- U2 pad 26: /gate_out/GATE_1_CALLBACK -> /gate_out/GATE_4_CALLBACK
- U2 pad 27: /gate_out/GATE_2_CALLBACK -> /gate_out/GATE_3_CALLBACK
- U2 pad 28: /gate_out/GATE_3_CALLBACK -> /gate_out/GATE_2_CALLBACK
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Routing:
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- added copper zone on B.Cu, net (none)
- added copper zone on F.Cu, net GNDREF
Other:
- board size 181 x 110 mm -> 101 x 110 mm
- board text added: "+12V"
- board text added: "+3.3V"
- board text added: "+5V"
- board text added: "-12V"
- board text added: "CH.1"
- board text added: "CH.2"
- board text added: "CH.3"
- board text added: "CH.4"
- board text added: "CHANNEL"
- board text added: "CV"
- board text added: "Channel 1"
- board text added: "Channel 2"
- board text added: "Channel 3"
- board text added: "Channel 4"
- board text added: "FIRST"
- board text added: "GATE"
- board text added: "GATE.1"
- board text added: "GATE.2"
- board text added: "GATE.3"
- board text added: "GATE.4"
- board text added: "GND"
- board text added: "King of MIDI"
- board text added: "LENIMAL PCB DESIGN - 09.2024"
- board text added: "MIDAS"
- board text added: "MIDI_IN"
- board text added: "MOD"
- board text added: "SEQ"
- board text added: "USB SIDE"
- board text added: "USE EITHER TRIM POT OR MARKED RESISTORS, NOT BOTH!"
- board text added: "Velocity"
