File: modules/effects/reverb/kiCad/reverb-dsp-brain/reverb-dsp-brain.kicad_pcb (KiCad board)
At the start: 4 copper layers, 50 x 60 mm, 50 parts, among them J1 AUDIO_IN_OUT, J10 Conn_01x06, J11 Conn_01x06, J2 LED_DRIVER, J3 Power, J4 V_VA_CONN, J5 BOOT_RUN, J6 UART, J7 SWD, J8 Conn_01x08, J9 Conn_01x06, U1 STM32F405RGT6, U2 WM8731SEDS, Y1 8MHZ, Y2 12.288MHZ

Commit message: finished clouds clone (weathering/the storm)
Parts:
- removed D2: LED, LED_SMD:LED_0805_2012Metric_Pad1.15x1.40mm_HandSolder
- removed the G*** at (91.7, 90.7)
- removed the G*** at (56.8, 74.3)
- removed the G*** at (56.9, 74.3)
- removed the G*** at (90.6, 90.7)
- removed J7: SWD, Connector_PinHeader_2.54mm:PinHeader_2x05_P2.54mm_Vertical
- removed R5: 10K, Resistor_SMD:R_0805_2012Metric_Pad1.20x1.40mm_HandSolder
- removed Y2: 12.288MHZ, Crystal:Crystal_HC49-U_Vertical
- added C22: 10uF, Capacitor_SMD:C_0805_2012Metric_Pad1.18x1.45mm_HandSolder, F.Cu at (53.0, 53.0)
- added G***: LOGO, Synth:lenimal_logo_full, F.Cu at (83.8, 62.5)
- added G***: LOGO, Synth:lenimal_logo_full, B.Cu at (83.5, 62.5)
- added R10: 5K1, Resistor_SMD:R_0805_2012Metric_Pad1.20x1.40mm_HandSolder, F.Cu at (56.8, 85.0)
- added R8: 5K1, Resistor_SMD:R_0805_2012Metric_Pad1.20x1.40mm_HandSolder, F.Cu at (55.2, 91.5)
- added R9: 5K1, Resistor_SMD:R_0805_2012Metric_Pad1.20x1.40mm_HandSolder, F.Cu at (55.2, 93.5)
- added U3: LM1117MP-5.0, Package_TO_SOT_SMD:SOT-223-3_TabPin2, F.Cu at (59.0, 55.5)
- C10: value 2.2uF -> 100nF
- C11: value 2.2uF -> 10uF
- C14: value 100nF -> 47uF
- C15: value 10uF -> 100nF
- C16: value 100nF -> 10uF
- C17: value 10uF -> 2.2uF
- C18: value 18pF -> 2.2uF
- C19: value 1uF -> 10uF
- C20: value 10uF -> 100nF; footprint Capacitor_THT:CP_Radial_D4.0mm_P2.00mm -> Capacitor_SMD:C_0805_2012Metric_Pad1.18x1.45mm_HandSolder
- C21: value 18pF -> 10uF
- J5: value BOOT_RUN -> SWD; footprint Connector_PinHeader_2.54mm:PinHeader_1x03_P2.54mm_Vertical -> Connector_PinHeader_2.54mm:PinHeader_2x03_P2.54mm_Vertical
- R2: value 1K -> 10R
- R3: value 10K -> 2K2
- R4: value 10R -> 2K2
- R6: value 2K2 -> 47K; moved to F.Cu
- R7: value 2K2 -> 5K1; moved to F.Cu
- U1: value STM32F405RGT6 -> STM32G474RBTx
- U2: value WM8731SEDS -> CS4270; footprint Package_SO:SSOP-28_5.3x10.2mm_P0.65mm -> Package_SO:TSSOP-24_4.4x7.8mm_P0.65mm
- Y1: value 8MHZ -> 20MHZ; footprint Crystal:Crystal_HC49-U_Vertical -> Crystal:Crystal_SMD_HC49-SD_HandSoldering
- moved D1 68.3 mm to (97.0, 103.8), turned to 180 degrees
- moved R1 64.6 mm to (97.0, 100.8)
- moved C10 51.2 mm to (56.8, 99.8), turned to 180 degrees
- moved C11 49.7 mm to (56.8, 102.0), turned to 180 degrees
- moved R7 44.5 mm to (55.2, 95.5), turned to 0 degrees
- moved C21 42.9 mm to (53.5, 71.0)
- moved J4 33.5 mm to (91.5, 53.0), turned to -90 degrees
- moved C18 29.2 mm to (57.0, 88.0), turned to 180 degrees
- moved C4 28.8 mm to (65.2, 80.2), turned to 90 degrees
- moved R6 27.6 mm to (68.5, 86.8), turned to 180 degrees
- moved FB1 25.7 mm to (87.0, 56.0), turned to 180 degrees
- moved C6 23.0 mm to (70.0, 64.2), turned to -90 degrees
- moved C7 22.8 mm to (83.8, 57.0), turned to 90 degrees
- moved C20 20.9 mm to (60.2, 87.2), turned to 90 degrees
- moved C9 19.6 mm to (91.2, 70.5), turned to 90 degrees
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Connections:
- C10 pad 1: /STM32/VCAP_1 -> Net-(U2-VQ)
- C11 pad 1: /STM32/VCAP_2 -> Net-(U2-VQ)
- C12 pad 1: GNDREF -> +3.3V
- C12 pad 2: /STM32/NRST -> GNDREF
- C13 pad 2: +3.3V -> Net-(U2-FIL+)
- C14 pad 2: +3.3V -> Net-(U2-FIL+)
- C15 pad 1: GNDREF -> +5VA
- C15 pad 2: +3.3V -> GNDREF
- C16 pad 1: GNDREF -> +5VA
- C16 pad 2: +3.3VA -> GNDREF
- C17 pad 1: GNDREF -> /CS4270/RST
- C17 pad 2: +3.3VA -> GNDREF
- C18 pad 1: Net-(U2-XTI/MCLK) -> Net-(U2-~{RST})
- C19 pad 1: GNDREF -> +3.3V
- C19 pad 2: Net-(U2-VMID) -> GNDREF
- C20 pad 1: Net-(U2-VMID) -> +3.3V
- C21 pad 1: Net-(U2-XTO) -> +5VA
- C8 pad 1: /STM32/HSC_OUT -> Net-(C8-Pad1)
- C9 pad 1: Net-(C9-Pad1) -> /STM32/HSC_OUT
- D1 pad 1: Net-(D1-K) -> GNDREF
- D1 pad 2: GNDREF -> Net-(D1-A)
- J1 pad 1: /audio-codec/L_IN -> /CS4270/INPUT_B
- J1 pad 2: /audio-codec/R_IN -> /CS4270/INPUT_A
- J1 pad 3: /audio-codec/L_OUT -> /CS4270/OUTPUT_B
- J1 pad 4: /audio-codec/R_OUT -> /CS4270/OUTPUT_A
- J3 pad 4: unconnected-(J3-Pin_4-Pad4) -> +12V
- J3 pad 5: unconnected-(J3-Pin_5-Pad5) -> +12V
- J5 pad 1: GNDREF -> +3.3V
- J5 pad 2: Net-(D2-A) -> /STM32/SWD_IO
- J5 pad 3: +3.3V -> GNDREF
- R1 pad 1: Net-(D1-K) -> Net-(D1-A)
- R2 pad 1: Net-(D2-K) -> Net-(C8-Pad1)
- R2 pad 2: GNDREF -> /STM32/HSC_IN
- R3 pad 1: Net-(D2-A) -> +3.3V
- R3 pad 2: /STM32/BOOT0 -> /CS4270/I2C_SDA
- R4 pad 1: Net-(C9-Pad1) -> /CS4270/I2C_SCL
- R4 pad 2: /STM32/HSC_IN -> +3.3V
- R6 pad 1: /STM32/I2C_SCL -> +3.3V
- R6 pad 2: +3.3V -> /CS4270/SAI_SDOUT
- R7 pad 1: +3.3V -> GNDREF
- R7 pad 2: /STM32/I2C_SDA -> Net-(U2-AD2/MDIV2)
- U1 pad 11: unconnected-(U1-PC3-Pad11) -> /CS4270/SAI_SDIN
- U1 pad 12: GNDREF -> /STM32/V_OCT
- U1 pad 13: +3.3VA -> /STM32/POSITION_CV
- U1 pad 14: /STM32/TEXTURE_CV -> /STM32/DENSITY_CV
- U1 pad 15: /STM32/SIZE_CV -> GNDREF
- U1 pad 16: /STM32/POSITION_CV -> +3.3V
- U1 pad 17: /STM32/DENSITY_CV -> /STM32/PITCH
- U1 pad 18: GNDREF -> unconnected-(U1-PA4-Pad18)
- U1 pad 19: +3.3V -> unconnected-(U1-PA5-Pad19)
- U1 pad 20: /STM32/V_OCT -> /STM32/TEXTURE
- U1 pad 21: /STM32/BLEND_CV -> /STM32/TEXTURE_CV
- U1 pad 22: /STM32/TEXTURE -> /STM32/BLEND
- U1 pad 23: /STM32/BLEND -> /STM32/RX
- U1 pad 24: /STM32/LED_ENABLE -> unconnected-(U1-PB0-Pad24)
- U1 pad 25: /STM32/LED_CLK -> unconnected-(U1-PB1-Pad25)
- U1 pad 26: GNDREF -> unconnected-(U1-PB2-Pad26)
- U1 pad 27: unconnected-(U1-PB1-Pad27) -> GNDREF
- U1 pad 28: GNDREF -> +3.3VA
- U1 pad 29: /STM32/I2C_SCL -> +3.3VA
- U1 pad 30: /STM32/I2C_SDA -> unconnected-(U1-PB10-Pad30)
- U1 pad 31: /STM32/VCAP_1 -> GNDREF
- U1 pad 33: /STM32/I2S_LRCK -> /CS4270/SAI_SCLK
- U1 pad 34: /STM32/I2S_SCK -> /CS4270/RST
- U1 pad 35: /STM32/I2S_SIN -> /STM32/SW_LOAD
- U1 pad 36: /STM32/I2S_SOUT -> /STM32/BLEND_CV
- U1 pad 37: unconnected-(U1-PC6-Pad37) -> /STM32/SW_MODE
- U1 pad 38: unconnected-(U1-PC7-Pad38) -> /STM32/SW_FREEZE
- U1 pad 39: unconnected-(U1-PC8-Pad39) -> /STM32/FREEZE_LED
- U1 pad 40: unconnected-(U1-PC9-Pad40) -> /STM32/PLAY_TRIGGER
- U1 pad 41: unconnected-(U1-PA8-Pad41) -> /STM32/FREEZE_TRIGGER
- U1 pad 42: /STM32/TX -> unconnected-(U1-PA8-Pad42)
- U1 pad 43: /STM32/RX -> /CS4270/SAI_LRCLK
- U1 pad 46: /STM32/SWD_IO -> unconnected-(U1-PA12-Pad46)
- U1 pad 47: /STM32/VCAP_2 -> GNDREF
- U1 pad 49: /STM32/SWD_CLK -> /STM32/SWD_IO
- U1 pad 5: /STM32/HSC_OUT -> /STM32/HSC_IN
- U1 pad 50: unconnected-(U1-PA15-Pad50) -> /STM32/SWD_CLK
- U1 pad 51: /STM32/SW_LOAD -> /CS4270/I2C_SCL
- U1 pad 52: /STM32/SW_MODE -> /STM32/LED_CLK
- U1 pad 53: unconnected-(U1-PC12-Pad53) -> /STM32/LED_ENABLE
- U1 pad 54: unconnected-(U1-PD2-Pad54) -> /STM32/LED_DATA
- U1 pad 55: /STM32/SWD_O -> unconnected-(U1-PD2-Pad55)
- U1 pad 56: unconnected-(U1-PB4-Pad56) -> /STM32/SWD_O
- U1 pad 57: /STM32/LED_DATA -> unconnected-(U1-PB4-Pad57)
- U1 pad 58: /STM32/PLAY_TRIGGER -> /CS4270/SAI_SDOUT
- U1 pad 59: /STM32/FREEZE_TRIGGER -> /STM32/TX
- U1 pad 6: /STM32/HSC_IN -> /STM32/HSC_OUT
- U1 pad 60: /STM32/BOOT0 -> /CS4270/I2C_SDA
- U1 pad 61: /STM32/SW_FREEZE -> /CS4270/SAI_MCLK
- U1 pad 62: /STM32/FREEZE_LED -> unconnected-(U1-PB9-Pad62)
- U1 pad 7: /STM32/NRST -> unconnected-(U1-PG10-Pad7)
- U1 pad 9: /STM32/PITCH -> /STM32/SIZE_CV
- U2 pad 1: +3.3V -> /CS4270/SAI_SDIN
- U2 pad 10: unconnected-(U2-RHPOUT-Pad10) -> /CS4270/I2C_SCL
- U2 pad 11: GNDREF -> Net-(U2-AD0/~{CS}/I2S/~{LJ})
- U2 pad 12: /audio-codec/L_OUT -> Net-(U2-AD1/CDIN/MDIV1)
- U2 pad 13: /audio-codec/R_OUT -> Net-(U2-AD2/MDIV2)
- U2 pad 14: +3.3VA -> Net-(U2-~{RST})
- U2 pad 15: GNDREF -> /CS4270/INPUT_A
- U2 pad 16: Net-(U2-VMID) -> /CS4270/INPUT_B
- U2 pad 17: unconnected-(U2-MICBIAS-Pad17) -> Net-(U2-VQ)
- U2 pad 18: unconnected-(U2-MICIN-Pad18) -> Net-(U2-FIL+)
- U2 pad 19: /audio-codec/R_IN -> +5VA
- U2 pad 2: unconnected-(U2-CLKOUT-Pad2) -> /CS4270/SAI_LRCLK
- U2 pad 20: /audio-codec/L_IN -> GNDREF
- U2 pad 21: GNDREF -> unconnected-(U2-~{MUTEA}-Pad21)
- U2 pad 22: GNDREF -> /CS4270/OUTPUT_A
- U2 pad 23: /STM32/I2C_SDA -> /CS4270/OUTPUT_B
- U2 pad 24: /STM32/I2C_SCL -> unconnected-(U2-~{MUTEB}-Pad24)
- U2 pad 3: /STM32/I2S_SCK -> /CS4270/SAI_MCLK
- U2 pad 4: /STM32/I2S_SOUT -> /CS4270/SAI_SCLK
- U2 pad 5: /STM32/I2S_LRCK -> +3.3V
- U2 pad 6: /STM32/I2S_SIN -> GNDREF
- U2 pad 7: /STM32/I2S_LRCK -> /CS4270/SAI_SDOUT
- U2 pad 8: +3.3VA -> +3.3V
- U2 pad 9: unconnected-(U2-LHPOUT-Pad9) -> /CS4270/I2C_SDA
- Y1 pad 1: /STM32/HSC_OUT -> Net-(C8-Pad1)
- Y1 pad 2: Net-(C9-Pad1) -> /STM32/HSC_OUT
Routing:
- net +3.3VA: track 167.4 -> 35.9 mm, vias 4 -> 2
- net +5VA: track 0.00 -> 78.2 mm, vias 0 -> 2
- net /STM32/I2C_SDA: track 72.2 -> 0.00 mm, vias 2 -> 0
- net /STM32/I2C_SCL: track 69.3 -> 0.00 mm, vias 2 -> 0
- net /STM32/I2S_SOUT: track 54.6 -> 0.00 mm, vias 2 -> 0
- net /STM32/I2S_SIN: track 51.8 -> 0.00 mm, vias 2 -> 0
- net /STM32/I2S_LRCK: track 50.7 -> 0.00 mm, vias 2 -> 0
- net /STM32/I2S_SCK: track 48.0 -> 0.00 mm, vias 2 -> 0
- net +3.3V: track 263.7 -> 220.0 mm, vias 11 -> 8
- net /STM32/LED_ENABLE: track 14.2 -> 42.6 mm, vias 0 -> 1
- net /CS4270/RST: track 0.00 -> 27.2 mm, vias 0 -> 2
- net /CS4270/SAI_SDIN: track 0.00 -> 27.0 mm, vias 0 -> 2
- net +12V: track 0.00 -> 26.9 mm, vias 0 -> 1
- net /CS4270/I2C_SDA: track 0.00 -> 26.8 mm, vias 0 -> 3
- net /STM32/BLEND: track 8.36 -> 32.4 mm
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Other:
- board text added: "3.3V"
- board text added: "3.3VA"
- board text added: "3V3"
- board text added: "Basilica"
- board text added: "Digital FX Processor"
- board text added: "LENIMAL PCB DESIGN 02.2025"
- board text added: "My Wife is the Best"
- board text added: "STM32 G474 RBTx"
- board text removed: "+3.3V"
- board text removed: "+3.3VA"
- board text removed: "12.288 MHZ"
- board text removed: "3.3V>3.3VA"
- board text removed: "8 MHZ"
- board text removed: "BOOT"
- board text removed: "BRAIN"
- board text removed: "LENIMAL PCB DESIGN - 01.2025"
- board text removed: "NRST"
- board text removed: "REV.2"
- board text removed: "RUN"
- board text removed: "STM32 F405 RGT6"
- board text removed: "WM8731"
- board text removed: "Weathering"
- board text removed: "cc-by-sa - Emilie Gillet [Mutable Instruments]"

Commit message: Setup of C code for Reverb
Parts:
- removed C21, C22: 10uF, Capacitor_SMD:C_0805_2012Metric_Pad1.18x1.45mm_HandSolder
- removed R6: 47K, Resistor_SMD:R_0805_2012Metric_Pad1.20x1.40mm_HandSolder
- removed U3: LM1117MP-5.0, Package_TO_SOT_SMD:SOT-223-3_TabPin2
Connections:
- C15 pad 1: +5VA -> +3.3VA
- C16 pad 1: +5VA -> +3.3VA
- J3 pad 4: +12V -> unconnected-(J3-Pin_4-Pad4)
- J3 pad 5: +12V -> unconnected-(J3-Pin_5-Pad5)
- U2 pad 19: +5VA -> +3.3VA
Routing:
- net +3.3VA: track 35.9 -> 127.6 mm, vias 2 -> 4
- net +5VA: track 78.2 -> 0.00 mm, vias 2 -> 0
- net +12V: track 26.9 -> 0.00 mm, vias 1 -> 0
- net /CS4270/SAI_SDOUT: track 22.1 -> 20.8 mm, vias 3 -> 2
- net /CS4270/I2C_SCL: track 22.2 -> 21.1 mm
- net GNDREF: vias 39 -> 32
Other:
- board text added: "CS4270"
