File: helpers/kiCad-templates/synth-module/Synth_Module.kicad_sch (KiCad schematic)
At the start: 37 parts, among them J1 INPUT, J2 OUTPUT, J3 PWR, U1 TL074

Commit message: Add: Quantizer init, Fix: Stereo-Delay, Fix: Midi-2-xc
Parts:
- removed C3, C4: 0.1uF, Capacitor_THT:CP_Radial_D4.0mm_P2.00mm, symbol Device:C_Polarized
- removed C5, C6: 0.1uF, Capacitor_THT:C_Rect_L4.6mm_W2.0mm_P2.50mm_MKS02_FKP02, symbol Device:C
- removed D1, D2: 1N5819, Synth:D_DO-41_SOD81_P10.16mm_Horizontal, symbol Diode:1N5819
- removed D3: LED, Synth:LED_D5.0mm (center Aligned), symbol synth:LED (5mm)
- removed H1: H1, Synth:PinHeader_1x04_P2.54mm_Vertical, symbol synth:PinHeader_01x04
- removed H10, H11, H12, H13, H14, H15, H16, H9: MountingHole, MountingHole:MountingHole_3.2mm_M3, symbol Mechanical:MountingHole
- removed H17: H17, Synth:PinHeader_1x08_P2.54mm_Vertical, symbol synth:PinHeader_01x08
- removed H18: H18, Synth:PinSocket_1x08_P2.54mm_Vertical, symbol synth:PinSocket_01x08
- removed H2: H3, Synth:PinSocket_1x04_P2.54mm_Vertical, symbol synth:PinSocket_01x04
- removed H3: H5, Synth:PinHeader_1x04_P2.54mm_Vertical, symbol synth:PinHeader_01x04
- removed H4: H6, Synth:PinSocket_1x04_P2.54mm_Vertical, symbol synth:PinSocket_01x04
- removed H5: H7, Synth:PinHeader_1x04_P2.54mm_Vertical, symbol synth:PinHeader_01x04
- removed H6: H8, Synth:PinSocket_1x04_P2.54mm_Vertical, symbol synth:PinSocket_01x04
- removed H7: H2, Synth:PinHeader_1x08_P2.54mm_Vertical, symbol synth:PinHeader_01x08
- removed H8: H4, Synth:PinSocket_1x08_P2.54mm_Vertical, symbol synth:PinSocket_01x08
- removed J1: INPUT, Synth:Jack_3.5mm_QingPu_WQP-PJ398SM_Vertical_CircularHoles, symbol synth:AudioJack_Mono_3.5mm
- removed J2: OUTPUT, Synth:Jack_3.5mm_QingPu_WQP-PJ398SM_Vertical_CircularHoles, symbol synth:AudioJack_Mono_3.5mm
- removed J3: PWR, Synth:IDC-Header_2x08_P2.54mm_Vertical, symbol synth:Conn_02x08_EuroRack_Power
- removed R3: 680R, Synth:R_Default (DIN0207), symbol synth:R_Default
- removed U1: TL074, Package_DIP:DIP-14_W7.62mm_Socket_LongPads, symbol Amplifier_Operational:TL074
- added C3, C4: 100nF, Capacitor_SMD:C_0805_2012Metric_Pad1.18x1.45mm_HandSolder, symbol Device:C
- added D3, D4: 1N5819WS, Diode_SMD:D_SOD-323_HandSoldering, symbol Diode:1N5819WS
- added H1: Conn_02x05_PWR_Eurorack, Synth:IDC-Header_2x05_P2.54mm_Vertical, symbol synth:Conn_02x05_EuroRack_Power
- R1, R2: footprint Synth:R_Default (DIN0207) -> Resistor_SMD:R_0805_2012Metric_Pad1.20x1.40mm_HandSolder
Connections:
- net +12V: now also C3.1
- net -12V: now also C4.2
- net GNDREF: now also C3.2, C4.1, H1.3 (Pin_3), H1.4 (Pin_4), H1.5 (Pin_5), H1.6 (Pin_6), H1.7 (Pin_7), H1.8 (Pin_8)
- net at R2.1: now also D4.2 (A)
- net at R1.1: now also D3.1 (K)
- new net: D4.1 (K), H1.1 (Pin_1), H1.2 (Pin_2)
- new net: D3.2 (A), H1.10 (Pin_10), H1.9 (Pin_9)
- no-connect marks 8 -> 0
Other:
- moved on the sheet: C1, C2, R1, R2, TP1, TP2, TP3
