File: modules/effects/stereo-delay/kiCad/input_stage.kicad_sch (KiCad schematic)
At the start: 10 parts, among them U3 TL074

Commit message: Add: Quantizer init, Fix: Stereo-Delay, Fix: Midi-2-xc
Parts:
- C32: renamed from C18; value 1nF -> 4.7nF
- renumbered C17 to C31, C19 to C33, R18 to R44, R20 to R46, R21 to R47
Changed lines of the file:
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@@
 	(text "This seems to be the most optimized solution, with an input of 16Vpp (+-8V)\n\nFinal Output Characteristics:\nVoltage: 1.46Vpp \nFrequency response:\nFull pass band: DC to 7.2 kHz\n-3dB point at 7.2 kHz\nRoll-off -20dB/decade from 7.2 kHz to 16 kHz\nRoll-off -40dB/decade above 16 kHz\nDC coupling removed by C29"
 		(exclude_from_sim no)
-		(at 230.886 106.68 0)
+		(at 224.282 91.186 0)
 		(effects
 			(font
@@
 	(text "This will control the gain, but the gain here is less than 1"
 		(exclude_from_sim no)
-		(at 181.356 107.442 0)
+		(at 181.356 90.424 0)
 		(effects
 			(font
@@
 		(shape input)
 		(at 139.7 119.38 180)
-		(fields_autoplaced yes)
 		(effects
 			(font
@@
 		(shape input)
 		(at 270.51 134.62 0)
-		(fields_autoplaced yes)
 		(effects
 			(font
@@
 		(shape input)
 		(at 139.7 134.62 180)
-		(fields_autoplaced yes)
 		(effects
 			(font
@@
 		(dnp no)
 		(fields_autoplaced yes)
-		(property "Reference" "R18"
+		(property "Reference" "R44"
 			(at 179.07 113.03 90)
 			(effects
@@
 		(dnp no)
 		(fields_autoplaced yes)
-		(property "Reference" "C17"
+		(property "Reference" "C31"
 			(at 244.729 127 90)
 			(effects
@@
 		(dnp no)
 		(fields_autoplaced yes)
-		(property "Reference" "C18"
+		(property "Reference" "C32"
 			(at 269.24 140.9699 0)
 			(effects
@@
 			)
 		)
-		(property "Value" "1nF"
+		(property "Value" "4.7nF"
 			(at 269.24 143.5099 0)
 			(effects
@@
 		(dnp no)
 		(fields_autoplaced yes)
-		(property "Reference" "R21"
+		(property "Reference" "R47"
 			(at 198.12 130.81 90)
 			(effects
@@
 		(dnp no)
 		(fields_autoplaced yes)
-		(property "Reference" "C19"
+		(property "Reference" "C33"
 			(at 205.74 144.7799 0)
 			(effects
@@
 		(dnp no)
 		(fields_autoplaced yes)
-		(property "Reference" "#PWR039"
+		(property "Reference" "#PWR057"
 			(at 201.93 156.21 0)
 			(effects
@@
 		(dnp no)
 		(fields_autoplaced yes)
-		(property "Reference" "R20"
+		(property "Reference" "R46"
 			(at 257.81 128.27 90)
 			(effects
@@
 		(dnp no)
 		(fields_autoplaced yes)
-		(property "Reference" "#PWR038"
+		(property "Reference" "#PWR056"
 			(at 265.43 152.4 0)
 			(effects
