File: modules/clones/wolkje/KiCad/inputs.kicad_sch (KiCad schematic)
At the start: 52 parts, among them J10 SIZE_IN, J11 BLEND_IN, J12 TEXTURE_IN, J5 FREEZE_IN, J6 V/OCT_IN, J7 POSITION_IN, J8 TRIGGER_IN, J9 DENSITY_IN, Q1 MMBT3904, Q2 MMBT3904, SW1 SW_ML6, SW2 SW_ML6, SW3 SW_RESEVERD, SW4 SW_MODE, U7 MCP6002, U8 MCP6004

Commit message: Update readme, get ready for third PCB run
Parts:
- R38: value 680R -> 2K
- SW1, SW2: symbol Library:SW_ML6 -> synth:SW_ML6
Connections:
- net BLEND_CV: now also U8.7; no longer U8.1
- net GNDREF: now also U8.10 (+), U8.3 (+), U8.5 (+); no longer U8.10 (+), U8.3 (+), U8.5 (+)
- net SIZE_CV: now also U8.1; no longer U8.8
- net TEXTURE_CV: now also U8.8; no longer U8.7
- net at C28.2, R39.2, R41.1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: now also U8.6 (-); no longer U8.2 (-)
- net at C29.2, R43.2, R44.1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: now also U8.9 (-); no longer U8.6 (-)
- net at C27.2, R33.2, R35.1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: now also U8.2 (-); no longer U8.9 (-)
Changed lines of the file:
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@@
 		(shape input)
 		(at 224.79 196.85 0)
-		(fields_autoplaced yes)
 		(effects
 			(font
@@
 		(shape output)
 		(at 384.81 160.02 0)
-		(fields_autoplaced yes)
 		(effects
 			(font
@@
 		(shape output)
 		(at 354.33 95.25 180)
-		(fields_autoplaced yes)
 		(effects
 			(font
@@
 		(shape input)
 		(at 114.3 101.6 0)
-		(fields_autoplaced yes)
 		(effects
 			(font
@@
 		(shape output)
 		(at 288.29 36.83 0)
-		(fields_autoplaced yes)
 		(effects
 			(font
@@
 		(shape input)
 		(at 114.3 50.8 0)
-		(fields_autoplaced yes)
 		(effects
 			(font
@@
 		(shape output)
 		(at 288.29 80.01 0)
-		(fields_autoplaced yes)
 		(effects
 			(font
@@
 		(shape output)
 		(at 388.62 31.75 0)
-		(fields_autoplaced yes)
 		(effects
 			(font
@@
 		(shape output)
 		(at 389.89 66.04 0)
-		(fields_autoplaced yes)
 		(effects
 			(font
@@
 		(shape output)
 		(at 354.33 125.73 180)
-		(fields_autoplaced yes)
 		(effects
 			(font
@@
 		(shape output)
 		(at 288.29 101.6 0)
-		(fields_autoplaced yes)
 		(effects
 			(font
@@
 		(shape input)
 		(at 355.6 107.95 180)
-		(fields_autoplaced yes)
 		(effects
 			(font
@@
 		(shape output)
 		(at 384.81 173.99 0)
-		(fields_autoplaced yes)
 		(effects
 			(font
@@
 		(shape input)
 		(at 228.6 152.4 0)
-		(fields_autoplaced yes)
 		(effects
 			(font
@@
 		(shape input)
 		(at 229.87 101.6 0)
-		(fields_autoplaced yes)
 		(effects
 			(font
@@
 		(shape output)
 		(at 288.29 58.42 0)
-		(fields_autoplaced yes)
 		(effects
 			(font
@@
 		(shape input)
 		(at 226.06 49.53 0)
-		(fields_autoplaced yes)
 		(effects
 			(font
@@
 		(at 204.47 152.4 0)
 		(mirror x)
-		(unit 1)
+		(unit 2)
 		(exclude_from_sim no)
 		(in_bom yes)
@@
 				(path "/ffcc7acb-943e-4c85-833d-d9691a289ebb/b8e374f8-4b03-4b6e-a5d5-fb7b54cd9525"
 					(reference "U8")
-					(unit 1)
+					(unit 2)
 				)
 			)
@@
 	)
 	(symbol
-		(lib_id "Library:SW_ML6")
+		(lib_id "synth:SW_ML6")
 		(at 379.73 105.41 0)
 		(unit 1)
@@
 		)
 		(property "Footprint" "Synth:ML6-H2T2GQA"
-			(at 379.73 95.25 0)
+			(at 379.476 117.602 0)
 			(effects
 				(font
@@
 			)
 		)
-		(property "Value" "680R"
+		(property "Value" "2K"
 			(at 363.22 104.14 90)
 			(effects
@@
 		(fields_autoplaced yes)
 		(property "Reference" "RV3"
-			(at 278.13 36.83 90)
+			(at 281.94 35.5599 0)
 			(effects
 				(font
 					(size 1.27 1.27)
 				)
+				(justify right)
 			)
 		)
 		(property "Value" "B10K"
-			(at 280.67 36.83 90)
+			(at 281.94 38.0999 0)
 			(effects
 				(font
 					(size 1.27 1.27)
 				)
+				(justify right)
 			)
 		)
@@
 		(fields_autoplaced yes)
 		(property "Reference" "RV7"
-			(at 278.13 101.6 90)
+			(at 281.94 100.3299 0)
 			(effects
 				(font
 					(size 1.27 1.27)
 				)
+				(justify right)
 			)
 		)
 		(property "Value" "B10K"
-			(at 280.67 101.6 90)
+			(at 281.94 102.8699 0)
 			(effects
 				(font
 					(size 1.27 1.27)
 				)
+				(justify right)
 			)
 		)
@@
 	)
 	(symbol
-		(lib_id "Library:SW_ML6")
+		(lib_id "synth:SW_ML6")
 		(at 379.73 135.89 0)
 		(unit 1)
@@
 		)
 		(property "Footprint" "Synth:ML6-H2T2GQA"
-			(at 379.73 125.73 0)
+			(at 379.476 148.082 0)
 			(effects
 				(font
@@
 					(size 1.27 1.27)
 				)
-				(hide yes)
 			)
 		)
@@
 					(size 1.27 1.27)
 				)
-				(hide yes)
 			)
 		)
@@
 		(fields_autoplaced yes)
 		(property "Reference" "RV4"
-			(at 278.13 58.42 90)
+			(at 281.94 57.1499 0)
 			(effects
 				(font
 					(size 1.27 1.27)
 				)
+				(justify right)
 			)
 		)
 		(property "Value" "B10K"
-			(at 280.67 58.42 90)
+			(at 281.94 59.6899 0)
 			(effects
 				(font
 					(size 1.27 1.27)
 				)
+				(justify right)
 			)
 		)
@@
 		(fields_autoplaced yes)
 		(property "Reference" "RV6"
-			(at 278.13 80.01 90)
+			(at 281.94 78.7399 0)
 			(effects
 				(font
 					(size 1.27 1.27)
 				)
+				(justify right)
 			)
 		)
 		(property "Value" "B10K"
-			(at 280.67 80.01 90)
+			(at 281.94 81.2799 0)
 			(effects
 				(font
 					(size 1.27 1.27)
 				)
+				(justify right)
 			)
 		)
@@
 		(at 203.2 196.85 0)
 		(mirror x)
-		(unit 2)
+		(unit 3)
 		(exclude_from_sim no)
 		(in_bom yes)
@@
 				(path "/ffcc7acb-943e-4c85-833d-d9691a289ebb/b8e374f8-4b03-4b6e-a5d5-fb7b54cd9525"
 					(reference "U8")
-					(unit 2)
+					(unit 3)
 				)
 			)
@@
 		(at 204.47 101.6 0)
 		(mirror x)
-		(unit 3)
+		(unit 1)
 		(exclude_from_sim no)
 		(in_bom yes)
@@
 				(path "/ffcc7acb-943e-4c85-833d-d9691a289ebb/b8e374f8-4b03-4b6e-a5d5-fb7b54cd9525"
 					(reference "U8")
-					(unit 3)
+					(unit 1)
 				)
 			)

Commit message: finished clouds clone (weathering/the storm)
Connections:
- net +3.3VA: now also RV3.3, RV4.3, RV6.3, RV7.3; no longer RV3.1, RV4.1, RV6.1, RV7.1
- net -10V: now also RV2.1, RV5.1; no longer RV2.3, RV5.3
- net GNDREF: now also RV2.3, RV3.1, RV4.1, RV5.3, RV6.1, RV7.1; no longer RV2.1, RV3.3, RV4.3, RV5.1, RV6.3, RV7.3
Other:
- moved on the sheet: RV2, RV5
Changed lines of the file:
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@@
 	(symbol
 		(lib_id "synth:R_Potentiometer (P0915N)")
-		(at 62.23 77.47 270)
+		(at 62.23 77.47 90)
+		(mirror x)
 		(unit 1)
 		(exclude_from_sim no)
@@
 		(on_board yes)
 		(dnp no)
-		(fields_autoplaced yes)
 		(property "Reference" "RV5"
 			(at 62.23 71.12 90)
@@
 		)
 		(property "Footprint" "Synth:Potentiometer_TT_P0915N"
-			(at 48.514 77.47 0)
+			(at 75.946 77.47 0)
 			(effects
 				(font
@@
 		)
 		(property "Datasheet" "~"
-			(at 51.562 77.47 0)
+			(at 72.898 77.47 0)
 			(effects
 				(font
@@
 		)
 		(property "Description" "Potentiometer"
-			(at 50.292 77.47 0)
+			(at 74.168 77.47 0)
 			(effects
 				(font
@@
 		(lib_id "synth:R_Potentiometer (P0915N)")
 		(at 284.48 36.83 0)
+		(mirror x)
 		(unit 1)
 		(exclude_from_sim no)
@@
 		(on_board yes)
 		(dnp no)
-		(fields_autoplaced yes)
 		(property "Reference" "RV3"
-			(at 281.94 35.5599 0)
+			(at 281.94 38.1001 0)
 			(effects
 				(font
@@
 		)
 		(property "Value" "B10K"
-			(at 281.94 38.0999 0)
+			(at 281.94 35.5601 0)
 			(effects
 				(font
@@
 		)
 		(property "Footprint" "Synth:Potentiometer_TT_P0915N"
-			(at 284.48 50.546 0)
+			(at 284.48 23.114 0)
 			(effects
 				(font
@@
 		)
 		(property "Datasheet" "~"
-			(at 284.48 47.498 0)
+			(at 284.48 26.162 0)
 			(effects
 				(font
@@
 		)
 		(property "Description" "Potentiometer"
-			(at 284.48 48.768 0)
+			(at 284.48 24.892 0)
 			(effects
 				(font
@@
 	(symbol
 		(lib_id "synth:R_Potentiometer (P0915N)")
-		(at 62.23 26.67 270)
+		(at 62.23 26.67 90)
+		(mirror x)
 		(unit 1)
 		(exclude_from_sim no)
@@
 		(on_board yes)
 		(dnp no)
-		(fields_autoplaced yes)
 		(property "Reference" "RV2"
 			(at 62.23 20.32 90)
@@
 		)
 		(property "Footprint" "Synth:Potentiometer_TT_P0915N"
-			(at 48.514 26.67 0)
+			(at 75.946 26.67 0)
 			(effects
 				(font
@@
 		)
 		(property "Datasheet" "~"
-			(at 51.562 26.67 0)
+			(at 72.898 26.67 0)
 			(effects
 				(font
@@
 		)
 		(property "Description" "Potentiometer"
-			(at 50.292 26.67 0)
+			(at 74.168 26.67 0)
 			(effects
 				(font
@@
 		(lib_id "synth:R_Potentiometer (P0915N)")
 		(at 284.48 101.6 0)
+		(mirror x)
 		(unit 1)
 		(exclude_from_sim no)
@@
 		(on_board yes)
 		(dnp no)
-		(fields_autoplaced yes)
 		(property "Reference" "RV7"
-			(at 281.94 100.3299 0)
+			(at 281.94 102.8701 0)
 			(effects
 				(font
@@
 		)
 		(property "Value" "B10K"
-			(at 281.94 102.8699 0)
+			(at 281.94 100.3301 0)
 			(effects
 				(font
@@
 		)
 		(property "Footprint" "Synth:Potentiometer_TT_P0915N"
-			(at 284.48 115.316 0)
+			(at 284.48 87.884 0)
 			(effects
 				(font
@@
 		)
 		(property "Datasheet" "~"
-			(at 284.48 112.268 0)
+			(at 284.48 90.932 0)
 			(effects
 				(font
@@
 		)
 		(property "Description" "Potentiometer"
-			(at 284.48 113.538 0)
+			(at 284.48 89.662 0)
 			(effects
 				(font
@@
 		(lib_id "synth:R_Potentiometer (P0915N)")
 		(at 284.48 58.42 0)
+		(mirror x)
 		(unit 1)
 		(exclude_from_sim no)
@@
 		(on_board yes)
 		(dnp no)
-		(fields_autoplaced yes)
 		(property "Reference" "RV4"
-			(at 281.94 57.1499 0)
+			(at 281.94 59.6901 0)
 			(effects
 				(font
@@
 		)
 		(property "Value" "B10K"
-			(at 281.94 59.6899 0)
+			(at 281.94 57.1501 0)
 			(effects
 				(font
@@
 		)
 		(property "Footprint" "Synth:Potentiometer_TT_P0915N"
-			(at 284.48 72.136 0)
+			(at 284.48 44.704 0)
 			(effects
 				(font
@@
 		)
 		(property "Datasheet" "~"
-			(at 284.48 69.088 0)
+			(at 284.48 47.752 0)
 			(effects
 				(font
@@
 		)
 		(property "Description" "Potentiometer"
-			(at 284.48 70.358 0)
+			(at 284.48 46.482 0)
 			(effects
 				(font
@@
 		(lib_id "synth:R_Potentiometer (P0915N)")
 		(at 284.48 80.01 0)
+		(mirror x)
 		(unit 1)
 		(exclude_from_sim no)
@@
 		(on_board yes)
 		(dnp no)
-		(fields_autoplaced yes)
 		(property "Reference" "RV6"
-			(at 281.94 78.7399 0)
+			(at 281.94 81.2801 0)
 			(effects
 				(font
@@
 		)
 		(property "Value" "B10K"
-			(at 281.94 81.2799 0)
+			(at 281.94 78.7401 0)
 			(effects
 				(font
@@
 		)
 		(property "Footprint" "Synth:Potentiometer_TT_P0915N"
-			(at 284.48 93.726 0)
+			(at 284.48 66.294 0)
 			(effects
 				(font
@@
 		)
 		(property "Datasheet" "~"
-			(at 284.48 90.678 0)
+			(at 284.48 69.342 0)
 			(effects
 				(font
@@
 		)
 		(property "Description" "Potentiometer"
-			(at 284.48 91.948 0)
+			(at 284.48 68.072 0)
 			(effects
 				(font
