File: modules/sequencers/1-sensei/kiCad/sensei.kicad_sch (KiCad schematic)
At the start: 77 parts, among them J1 CV OUT, J100 PWR, J2 CLK_IN, J3 CLK OUT, J4 GATE OUT, Q50 BC547, U1 TL074, U2 4017

Commit message: update sparkle pcb and schema
Parts:
- removed unit 7 of H8
- removed unit 6 of H8
- removed unit 7 of H9
- removed unit 6 of H9
- added unit 7 of H3
- added unit 6 of H3
- added unit 6 of H4
- added unit 7 of H4
- added J6: GATE_BUS_ENABLE, Connector_PinHeader_2.54mm:PinHeader_1x03_P2.54mm_Vertical, symbol Connector_Generic:Conn_01x03
- added J7: CV_BUS_ENABLE, Connector_PinHeader_2.54mm:PinHeader_1x03_P2.54mm_Vertical, symbol Connector_Generic:Conn_01x03
- added TP1, TP10, TP11, TP2, TP3, TP4, TP5, TP6, TP7, TP8, TP9: TestPoint, Connector_Pin:Pin_D1.0mm_L10.0mm, symbol Connector:TestPoint
- CV_LVL1, SW_CLK1: footprint synth-custom:SPDT_Toggle -> synth-custom:SW_default
- D1: renamed from D40; footprint Diode_THT:D_DO-35_SOD27_P7.62mm_Horizontal -> synth-custom:D_default
- D10: renamed from D5; footprint Diode_THT:D_DO-35_SOD27_P7.62mm_Horizontal -> synth-custom:D_default
- D11: renamed from D6; footprint Diode_THT:D_DO-35_SOD27_P7.62mm_Horizontal -> synth-custom:D_default
- D12: renamed from D7; footprint Diode_THT:D_DO-35_SOD27_P7.62mm_Horizontal -> synth-custom:D_default
- D13: renamed from D8; footprint Diode_THT:D_DO-35_SOD27_P7.62mm_Horizontal -> synth-custom:D_default
- D2: renamed from D41; footprint Diode_THT:D_DO-35_SOD27_P7.62mm_Horizontal -> synth-custom:D_default
- D3: renamed from D100; footprint Diode_THT:D_DO-35_SOD27_P7.62mm_Horizontal -> synth-custom:D_PWR_default
- D4: renamed from D200; footprint Diode_THT:D_DO-35_SOD27_P7.62mm_Horizontal -> synth-custom:D_PWR_default
- D5: renamed from D50; footprint Diode_THT:D_DO-35_SOD27_P7.62mm_Horizontal -> synth-custom:D_default
- D6: renamed from D1; footprint Diode_THT:D_DO-35_SOD27_P7.62mm_Horizontal -> synth-custom:D_default
- D7: renamed from D2; footprint Diode_THT:D_DO-35_SOD27_P7.62mm_Horizontal -> synth-custom:D_default
- D8: renamed from D3; footprint Diode_THT:D_DO-35_SOD27_P7.62mm_Horizontal -> synth-custom:D_default
- D9: renamed from D4; footprint Diode_THT:D_DO-35_SOD27_P7.62mm_Horizontal -> synth-custom:D_default
- H1: renamed from H12; footprint synth-custom:PinSocket_1x04_P2.00mm_Vertical -> synth-custom:PinSocket_1x04_P2.54mm_Vertical
- H10: renamed from H20; footprint MountingHole:MountingHole_3.5mm -> MountingHole:MountingHole_3.2mm_M3
- H11: renamed from H1; footprint MountingHole:MountingHole_3.5mm -> MountingHole:MountingHole_3.2mm_M3
- H12: renamed from H17; footprint MountingHole:MountingHole_3.5mm -> MountingHole:MountingHole_3.2mm_M3
- H13: renamed from H21; footprint MountingHole:MountingHole_3.5mm -> MountingHole:MountingHole_3.2mm_M3
- H14: renamed from H22; footprint MountingHole:MountingHole_3.5mm -> MountingHole:MountingHole_3.2mm_M3
- H15: renamed from H2; footprint MountingHole:MountingHole_3.5mm -> MountingHole:MountingHole_3.2mm_M3
- H16: renamed from H18; footprint MountingHole:MountingHole_3.5mm -> MountingHole:MountingHole_3.2mm_M3
- H17: renamed from H4; footprint synth-custom:PinHeader_1x08_P2.00mm_Vertical -> synth-custom:PinHeader_1x08_P2.54mm_Vertical
- H18: renamed from H3; footprint synth-custom:PinSocket_1x08_P2.00mm_Vertical -> synth-custom:PinSocket_1x08_P2.54mm_Vertical
- H2: renamed from H11; footprint synth-custom:PinHeader_1x04_P2.00mm_Vertical -> synth-custom:PinHeader_1x04_P2.54mm_Vertical
- H3: renamed from H8; footprint synth-custom:PinSocket_1x08_P2.00mm_Vertical -> synth-custom:PinSocket_1x08_P2.54mm_Vertical
- H4: renamed from H9; footprint synth-custom:PinHeader_1x08_P2.00mm_Vertical -> synth-custom:PinHeader_1x08_P2.54mm_Vertical
- H5: renamed from H16; footprint synth-custom:PinSocket_1x04_P2.00mm_Vertical -> synth-custom:PinSocket_1x04_P2.54mm_Vertical
- H6: renamed from H15; footprint synth-custom:PinSocket_1x04_P2.00mm_Vertical -> synth-custom:PinSocket_1x04_P2.54mm_Vertical
- H7: footprint synth-custom:PinHeader_1x04_P2.00mm_Vertical -> synth-custom:PinHeader_1x04_P2.54mm_Vertical
- H8: renamed from H6; footprint synth-custom:PinHeader_1x04_P2.00mm_Vertical -> synth-custom:PinHeader_1x04_P2.54mm_Vertical
- H9: renamed from H19; footprint MountingHole:MountingHole_3.5mm -> MountingHole:MountingHole_3.2mm_M3
- J1: renamed from J2; footprint synth-custom:Jack_3.5mm_QingPu_WQP-PJ398SM_Vertical_CircularHoles -> synth-custom:Jack_default; symbol Synth_Custom:AudioJack2_PJ398SM -> Synth_Custom:Jack_default
- J2: renamed from J3; footprint synth-custom:Jack_3.5mm_QingPu_WQP-PJ398SM_Vertical_CircularHoles -> synth-custom:Jack_default; symbol Synth_Custom:AudioJack2_PJ398SM -> Synth_Custom:Jack_default
- J3: renamed from J100; symbol Synth_Custom:Conn_02x08_PWR_Eurorack -> Synth_Custom:CONN_02x08_PWR_Eurorack
- J4: footprint synth-custom:Jack_3.5mm_QingPu_WQP-PJ398SM_Vertical_CircularHoles -> synth-custom:Jack_default; symbol Synth_Custom:AudioJack2_PJ398SM -> Synth_Custom:Jack_default
- J5: renamed from J1; footprint synth-custom:Jack_3.5mm_QingPu_WQP-PJ398SM_Vertical_CircularHoles -> synth-custom:Jack_default; symbol Synth_Custom:AudioJack2_PJ398SM -> Synth_Custom:Jack_default
- Q1: renamed from Q50; footprint Package_TO_SOT_THT:TO-92_Inline -> Package_TO_SOT_THT:TO-92_HandSolder
- R1: renamed from R7; footprint Resistor_THT:R_Axial_DIN0207_L6.3mm_D2.5mm_P10.16mm_Horizontal -> synth-custom:R_default
- R10: renamed from R200; footprint Resistor_THT:R_Axial_DIN0207_L6.3mm_D2.5mm_P10.16mm_Horizontal -> synth-custom:R_default
- R11: renamed from R53; footprint Resistor_THT:R_Axial_DIN0207_L6.3mm_D2.5mm_P10.16mm_Horizontal -> synth-custom:R_default
- R12: renamed from R54; footprint Resistor_THT:R_Axial_DIN0207_L6.3mm_D2.5mm_P10.16mm_Horizontal -> synth-custom:R_default
- R13: renamed from R1; footprint Resistor_THT:R_Axial_DIN0207_L6.3mm_D2.5mm_P10.16mm_Horizontal -> synth-custom:R_default
- R14: renamed from R6; footprint Resistor_THT:R_Axial_DIN0207_L6.3mm_D2.5mm_P10.16mm_Horizontal -> synth-custom:R_default
- R15: renamed from R4; footprint Resistor_THT:R_Axial_DIN0207_L6.3mm_D2.5mm_P10.16mm_Horizontal -> synth-custom:R_default
- R16: renamed from R3; footprint Resistor_THT:R_Axial_DIN0207_L6.3mm_D2.5mm_P10.16mm_Horizontal -> synth-custom:R_default
- R17: renamed from R2; footprint Resistor_THT:R_Axial_DIN0207_L6.3mm_D2.5mm_P10.16mm_Horizontal -> synth-custom:R_default
- R2: renamed from R8; footprint Resistor_THT:R_Axial_DIN0207_L6.3mm_D2.5mm_P10.16mm_Horizontal -> synth-custom:R_default
- R3: renamed from R9; footprint Resistor_THT:R_Axial_DIN0207_L6.3mm_D2.5mm_P10.16mm_Horizontal -> synth-custom:R_default
- R4: renamed from R40; footprint Resistor_THT:R_Axial_DIN0207_L6.3mm_D2.5mm_P10.16mm_Horizontal -> synth-custom:R_default
- R5: footprint Resistor_THT:R_Axial_DIN0207_L6.3mm_D2.5mm_P10.16mm_Horizontal -> synth-custom:R_default
- R6: renamed from R51; footprint Resistor_THT:R_Axial_DIN0207_L6.3mm_D2.5mm_P10.16mm_Horizontal -> synth-custom:R_default
- R7: renamed from R50; footprint Resistor_THT:R_Axial_DIN0207_L6.3mm_D2.5mm_P10.16mm_Horizontal -> synth-custom:R_default
- R8: renamed from R52; footprint Resistor_THT:R_Axial_DIN0207_L6.3mm_D2.5mm_P10.16mm_Horizontal -> synth-custom:R_default
- R9: renamed from R100; footprint Resistor_THT:R_Axial_DIN0207_L6.3mm_D2.5mm_P10.16mm_Horizontal -> synth-custom:R_default
- renumbered C103 to C2, C100 to C3, C200 to C4, C101 to C5, C201 to C6, C102 to C7, C202 to C8, RV9 to RV10, RV10 to RV9
Connections:
- net GNDD is gone; now on net GNDREF: C1.1, C2.2, C3.2, C4.1, C5.2, C6.1, C7.2, C8.1, H17.4, H17.5, H18.4, H18.5, J1.S, J2.S, J3.3 (GND), J3.4 (GND), J3.5 (GND), J3.6 (GND), J3.7 (GND), J3.8 (GND), J4.S, J5.S, R1.2, R11.1, R12.1, R4.1, R6.1, R7.1, RV1.3, RV10.2, RV10.3, RV2.3, RV3.3, RV4.3, RV5.3, RV6.3, RV7.3, RV8.3, RV9.2, RV9.3, U2.13 (CKEN), U2.8 (VSS)
- net +12V: now also TP9.1
- net -12V: now also TP11.1
- net at H1.1, H1.4, R3.1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: now also TP8.1
- net at J4.TN: now also H4.7
- net at H3.3, R14.1: now also TP2.1
- net at D5.1 (K), Q1.2 (B), R11.2: now also TP6.1
- net at D2.2 (A), H3.8, R7.2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: now also TP4.1
- net at D2.1 (K), R5.2, U1.6 (-)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: now also TP3.1
- net GNDREF: now reaches H18.8
- net GNDREF: now also H17.6, H17.8, H18.6, J6.1 (Pin_1), J7.1 (Pin_1), TP10.1
- net at U2.15 (Reset), U2.9 (Q8): now also TP5.1
- net at H3.2, R15.1: now also TP1.1
- net at J5.TN: now also H4.6
- net at D1.1 (K), R4.2, U1.5 (+): now also TP7.1
- net at J3.13 (CV): now also J3.14 (CV), J7.3 (Pin_3)
- net at J3.15 (GATE): now also J3.16 (GATE), J6.3 (Pin_3)
- new net: H3.7, J6.2 (Pin_2)
- new net: H3.6, J7.2 (Pin_2)
- no-connect marks 26 -> 12
Other:
- note added: "Clock System + Clock Input"
- note added: "Control Voltage Levels"
- note added: "Gate Out"
- note added: "Sequencer Clock System"
- note removed: "Clock System + Clock Input RESERVED 20-30 R20-30 RV20 C20 J20 CLK_input (output to other parts of the system"
- note removed: "Control Voltage Levels Reserved 1-10 RV1 - RV10 D1 - D10 R1 - R10 J1 - J10 SW1 - SW10"
- note removed: "Gate Out System Reserved 50-60 R50 - R60 D50 - D60 Q50 - Q60 J50 - J60"
- note removed: "Sequencer Clock System Reserved 40-50 R40 - R50 D40 - D50 J40 - J50"
- moved on the sheet: CV_LVL1, H10, H11, H12, H13, H14, H15, H16, H4A, H9

Commit message: update pcbs and symbols
Parts:
- CV_LVL1, SW_CLK1: footprint synth-custom:SW_default -> Synth:SW_default; symbol Synth_Custom:SW_SPDT -> synth:SW_SPDT
- D1, D10, D11, D12, D13, D2, D5, D6, D7, D8, D9: footprint synth-custom:D_default -> Synth:D_DO-35_SOD27_P7.62mm_Horizontal; symbol Diode:1N4148 -> synth:D_Signal (1N4148)
- D3, D4: footprint synth-custom:D_PWR_default -> Synth:D_DO-41_SOD81_P10.16mm_Horizontal; symbol Diode:1N5819 -> synth:D_Schottky (1N5819)
- H1, H5, H6: footprint synth-custom:PinSocket_1x04_P2.54mm_Vertical -> Synth:PinSocket_1x04_P2.54mm_Vertical; symbol Synth_Custom:CONN_Socket_01x04 -> synth:PinSocket_01x04
- H17, H4: footprint synth-custom:PinHeader_1x08_P2.54mm_Vertical -> Synth:PinHeader_1x08_P2.54mm_Vertical; symbol Synth_Custom:CONN_Header_01x08 -> synth:PinHeader_01x08
- H18, H3: footprint synth-custom:PinSocket_1x08_P2.54mm_Vertical -> Synth:PinSocket_1x08_P2.54mm_Vertical; symbol Synth_Custom:CONN_Socket_01x08 -> synth:PinSocket_01x08
- H2, H7, H8: footprint synth-custom:PinHeader_1x04_P2.54mm_Vertical -> Synth:PinHeader_1x04_P2.54mm_Vertical; symbol Synth_Custom:CONN_Header_01x04 -> synth:PinHeader_01x04
- J1, J2, J4, J5: footprint synth-custom:Jack_default -> Connector_Audio:Jack_3.5mm_QingPu_WQP-PJ398SM_Vertical_CircularHoles; symbol Synth_Custom:Jack_default -> synth:AudioJack_Mono_3.5mm
- J3: footprint synth-custom:CONN_02x08_PWR -> Synth:IDC-Header_2x08_P2.54mm_Vertical; symbol Synth_Custom:CONN_02x08_PWR_Eurorack -> synth:Conn_02x08_EuroRack_Power
- R1, R10, R11, R12, R13, R14, R15, R16, R17, R2, R3, R4, R5, R6, R7, R8, R9: footprint synth-custom:R_default -> Synth:R_Default (DIN0207); symbol Device:R -> synth:R_Default
Connections:
- net +12V: now also R8.2, R9.2; no longer R8.1, R9.1
- net -12V: now also R10.2; no longer R10.1
- net GNDREF: now also R1.1, R11.2, R12.2, R4.2, R6.2, R7.2; no longer R1.2, R11.1, R12.1, R4.1, R6.1, R7.1
- net at D10.1 (K), D11.1 (K), D12.1 (K)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: now also R13.2; no longer R13.1
- net at H3.2 (Pin_2), TP1.1: now also R15.2; no longer R15.1
- net at H1.1 (Pin_1), H1.4 (Pin_4), TP8.1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: now also R3.2; no longer R3.1
- net at H3.3 (Pin_3), TP2.1: now also R14.2; no longer R14.1
- net at U1.8, U1.9 (-): now also R15.1; no longer R15.2
- net at D5.1 (K), Q1.2 (B), TP6.1: now also R11.1; no longer R11.2
- net at R2.1: now also C1.2, U1.2 (-); no longer H1.2
- net at D2.2 (A), H3.8 (Pin_8), TP4.1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: now also R7.1; no longer R7.2
- net at D2.1 (K), TP3.1, U1.6 (-)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: now also R5.1; no longer R5.2
- net at H3.4 (Pin_4): now also R5.2; no longer R5.1
- net at H4.5 (Pin_5): now also R13.1; no longer R13.2
- net at D4.2 (A): now also R10.1; no longer R10.2
- net at D1.1 (K), TP7.1, U1.5 (+): now also R4.1; no longer R4.2
- net at D3.1 (K): now also R9.1; no longer R9.2
- net at CV_LVL1.1 (A): now also R16.1; no longer R16.2
- net at CV_LVL1.3 (C): now also R17.1; no longer R17.2
- net at RV9.1: now also R16.2; no longer R16.1
- net at RV10.1: now also R17.2; no longer R17.1
- new net: Q1.3 (E), R12.1, R14.1
- new net: H1.2 (Pin_2), R2.2
- new net: R6.1, R8.1, U1.13 (-)
- new net: R1.2, R3.1, U1.3 (+)
Other:
- moved on the sheet: J1, J2, J4, J5, J6, J7, TP1, TP2, TP3, TP4, TP6, TP7

Commit message: Sensei files & poem
Parts:
- added J8: CV_LVL_BTM, Synth:PinHeader_1x04_P2.54mm_Vertical, symbol synth:PinHeader_01x04
- added J9: CV_LVL_TOP, Synth:PinSocket_1x04_P2.54mm_Vertical, symbol synth:PinSocket_01x04
- C1: footprint Capacitor_THT:C_Rect_L7.2mm_W3.5mm_P5.00mm_FKS2_FKP2_MKS2_MKP2 -> Synth:C_RECT_MKT_1uF; symbol Device:C -> synth:C_1uF (MKS)
- CLK_SPD1, RV1, RV2, RV3, RV4, RV5, RV6, RV7, RV8: footprint Potentiometer_THT:Potentiometer_TT_P0915N -> Synth:Potentiometer_TT_P0915N; symbol Device:R_Potentiometer -> synth:R_Potentiometer (P0915N)
- J1, J2, J4, J5: footprint Connector_Audio:Jack_3.5mm_QingPu_WQP-PJ398SM_Vertical_CircularHoles -> Synth:Jack_3.5mm_QingPu_WQP-PJ398SM_Vertical_CircularHoles
Connections:
- net GNDREF: now also J8.3 (Pin_3), J8.4 (Pin_4), J9.3 (Pin_3), J9.4 (Pin_4)
- net at RV9.1: now also J8.2 (Pin_2); no longer R16.2
- net at RV10.1: now also J8.1 (Pin_1); no longer R17.2
- new net: J9.2 (Pin_2), R16.2
- new net: J9.1 (Pin_1), R17.2
Other:
- moved on the sheet: CV_LVL1, R16, R17, RV10, RV9

Commit message: add gerber files and ZIPs for V2
Parts:
- H10: renamed from J8; footprint Synth:PinHeader_1x04_P2.54mm_Vertical -> Synth:PinSocket_1x04_P2.54mm_Vertical; symbol synth:PinHeader_01x04 -> synth:PinSocket_01x04
- H9: renamed from J9; footprint Synth:PinSocket_1x04_P2.54mm_Vertical -> Synth:PinHeader_1x04_P2.54mm_Vertical; symbol synth:PinSocket_01x04 -> synth:PinHeader_01x04
- renumbered J8 to H10, J9 to H9, H9 to M1, H10 to M2, H11 to M3, H12 to M4, H13 to M5, H14 to M6, H15 to M7, H16 to M8
Other:
- moved on the sheet: H10C, H10D, H9A

Commit message: update to BOM and add panels
Parts:
- C1: value 0.1 uF -> 1uF
- C2, C7, C8: footprint Capacitor_THT:CP_Radial_D4.0mm_P2.00mm -> Capacitor_THT:C_Disc_D5.0mm_W2.5mm_P5.00mm; symbol Device:C_Polarized -> Device:C
- H1: value BTM_CLK -> PinSocket_1x04
- H10: value CV_LVL_BTM -> PinSocket_1x04
- H17: value TOP_PWR -> PinHeader_1x08
- H18: value BTM_PWR -> PinSocket_1x08
- H2: value TOP_CLK -> PinHeader_1x04
- H3: value BTM_CTRL -> PinSocket_1x08
- H4: value TOP_CTRL -> PinHeader_1x08
- H5: value BTM_SGL_RW_2 -> PinSocket_1x04
- H6: value BTM_SGL_RW_1 -> PinSocket_1x04
- H7: value TOP_SGL_RW_2 -> PinHeader_1x04
- H8: value TOP_SGL_RW_1 -> PinHeader_1x04
- H9: value CV_LVL_TOP -> PinHeader_1x04
- J6: value GATE_BUS_ENABLE -> PinHeader_1x03
- J7: value CV_BUS_ENABLE -> PinHeader_1x03
- M1, M2, M3, M4, M5, M6, M7, M8, TP1, TP10, TP11, TP2, TP3, TP4, TP5, TP6, TP7, TP8, TP9: now left out of the parts list
- R10, R9: value 10 -> 10R
- R14: value 200 -> 200R
- U2: value 4017 -> CD4017
Other:
- note removed: "I have 1uF here, and works pretty fine?"
- moved on the sheet: H2C, H2D, H4E, TP11, TP3, TP5
