File: modules/sequencers/1-sensei/kiCad/toggle_driver.kicad_sch (KiCad schematic)
At the start: 17 parts

Commit message: update sparkle pcb and schema
Parts:
- D22: renamed from D31; footprint Diode_THT:D_DO-35_SOD27_P7.62mm_Horizontal -> synth-custom:D_default
- D23: renamed from D32; footprint Diode_THT:D_DO-35_SOD27_P7.62mm_Horizontal -> synth-custom:D_default
- D24: renamed from D33; footprint Diode_THT:D_DO-35_SOD27_P7.62mm_Horizontal -> synth-custom:D_default
- D25: renamed from D34; footprint Diode_THT:D_DO-35_SOD27_P7.62mm_Horizontal -> synth-custom:D_default
- D26: renamed from D35; footprint Diode_THT:D_DO-35_SOD27_P7.62mm_Horizontal -> synth-custom:D_default
- D27: renamed from D36; footprint Diode_THT:D_DO-35_SOD27_P7.62mm_Horizontal -> synth-custom:D_default
- D28: renamed from D37; footprint Diode_THT:D_DO-35_SOD27_P7.62mm_Horizontal -> synth-custom:D_default
- D29: renamed from D38; footprint Diode_THT:D_DO-35_SOD27_P7.62mm_Horizontal -> synth-custom:D_default
- R27: renamed from R31; footprint Resistor_THT:R_Axial_DIN0207_L6.3mm_D2.5mm_P10.16mm_Horizontal -> synth-custom:R_default
- SW1: renamed from SW31; footprint synth-custom:SPDT_Toggle -> synth-custom:SW_default
- SW2: renamed from SW32; footprint synth-custom:SPDT_Toggle -> synth-custom:SW_default
- SW3: renamed from SW33; footprint synth-custom:SPDT_Toggle -> synth-custom:SW_default
- SW4: renamed from SW34; footprint synth-custom:SPDT_Toggle -> synth-custom:SW_default
- SW5: renamed from SW35; footprint synth-custom:SPDT_Toggle -> synth-custom:SW_default
- SW6: renamed from SW36; footprint synth-custom:SPDT_Toggle -> synth-custom:SW_default
- SW7: renamed from SW37; footprint synth-custom:SPDT_Toggle -> synth-custom:SW_default
- SW8: renamed from SW38; footprint synth-custom:SPDT_Toggle -> synth-custom:SW_default

Commit message: update pcbs and symbols
Parts:
- D22, D23, D24, D25, D26, D27, D28, D29: footprint synth-custom:D_default -> Synth:D_DO-35_SOD27_P7.62mm_Horizontal; symbol Diode:1N4148 -> synth:D_Signal (1N4148)
- R27: footprint synth-custom:R_default -> Synth:R_Default (DIN0207); symbol Device:R -> synth:R_Default
- SW1, SW2, SW3, SW4, SW5, SW6, SW7, SW8: footprint synth-custom:SW_default -> Synth:SW_default; symbol Synth_Custom:SW_SPDT -> synth:SW_SPDT
Connections:
- net SW_OUT: now also R27.1; no longer R27.2
- net at D22.1 (K), D23.1 (K), D24.1 (K)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: now also R27.2; no longer R27.1
