File: modules/utility/2-quantizer/kiCad/controls.kicad_sch (KiCad schematic)
At the start: 5 parts, among them SW1 CH_1_SW, SW2 CH_2_SW, SW3 ENCODER

Commit message: firmware for midas, quantizer updates
Parts:
- renumbered R43 to R10, R42 to R9, SW3 to SW2, SW2 to SW3
Changed lines of the file:
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@@
 		(dnp no)
 		(fields_autoplaced yes)
-		(property "Reference" "#PWR074"
+		(property "Reference" "#PWR053"
 			(at 184.15 85.09 0)
 			(effects
@@
 			(project "quantizer"
 				(path "/ffcc7acb-943e-4c85-833d-d9691a289ebb/6fd7f6d5-4064-4762-9c1a-399683bec6ab"
-					(reference "#PWR074")
+					(reference "#PWR053")
 					(unit 1)
 				)
@@
 		(dnp no)
 		(fields_autoplaced yes)
-		(property "Reference" "#PWR076"
+		(property "Reference" "#PWR050"
 			(at 247.65 44.45 0)
 			(effects
@@
 			(project "quantizer"
 				(path "/ffcc7acb-943e-4c85-833d-d9691a289ebb/6fd7f6d5-4064-4762-9c1a-399683bec6ab"
-					(reference "#PWR076")
+					(reference "#PWR050")
 					(unit 1)
 				)
@@
 		(dnp no)
 		(fields_autoplaced yes)
-		(property "Reference" "#PWR075"
+		(property "Reference" "#PWR052"
 			(at 228.6 59.69 0)
 			(effects
@@
 			(project "quantizer"
 				(path "/ffcc7acb-943e-4c85-833d-d9691a289ebb/6fd7f6d5-4064-4762-9c1a-399683bec6ab"
-					(reference "#PWR075")
+					(reference "#PWR052")
 					(unit 1)
 				)
@@
 		(dnp no)
 		(fields_autoplaced yes)
-		(property "Reference" "R43"
+		(property "Reference" "R10"
 			(at 161.29 72.39 90)
 			(effects
@@
 			(project "quantizer"
 				(path "/ffcc7acb-943e-4c85-833d-d9691a289ebb/6fd7f6d5-4064-4762-9c1a-399683bec6ab"
-					(reference "R43")
+					(reference "R10")
 					(unit 1)
 				)
@@
 		(dnp no)
 		(fields_autoplaced yes)
-		(property "Reference" "#PWR073"
+		(property "Reference" "#PWR051"
 			(at 184.15 53.34 0)
 			(effects
@@
 			(project "quantizer"
 				(path "/ffcc7acb-943e-4c85-833d-d9691a289ebb/6fd7f6d5-4064-4762-9c1a-399683bec6ab"
-					(reference "#PWR073")
+					(reference "#PWR051")
 					(unit 1)
 				)
@@
 		(dnp no)
 		(fields_autoplaced yes)
-		(property "Reference" "R42"
+		(property "Reference" "R9"
 			(at 161.29 40.64 90)
 			(effects
@@
 			(project "quantizer"
 				(path "/ffcc7acb-943e-4c85-833d-d9691a289ebb/6fd7f6d5-4064-4762-9c1a-399683bec6ab"
-					(reference "R42")
+					(reference "R9")
 					(unit 1)
 				)
@@
 		(dnp no)
 		(fields_autoplaced yes)
-		(property "Reference" "SW2"
+		(property "Reference" "SW3"
 			(at 176.53 55.88 0)
 			(effects
@@
 			(project "quantizer"
 				(path "/ffcc7acb-943e-4c85-833d-d9691a289ebb/6fd7f6d5-4064-4762-9c1a-399683bec6ab"
-					(reference "SW2")
+					(reference "SW3")
 					(unit 1)
 				)
@@
 		(dnp no)
 		(fields_autoplaced yes)
-		(property "Reference" "SW3"
+		(property "Reference" "SW2"
 			(at 218.44 45.72 0)
 			(effects
@@
 			(project ""
 				(path "/ffcc7acb-943e-4c85-833d-d9691a289ebb/6fd7f6d5-4064-4762-9c1a-399683bec6ab"
-					(reference "SW3")
-					(unit 1)
-				)
+					(reference "SW2")
+					(unit 1)
+				)

Commit message: quantizers_stls
Parts:
- added C25, C26, C27, C28: 100nF, Capacitor_SMD:C_0805_2012Metric_Pad1.18x1.45mm_HandSolder, symbol Device:C
- added R10, R12, R14, R16, R18, R20, R22, R24, R26, R28, R30, R32: 10K, Resistor_SMD:R_0805_2012Metric_Pad1.20x1.40mm_HandSolder, symbol Device:R
- added R13, R17, R19, R21, R23, R25, R27, R29, R31, R33: 470R, Resistor_SMD:R_0805_2012Metric_Pad1.20x1.40mm_HandSolder, symbol Device:R
- added SW10, SW2, SW5, SW6, SW9: CH_1_SW, Synth:ML6-H2T2GQA, symbol synth:SW_ML6
- added SW11, SW12, SW4, SW7, SW8: CH_2_SW, Synth:ML6-H2T2GQA, symbol synth:SW_ML6
- added SW13, SW15: SW_Push, Synth:SW_PUSH_6mm, symbol Switch:SW_Push
- added U10, U7: 74HC165, Synth:SOIC-16, symbol 74xx:74HC165
- added U8, U9: 74HC595, Synth:SOIC-16, symbol 74xx:74HC595
- renumbered R9 to R11, R10 to R15, SW2 to SW14
Connections:
- net LED_SW_2 is gone; now on net +3.3V: SW3.1, SW3.2
- net GNDREF: now also C25.2, C26.2, C27.2, C28.2, R10.1, R12.1, R14.1, R16.1, R18.1, R20.1, R22.1, R24.1, R26.1, R28.1, R30.1, R32.1, SW10.L2, SW11.L2, SW12.L2, SW13.1, SW15.1, SW2.L2, SW4.L2, SW5.L2, SW6.L2, SW7.L2, SW8.L2, SW9.L2, U10.15 (~{CE}), U10.8 (GND), U7.15 (~{CE}), U7.8 (GND), U8.13 (~{OE}), U8.8 (GND), U9.13 (~{OE}), U9.8 (GND); no longer SW1.3, SW1.4 (A), SW3.3, SW3.4 (A)
- net LED_1: no longer names the net of R11.1
- net LED_1: now also U8.1 (QB)
- net LED_2: no longer names the net of R15.1
- net LED_2: now also U8.3 (QD)
- net LED_SW_1 renamed +3.3V
- net +3.3V: now also C25.1, C26.1, C27.1, C28.1, SW10.1, SW10.2, SW11.1, SW11.2, SW12.1, SW12.2, SW2.1, SW2.2, SW4.1, SW4.2, SW5.1, SW5.2, SW6.1, SW6.2, SW7.1, SW7.2, SW8.1, SW8.2, SW9.1, SW9.2, U10.16 (VCC), U7.16 (VCC), U8.10 (~{SRCLR}), U8.16 (VCC), U9.10 (~{SRCLR}), U9.16 (VCC)
- new net: R10.2, SW1.3, SW1.4 (A), U7.11 (D0)
- new net: R12.2, SW2.3, SW2.4 (A), U7.12 (D1)
- new net: R14.2, SW3.3, SW3.4 (A), U7.13 (D2)
- new net: R16.2, SW4.3, SW4.4 (A), U7.14 (D3)
- new net: R18.2, SW5.3, SW5.4 (A), U7.3 (D4)
- new net: R20.2, SW6.3, SW6.4 (A), U7.4 (D5)
- new net: U10.10 (DS), U7.9 (Q7)
- new net: R19.2, SW5.L1
- new net: R30.2, SW11.3, SW11.4 (A), U10.3 (D4)
- new net: R31.2, SW11.L1
- new net: R17.1, U8.4 (QE)
- new net: R17.2, SW4.L1
- new net: R28.2, SW10.3, SW10.4 (A), U10.14 (D3)
- new net: R13.1, U8.2 (QC)
- new net: R13.2, SW2.L1
- new net: R19.1, U8.5 (QF)
- new net: R31.1, U9.5 (QF)
- new net: R21.1, U8.6 (QG)
- new net: U8.9 (QH'), U9.14 (SER)
- new net: R33.1, U9.6 (QG)
- new net: R33.2, SW12.L1
- new net: R24.2, SW8.3, SW8.4 (A), U10.12 (D1)
- new net: R25.2, SW8.L1
- new net: R27.1, U9.3 (QD)
- new net: R27.2, SW9.L1
- new net: R26.2, SW9.3, SW9.4 (A), U10.13 (D2)
- new net: R21.2, SW6.L1
- new net: R22.2, SW7.3, SW7.4 (A), U10.11 (D0)
- new net: R23.2, SW7.L1
- new net: R32.2, SW12.3, SW12.4 (A), U10.4 (D5)
- new net: R29.2, SW10.L1
- new net: R29.1, U9.4 (QE)
- new net: R23.1, U9.1 (QB)
- new net: R25.1, U9.2 (QC)
- new net LED_SCK: U8.11 (SRCLK), U9.11 (SRCLK)
- new net LED_SDIN: U8.14 (SER)
- new net LED_WRITE: U8.12 (RCLK), U9.12 (RCLK)
- new net SW_A: SW13.2
- new net SW_B: SW15.2
- new net SW_READ: U10.1 (~{PL}), U7.1 (~{PL})
- new net SW_SCK: U10.2 (CP), U7.2 (CP)
- new net SW_SDOUT: U10.9 (Q7)
- no-connect marks 0 -> 12
Other:
- moved on the sheet: R11, R15, SW1, SW14, SW3
