File: modules/utility/2-quantizer/kiCad/power.kicad_sch (KiCad schematic)
At the start: 27 parts, among them U1 TL072, U10 LM1117DT-3.3, U11 LM4040DBZ-2.5, U2 MCP6002, U4 OPA2277

Commit message: firmware for midas, quantizer updates
Parts:
- H1: value Conn_02x05_PWR_Eurorack -> POWER_CONN; footprint Connector_PinSocket_2.54mm:PinSocket_2x05_P2.54mm_Vertical -> Synth:IDC-Header_2x05_P2.54mm_Vertical
- renumbered C21 to C13, C22 to C14, C17 to C15, C18 to C16, C19 to C17, C23 to C18, C24 to C19, C25 to C21, C26 to C22, C27 to C23, R38 to R5, R39 to R6, R40 to R7, R41 to R8, U10 to U4, U1 to U5, U4 to U6, U2 to U7, U11 to U8

Commit message: quantizers_stls
Parts:
- added C21: 100nF, Capacitor_SMD:C_0805_2012Metric_Pad1.18x1.45mm_HandSolder, symbol Device:C
- added XP10, XP11, XP13, XP16, XP4, XP5, XP7: Conn_01x04_Pin, Connector_PinHeader_2.54mm:PinHeader_1x04_P2.54mm_Vertical, symbol synth:Conn_01x04_Pin
- added XP12, XP14, XP15, XP3, XP6, XP8, XP9: Conn_01x04_Socket, Connector_PinSocket_2.54mm:PinSocket_1x04_P2.54mm_Vertical, symbol synth:Conn_01x04_Socket
- renumbered C21 to C22, C22 to C23, C23 to C24, R5 to R6, R6 to R7, R7 to R8, R8 to R9, U4 to U2, U5 to U3, U6 to U4, U7 to U5, U8 to U6
Connections:
- net +12V: now also XP13.1 (Pin_1), XP13.2 (Pin_2); no longer C15.1, U3.8 (V+)
- net +3.3V: now also XP16.1 (Pin_1), XP16.2 (Pin_2), XP4.2 (Pin_2), XP4.3 (Pin_3); no longer C17.1, R7.2, U5.8 (V+)
- net -12V: now also U4.4 (V-), C21.2, XP16.3 (Pin_3); no longer C20.2, U3.4 (V-)
- net GNDREF: now also C21.1, XP10.4 (Pin_4), XP11.4 (Pin_4), XP13.3 (Pin_3), XP13.4 (Pin_4), XP16.4 (Pin_4), XP4.4 (Pin_4), XP5.4 (Pin_4), XP7.4 (Pin_4); no longer C15.2, C17.2, C20.1, C24.2, U4.4 (V-), U5.4 (V-), U6.2 (A)
- new net +12VB: C15.1, U3.8 (V+), XP14.1 (Pin_1), XP14.2 (Pin_2)
- new net +3.3VB: C17.1, R7.2, U5.8 (V+), XP15.1 (Pin_1), XP15.2 (Pin_2), XP3.2 (Pin_2), XP3.3 (Pin_3)
- new net -12VB: C20.2, U3.4 (V-), XP15.3 (Pin_3)
- new net GND: C15.2, C17.2, C20.1, C24.2, U5.4 (V-), U6.2 (A), XP12.4 (Pin_4), XP14.3 (Pin_3), XP14.4 (Pin_4), XP15.4 (Pin_4), XP3.4 (Pin_4), XP6.4 (Pin_4), XP8.4 (Pin_4), XP9.4 (Pin_4)
Other:
- note added: "Maybe requires a dedicated LDO regulator to decouple it from the STM power supply?"
- moved on the sheet: C16
