File: modules/utility/2-quantizer/kiCad/quantizer.kicad_pcb (KiCad board)
At the start: 6 copper layers, 30 x 110 mm, 98 parts, among them J1 CV_INPUT, J2 CV_OUTPUT, J3 CV_INPUT, J4 CV_OUTPUT, J5 BOOT_RUN, J6 RX/TX, J7 Conn_01x04, Q1 MMBT3904, Q2 MMBT3904, SW1 CH_1_SW, SW2 CH_2_SW, SW3 ENCODER, U1 TL072, U10 LM1117DT-3.3, U11 LM4040DBZ-2.5, U2 MCP6002, U3 MCP47256, U4 OPA2277, U5 MCP47256, U6 STM32F411RETx, U7 74HC595, U8 dual_segment_display, U9 74HC595

Commit message: firmware for midas, quantizer updates
Parts:
- removed C26: 100nF, Capacitor_SMD:C_0805_2012Metric_Pad1.18x1.45mm_HandSolder
- removed C27: 470nF, Capacitor_SMD:C_0805_2012Metric_Pad1.18x1.45mm_HandSolder
- removed U11: LM4040DBZ-2.5, Package_TO_SOT_SMD:SOT-23
- added C12: 100nF, Capacitor_SMD:C_0805_2012Metric_Pad1.18x1.45mm_HandSolder, B.Cu at (95.4, 99.6)
- added C13: 47uF, Capacitor_THT:CP_Radial_D6.3mm_P2.50mm, B.Cu at (65.0, 53.5)
- added D4: 1N4148WS, Diode_SMD:D_SOD-323_HandSoldering, B.Cu at (99.6, 135.9)
- added D5: 1N4148WS, Diode_SMD:D_SOD-323_HandSoldering, B.Cu at (89.5, 141.5)
- added J8: CV_INPUT, Synth:Jack_3.5mm_QingPu_WQP-PJ398SM_Vertical_CircularHoles, F.Cu at (86.0, 137.6)
- added J9: CV_OUTPUT, Synth:Jack_3.5mm_QingPu_WQP-PJ398SM_Vertical_CircularHoles, F.Cu at (86.0, 152.5)
- added Q3: MMBT3904, Package_TO_SOT_SMD:SOT-23, B.Cu at (99.6, 140.9)
- added Q4: MMBT3904, Package_TO_SOT_SMD:SOT-23, B.Cu at (89.5, 136.5)
- added R35: 30K [0.1%], Resistor_SMD:R_0805_2012Metric_Pad1.20x1.40mm_HandSolder, B.Cu at (93.0, 146.7)
- added R44: 1K, Resistor_SMD:R_0805_2012Metric_Pad1.20x1.40mm_HandSolder, B.Cu at (87.0, 155.0)
- added R45: 3K3, Resistor_SMD:R_0805_2012Metric_Pad1.20x1.40mm_HandSolder, B.Cu at (167.5, 109.0)
- added R46: 3K3, Resistor_SMD:R_0805_2012Metric_Pad1.20x1.40mm_HandSolder, B.Cu at (167.5, 112.0)
- added R47: 30K [0.1%], Resistor_SMD:R_0805_2012Metric_Pad1.20x1.40mm_HandSolder, B.Cu at (95.0, 156.2)
- added R48: 10K [0.1%], Resistor_SMD:R_0805_2012Metric_Pad1.20x1.40mm_HandSolder, B.Cu at (98.0, 157.5)
- added U13: MCP47256, Package_TO_SOT_SMD:SOT-23-6_Handsoldering, B.Cu at (178.0, 122.5)
- C10: value 1uF -> 2.2uF
- C11: value 1uF -> 100nF
- C14: value 2.2uF -> 100nF
- C18, C19: value 100nF -> 10uF; footprint Capacitor_SMD:C_0805_2012Metric_Pad1.18x1.45mm_HandSolder -> Capacitor_THT:CP_Radial_D4.0mm_P2.00mm; moved to F.Cu
- C22, D1, D3: moved to B.Cu
- C23: value 10uF -> 470nF; footprint Capacitor_THT:CP_Radial_D4.0mm_P2.00mm -> Capacitor_SMD:C_0805_2012Metric_Pad1.18x1.45mm_HandSolder
- C24: value 10uF -> 100nF; footprint Capacitor_THT:CP_Radial_D4.0mm_P2.00mm -> Capacitor_SMD:C_0805_2012Metric_Pad1.18x1.45mm_HandSolder
- C25: value 47uF -> 100nF; footprint Capacitor_THT:CP_Radial_D6.3mm_P2.50mm -> Capacitor_SMD:C_0805_2012Metric_Pad1.18x1.45mm_HandSolder
- C5: value 100nF -> 10uF
- C7: value 10uF -> 100nF
- C8, C9: value 100nF -> 1uF
- H1: value Conn_02x05_PWR_Eurorack -> POWER_CONN; footprint Connector_PinSocket_2.54mm:PinSocket_2x05_P2.54mm_Vertical -> Synth:IDC-Header_2x05_P2.54mm_Vertical
- J1: value CV_INPUT -> BOOT_RUN; footprint Synth:Jack_3.5mm_QingPu_WQP-PJ398SM_Vertical_CircularHoles -> Connector_PinHeader_2.54mm:PinHeader_1x03_P2.54mm_Vertical; moved to B.Cu
- J2: value CV_OUTPUT -> RX/TX; footprint Synth:Jack_3.5mm_QingPu_WQP-PJ398SM_Vertical_CircularHoles -> Connector_PinHeader_2.54mm:PinHeader_1x03_P2.54mm_Vertical; moved to B.Cu
- J3: value CV_INPUT -> Conn_01x04; footprint Synth:Jack_3.5mm_QingPu_WQP-PJ398SM_Vertical_CircularHoles -> Connector_PinHeader_2.54mm:PinHeader_1x04_P2.54mm_Vertical; moved to B.Cu
- J4: value CV_OUTPUT -> CV_INPUT
- J5: value BOOT_RUN -> CV_INPUT; footprint Connector_PinHeader_2.54mm:PinHeader_1x03_P2.54mm_Vertical -> Synth:Jack_3.5mm_QingPu_WQP-PJ398SM_Vertical_CircularHoles; moved to F.Cu
- J6: value RX/TX -> CV_OUTPUT; footprint Connector_PinHeader_2.54mm:PinHeader_1x03_P2.54mm_Vertical -> Synth:Jack_3.5mm_QingPu_WQP-PJ398SM_Vertical_CircularHoles; moved to F.Cu
- J7: value Conn_01x04 -> CV_INPUT; footprint Connector_PinHeader_2.54mm:PinHeader_1x04_P2.54mm_Vertical -> Synth:Jack_3.5mm_QingPu_WQP-PJ398SM_Vertical_CircularHoles; moved to F.Cu
- R1, R2: value 22K -> 10K
- R10, R9: value 22K -> 470R
- R11, R18: value 10K [0.1%] -> 100R
- R12: value 120K -> 100R
- R13: value 22K -> 100R
- R14: value 1K -> 100R
- R15, R16: value 3K3 -> 100R
- R17: value 30K [0.1%] -> 100R
- R19, R20: value 10K -> 100R
- R25, R26: value 100R -> 10K
- R27: value 100R -> 100K
- R28, R29, R31: value 100R -> 22K
- R3: value 120K -> 1K
- R30: value 100R -> 120K
- R32: value 100R -> 1K
- R33, R34: value 100R -> 3K3
- R36: value 1K -> 10K [0.1%]
- R37: value 1K -> 22K
- R38: value 10R -> 22K; moved to B.Cu
- R39: value 1K -> 120K
- R4: value 22K -> 1K
- R40: value 2K -> 22K
- R41: value 10R -> 10K; moved to B.Cu
- R42: value 470R -> 10K
- R43: value 470R -> 100K
- R5: value 1K -> 10R
- R6: value 3K3 -> 1K
- R7: value 3K3 -> 2K
- R8: value 30K [0.1%] -> 10R
- SW2: value CH_2_SW -> ENCODER; footprint Synth:ML6-H2T2GQA -> Synth:RotaryEncoder_Alps_EC11E-Switch_Vertical_H20mm_CircularMountingHoles
- SW3: value ENCODER -> CH_2_SW; footprint Synth:RotaryEncoder_Alps_EC11E-Switch_Vertical_H20mm_CircularMountingHoles -> Synth:ML6-H2T2GQA
- U1: value TL072 -> STM32F411RETx; footprint Synth:SOIC-8 -> Package_QFP:LQFP-64_10x10mm_P0.5mm
- U10: value LM1117DT-3.3 -> MCP47256; footprint Package_TO_SOT_SMD:TO-252-3_TabPin2 -> Package_TO_SOT_SMD:SOT-23-6_Handsoldering
- U2: value MCP6002 -> 74HC595; footprint Synth:SOIC-8 -> Synth:SOIC-16
- U3: value MCP47256 -> 74HC595; footprint Package_TO_SOT_SMD:SOT-23-6_Handsoldering -> Synth:SOIC-16
- U4: value OPA2277 -> LM1117DT-3.3; footprint Synth:SOIC-8 -> Package_TO_SOT_SMD:TO-252-3_TabPin2; moved to F.Cu
- U5: value MCP47256 -> TL072; footprint Package_TO_SOT_SMD:SOT-23-6_Handsoldering -> Synth:SOIC-8
- U6: value STM32F411RETx -> OPA2277; footprint Package_QFP:LQFP-64_10x10mm_P0.5mm -> Synth:SOIC-8
- U7: value 74HC595 -> MCP6002; footprint Synth:SOIC-16 -> Synth:SOIC-8
- U8: value dual_segment_display -> LM4040DBZ-2.5; footprint Synth:7-segment-display_DA56 -> Package_TO_SOT_SMD:SOT-23; moved to B.Cu
- U9: value 74HC595 -> dual_segment_display; footprint Synth:SOIC-16 -> Synth:7-segment-display_DA56; moved to F.Cu
- moved C17 137.6 mm to (158.5, 61.0), turned to 180 degrees
- moved C20 133.2 mm to (158.5, 64.0), turned to 180 degrees
- moved R39 129.3 mm to (187.8, 106.0)
- moved R9 113.0 mm to (162.1, 98.2), turned to 180 degrees
- moved R5 110.8 mm to (158.5, 73.0), turned to 180 degrees
- moved C15 110.1 mm to (158.5, 55.0), turned to 180 degrees
- moved C14 109.3 mm to (158.5, 52.0), turned to 180 degrees
- moved R10 107.9 mm to (162.1, 101.1), turned to 180 degrees
- moved C25 106.2 mm to (172.7, 121.5), turned to 180 degrees
- moved C16 104.3 mm to (91.0, 153.2), turned to 90 degrees
- moved R8 104.1 mm to (158.5, 81.8), turned to 180 degrees
- moved C24 97.8 mm to (151.0, 118.7)
- moved R6 97.5 mm to (158.5, 76.0), turned to 180 degrees
- moved R12 97.1 mm to (120.8, 71.0)
- moved R7 97.0 mm to (158.5, 78.9), turned to 180 degrees
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Connections:
- C10 pad 1: GNDREF -> /stm32F411/VCap
- C10 pad 2: +3.3VA -> GNDREF
- C11 pad 1: GNDREF -> +3.3V
- C11 pad 2: +3.3V -> GNDREF
- C14 pad 1: /stm32F411/VCap -> +12V
- C15 pad 1: +3.3V -> +12V
- C16 pad 1: +3.3V -> +12V
- C17 pad 1: +12V -> +3.3V
- C21 pad 1: +12V -> GNDREF
- C21 pad 2: GNDREF -> -12V
- C22 pad 1: +12V -> GNDREF
- C22 pad 2: GNDREF -> -12V
- C23 pad 1: +12V -> VREF__2_5V
- C24 pad 1: +3.3V -> GNDREF
- C24 pad 2: GNDREF -> +3.3V
- C25 pad 2: -12V -> +3.3V
- C6 pad 1: GNDREF -> /stm32F411/NRST
- C6 pad 2: +3.3V -> GNDREF
- C7 pad 2: +3.3V -> +3.3VA
- C8 pad 1: /stm32F411/NRST -> GNDREF
- C8 pad 2: GNDREF -> +3.3VA
- C9 pad 2: +3.3VA -> +3.3V
- J4 pad TN: unconnected-(J4-PadTN) -> Net-(J4-PadTN)
- R1 pad 1: Net-(R1-Pad1) -> /stm32F411/NRST
- R1 pad 2: Net-(U1A-+) -> +3.3V
- R10 pad 1: /stm32F411/ADC_2 -> /controls/LED_2
- R10 pad 2: Net-(U2B--) -> Net-(R10-Pad2)
- R11 pad 1: GNDREF -> Net-(U9-A)
- R11 pad 2: Net-(U4A--) -> /display/segment_display/A_12
- R12 pad 1: Net-(U1B-+) -> Net-(U9-B)
- R12 pad 2: Net-(J3-PadT) -> /display/segment_display/B_10
- R13 pad 1: Net-(U2B--) -> Net-(U9-C)
- R13 pad 2: Net-(R13-Pad2) -> /display/segment_display/C_9
- R14 pad 1: Net-(R14-Pad1) -> Net-(U9-D)
- R14 pad 2: Net-(J4-PadT) -> /display/segment_display/D_7
- R15 pad 1: /stm32F411/I2C2_SCL -> Net-(U9-E)
- R15 pad 2: +3.3V -> /display/segment_display/E_1
- R16 pad 1: /stm32F411/I2C2_SDA -> Net-(U9-F)
- R16 pad 2: +3.3V -> /display/segment_display/F_18
- R17 pad 1: Net-(U4B--) -> Net-(U9-G)
- R17 pad 2: Net-(R14-Pad1) -> /display/segment_display/G_17
- R18 pad 1: GNDREF -> Net-(U9-H)
- R18 pad 2: Net-(U4B--) -> /display/segment_display/H_15
- R19 pad 1: /stm32F411/NRST -> Net-(U9-J)
- R19 pad 2: +3.3V -> /display/segment_display/J_14
- R2 pad 1: /stm32F411/ADC_1 -> /stm32F411/BOOT0
- R2 pad 2: Net-(U2A--) -> /stm32F411/BOOT0_MCU
- R20 pad 1: /stm32F411/BOOT0 -> Net-(U9-K)
- R20 pad 2: /stm32F411/BOOT0_MCU -> /display/segment_display/K_6
- R21 pad 1: Net-(U8-A) -> Net-(U9-L)
- R21 pad 2: /display/segment_display/A_12 -> /display/segment_display/L_5
- R22 pad 1: Net-(U8-B) -> Net-(U9-M)
- R22 pad 2: /display/segment_display/B_10 -> /display/segment_display/M_4
- R23 pad 1: Net-(U8-C) -> Net-(U9-N)
- R23 pad 2: /display/segment_display/C_9 -> /display/segment_display/N_2
- R24 pad 1: Net-(U8-D) -> Net-(U9-P)
- R24 pad 2: /display/segment_display/D_7 -> /display/segment_display/P_13
- R25 pad 1: Net-(U8-E) -> /stm32F411/TRIG_1_EN
- R25 pad 2: /display/segment_display/E_1 -> Net-(J4-PadTN)
- R26 pad 1: Net-(U8-F) -> Net-(D4-K)
- R26 pad 2: /display/segment_display/F_18 -> Net-(J4-PadT)
- R27 pad 1: Net-(U8-G) -> Net-(D4-K)
- R27 pad 2: /display/segment_display/G_17 -> GNDREF
- R28 pad 1: Net-(U8-H) -> Net-(R28-Pad1)
- R28 pad 2: /display/segment_display/H_15 -> Net-(U5A-+)
- R29 pad 1: Net-(U8-J) -> /cv_input/CV_OUT
- R29 pad 2: /display/segment_display/J_14 -> Net-(U7A--)
- R3 pad 1: Net-(U1A-+) -> Net-(Q1-B)
- R3 pad 2: Net-(J1-PadT) -> /display/DISPLAY_CHAR_1
- R30 pad 1: Net-(U8-K) -> Net-(U5A-+)
- R30 pad 2: /display/segment_display/K_6 -> Net-(J5-PadT)
- R31 pad 1: Net-(U8-L) -> Net-(U7A--)
- R31 pad 2: /display/segment_display/L_5 -> Net-(R28-Pad1)
- R32 pad 1: Net-(U8-M) -> Net-(R32-Pad1)
- R32 pad 2: /display/segment_display/M_4 -> Net-(J6-PadT)
- R33 pad 1: Net-(U8-N) -> /cv_output/SCL_IN
- R33 pad 2: /display/segment_display/N_2 -> +3.3V
- R34 pad 1: Net-(U8-P) -> /cv_output/SDA_IN
- R34 pad 2: /display/segment_display/P_13 -> +3.3V
- R36 pad 1: Net-(Q1-B) -> GNDREF
- R36 pad 2: /display/DISPLAY_CHAR_1 -> Net-(U6A--)
- R37 pad 1: Net-(Q2-B) -> Net-(R37-Pad1)
- R37 pad 2: /display/DISPLAY_CHAR_2 -> Net-(U5B-+)
- R38 pad 1: Net-(D1-K) -> /cv_input1/CV_OUT
- R38 pad 2: +12V -> Net-(U7B--)
- R39 pad 1: VREF__2_5V -> Net-(U5B-+)
- R39 pad 2: +3.3V -> Net-(J7-PadT)
- R4 pad 1: Net-(U2A--) -> Net-(Q2-B)
- R4 pad 2: Net-(R1-Pad1) -> /display/DISPLAY_CHAR_2
- R40 pad 1: GNDREF -> Net-(U7B--)
- R40 pad 2: Net-(D2-K) -> Net-(R37-Pad1)
- R41 pad 1: Net-(D3-A) -> /stm32F411/TRIG_2_EN
- R41 pad 2: -12V -> Net-(J8-PadTN)
- R42 pad 1: /controls/LED_1 -> Net-(D5-K)
- R42 pad 2: Net-(R42-Pad2) -> Net-(J8-PadT)
- R43 pad 1: /controls/LED_2 -> Net-(D5-K)
- R43 pad 2: Net-(R43-Pad2) -> GNDREF
- R5 pad 1: Net-(R5-Pad1) -> Net-(D1-K)
- R5 pad 2: Net-(J2-PadT) -> +12V
- R6 pad 1: /stm32F411/I2C1_SCL -> VREF__2_5V
- R7 pad 1: /stm32F411/I2C1_SDA -> GNDREF
- R7 pad 2: +3.3V -> Net-(D2-K)
- R8 pad 1: Net-(U4A--) -> Net-(D3-A)
- R8 pad 2: Net-(R5-Pad1) -> -12V
- R9 pad 1: Net-(R13-Pad2) -> /controls/LED_1
- R9 pad 2: Net-(U1B-+) -> Net-(R9-Pad2)
- SW1 pad L1: Net-(R42-Pad2) -> Net-(R9-Pad2)
- U1 pad 1: Net-(R1-Pad1) -> +3.3V
- U1 pad 2: GNDREF -> unconnected-(U1-PC13-Pad2)
- U1 pad 3: Net-(U1A-+) -> /stm32F411/TRIG_1_IN
- U1 pad 4: -12V -> /stm32F411/TRIG_2_IN
- U1 pad 5: Net-(U1B-+) -> unconnected-(U1-PH0-Pad5)
- U1 pad 6: GNDREF -> unconnected-(U1-PH1-Pad6)
- U1 pad 7: Net-(R13-Pad2) -> /stm32F411/NRST
- U1 pad 8: +12V -> /stm32F411/TRIG_1_EN
- U10 pad 1: GNDREF -> Net-(U10-VOUT)
- U10 pad 2: +3.3V -> GNDREF
- U10 pad 3: +12V -> +3.3V
- U2 pad 1: /stm32F411/ADC_1 -> /display/segment_display/E_1
- U2 pad 2: Net-(U2A--) -> /display/segment_display/N_2
- U2 pad 3: GNDREF -> /display/segment_display/M_4
- U2 pad 4: GNDREF -> /display/segment_display/L_5
- U2 pad 5: GNDREF -> /display/segment_display/K_6
- U2 pad 6: Net-(U2B--) -> /display/segment_display/D_7
- U2 pad 7: /stm32F411/ADC_2 -> /display/segment_display/C_9
- U2 pad 8: +3.3V -> GNDREF
- U3 pad 1: Net-(U3-VOUT) -> /display/segment_display/B_10
- U3 pad 2: GNDREF -> /display/segment_display/A_12
- U3 pad 3: +3.3V -> /display/segment_display/P_13
- U3 pad 4: /stm32F411/I2C1_SDA -> /display/segment_display/J_14
- U3 pad 5: /stm32F411/I2C1_SCL -> /display/segment_display/H_15
- U3 pad 6: VREF__2_5V -> /display/segment_display/G_17
- U4 pad 1: Net-(R5-Pad1) -> GNDREF
- U4 pad 2: Net-(U4A--) -> +3.3V
- U4 pad 3: Net-(U3-VOUT) -> +12V
- U5 pad 1: Net-(U4B-+) -> Net-(R28-Pad1)
- U5 pad 3: +3.3V -> Net-(U5A-+)
- U5 pad 4: /stm32F411/I2C2_SDA -> -12V
- U5 pad 5: /stm32F411/I2C2_SCL -> Net-(U5B-+)
- U5 pad 6: VREF__2_5V -> GNDREF
- U6 pad 1: +3.3V -> Net-(R32-Pad1)
- U6 pad 2: unconnected-(U6-PC13-Pad2) -> Net-(U6A--)
- U6 pad 3: unconnected-(U6-PC14-Pad3) -> Net-(U10-VOUT)
- U6 pad 4: unconnected-(U6-PC15-Pad4) -> GNDREF
- U6 pad 5: unconnected-(U6-PH0-Pad5) -> Net-(U13-VOUT)
- U6 pad 6: unconnected-(U6-PH1-Pad6) -> Net-(U6B--)
- U6 pad 7: /stm32F411/NRST -> Net-(R44-Pad1)
- U6 pad 8: unconnected-(U6-PC0-Pad8) -> +12V
- U7 pad 1: /display/segment_display/E_1 -> /cv_input/CV_OUT
- U7 pad 2: /display/segment_display/N_2 -> Net-(U7A--)
- U7 pad 3: /display/segment_display/M_4 -> GNDREF
- U7 pad 4: /display/segment_display/L_5 -> GNDREF
- U7 pad 5: /display/segment_display/K_6 -> GNDREF
- U7 pad 6: /display/segment_display/D_7 -> Net-(U7B--)
- U7 pad 7: /display/segment_display/C_9 -> /cv_input1/CV_OUT
- U7 pad 8: GNDREF -> +3.3V
- U8 pad 1: Net-(U8-E) -> VREF__2_5V
- U8 pad 2: Net-(U8-N) -> GNDREF
- U8 pad 3: (no net) -> unconnected-(U8-NC-Pad3)
- U9 pad 1: /display/segment_display/B_10 -> Net-(U9-E)
- U9 pad 10: +3.3V -> Net-(U9-B)
- U9 pad 11: /display/DISPLAY_CLOCK -> /display/segment_display/K2
- U9 pad 12: /display/DISPLAY_ENABLE -> Net-(U9-A)
- U9 pad 13: GNDREF -> Net-(U9-P)
- U9 pad 14: Net-(U7-QH') -> Net-(U9-J)
- U9 pad 15: unconnected-(U9-QA-Pad15) -> Net-(U9-H)
- U9 pad 16: +3.3V -> /display/segment_display/K1
- U9 pad 2: /display/segment_display/A_12 -> Net-(U9-N)
- U9 pad 3: /display/segment_display/P_13 -> (no net)
- U9 pad 4: /display/segment_display/J_14 -> Net-(U9-M)
- U9 pad 5: /display/segment_display/H_15 -> Net-(U9-L)
- U9 pad 6: /display/segment_display/G_17 -> Net-(U9-K)
- U9 pad 7: /display/segment_display/F_18 -> Net-(U9-D)
- U9 pad 8: GNDREF -> unconnected-(U9-DP1-Pad8)
- U9 pad 9: unconnected-(U9-QH'-Pad9) -> Net-(U9-C)
Routing:
- net /stm32F411/I2C1_SCL: track 5.56 -> 0.00 mm
- net /stm32F411/I2C1_SDA: track 3.19 -> 0.00 mm
- net Net-(U8-E): track 1.94 -> 0.00 mm
- net Net-(U8-N): track 1.93 -> 0.00 mm
- removed copper zone on In4.Cu, net GNDREF
Other:
- board size 30 x 110 mm -> 59 x 110 mm
- copper layers 6 -> 4

Commit message: quantizers_stls
Parts:
- removed U13: MCP47256, Package_TO_SOT_SMD:SOT-23-6_Handsoldering
- added C26: 100nF, Capacitor_SMD:C_0805_2012Metric_Pad1.18x1.45mm_HandSolder, B.Cu at (66.3, 90.5)
- added C27: 100nF, Capacitor_SMD:C_0805_2012Metric_Pad1.18x1.45mm_HandSolder, B.Cu at (90.2, 90.5)
- added C28: 100nF, Capacitor_SMD:C_0805_2012Metric_Pad1.18x1.45mm_HandSolder, B.Cu at (66.2, 77.5)
- added C29: 100nF, Capacitor_SMD:C_0805_2012Metric_Pad1.18x1.45mm_HandSolder, B.Cu at (171.1, 123.9)
- added C30: 100nF, Capacitor_SMD:C_0805_2012Metric_Pad1.18x1.45mm_HandSolder, B.Cu at (172.9, 117.2)
- added D6: 1N5817, Diode_SMD:D_SOD-323_HandSoldering, B.Cu at (151.2, 104.4)
- added D7: 1N5817, Diode_SMD:D_SOD-323_HandSoldering, B.Cu at (133.8, 101.8)
- added D8: 1N5817, Diode_SMD:D_SOD-323_HandSoldering, B.Cu at (133.8, 106.0)
- added D9: 1N4148WS, Diode_SMD:D_SOD-323_HandSoldering, B.Cu at (72.0, 153.8)
- added G***: LOGO, Synth:lenimal_logo_full, F.Cu at (79.6, 124.2)
- added G***: LOGO, Synth:lenimal_logo_full, B.Cu at (183.3, 130.8)
- added G***: LOGO, Synth:lenimal_logo_full, B.Cu at (79.6, 124.3)
- added J10: TRIG_INPUT, Synth:Jack_3.5mm_QingPu_WQP-PJ398SM_Vertical_CircularHoles, F.Cu at (67.0, 153.0)
- added J11: TRIG_OUT, Synth:Jack_3.5mm_QingPu_WQP-PJ398SM_Vertical_CircularHoles, F.Cu at (104.0, 138.1)
- added J12: TRIG_OUT, Synth:Jack_3.5mm_QingPu_WQP-PJ398SM_Vertical_CircularHoles, F.Cu at (104.0, 153.0)
- added J13: Conn_02x03_Odd_Even, Connector_PinHeader_2.54mm:PinHeader_2x03_P2.54mm_Vertical, B.Cu at (77.7, 138.4)
- added R49: 10K [0.1%], Resistor_SMD:R_0805_2012Metric_Pad1.20x1.40mm_HandSolder, B.Cu at (136.8, 101.0)
- added R50: 22K [1%], Resistor_SMD:R_0805_2012Metric_Pad1.20x1.40mm_HandSolder, B.Cu at (140.5, 119.5)
- added R51: 10K [0.1%], Resistor_SMD:R_0805_2012Metric_Pad1.20x1.40mm_HandSolder, B.Cu at (136.8, 103.0)
- added R52: 18K [1%], Resistor_SMD:R_0805_2012Metric_Pad1.20x1.40mm_HandSolder, B.Cu at (144.5, 119.5)
- added R53: 10K, Resistor_SMD:R_0805_2012Metric_Pad1.20x1.40mm_HandSolder, B.Cu at (64.5, 150.5)
- added R54: 10K, Resistor_SMD:R_0805_2012Metric_Pad1.20x1.40mm_HandSolder, B.Cu at (72.0, 157.8)
- added R55: 100K, Resistor_SMD:R_0805_2012Metric_Pad1.20x1.40mm_HandSolder, B.Cu at (72.2, 155.8)
- added R56: 1K, Resistor_SMD:R_0805_2012Metric_Pad1.20x1.40mm_HandSolder, B.Cu at (100.0, 141.0)
- added R57: 1K, Resistor_SMD:R_0805_2012Metric_Pad1.20x1.40mm_HandSolder, B.Cu at (100.0, 143.0)
- added R59: 1K, Resistor_SMD:R_0805_2012Metric_Pad1.20x1.40mm_HandSolder, B.Cu at (100.0, 156.0)
- added R60: 1K, Resistor_SMD:R_0805_2012Metric_Pad1.20x1.40mm_HandSolder, B.Cu at (100.0, 158.0)
- added REF**: WEEE-Logo_5.6x8mm_SilkScreen, Symbol:WEEE-Logo_5.6x8mm_SilkScreen, B.Cu at (133.7, 86.3)
- added REF**: WEEE-Logo_5.6x8mm_SilkScreen, Symbol:WEEE-Logo_5.6x8mm_SilkScreen, B.Cu at (54.1, 112.5)
- added SW10: CH_1_SW, Synth:ML6-H2T2GQA, F.Cu at (56.0, 90.0)
- added SW11: CH_2_SW, Synth:ML6-H2T2GQA, F.Cu at (59.2, 78.0)
- added SW12: CH_2_SW, Synth:ML6-H2T2GQA, F.Cu at (68.0, 69.2)
- added SW13: SW_Push, Synth:SW_PUSH_6mm, F.Cu at (61.0, 124.0)
- added SW14: ENCODER, Synth:RotaryEncoder_Alps_EC11E-Switch_Vertical_H20mm_CircularMountingHoles, F.Cu at (80.0, 90.0)
- added SW15: SW_Push, Synth:SW_PUSH_6mm, F.Cu at (99.0, 124.0)
- added SW4: CH_2_SW, Synth:ML6-H2T2GQA, F.Cu at (104.0, 90.0)
- added SW5: CH_1_SW, Synth:ML6-H2T2GQA, F.Cu at (100.8, 102.0)
- added SW6: CH_1_SW, Synth:ML6-H2T2GQA, F.Cu at (92.0, 110.8)
- added SW7: CH_2_SW, Synth:ML6-H2T2GQA, F.Cu at (80.0, 114.0)
- added SW8: CH_2_SW, Synth:ML6-H2T2GQA, F.Cu at (68.0, 110.8)
- added SW9: CH_1_SW, Synth:ML6-H2T2GQA, F.Cu at (59.2, 102.0)
- added TP4: CV_IN, TestPoint:TestPoint_Loop_D2.50mm_Drill1.0mm, B.Cu at (156.4, 122.6)
- added TP5: CV_OUT_1, TestPoint:TestPoint_Loop_D2.50mm_Drill1.0mm, B.Cu at (150.2, 110.5)
- added TP6: CV_OUT_2, TestPoint:TestPoint_Loop_D2.50mm_Drill1.0mm, B.Cu at (147.2, 95.2)
- added TP7: CV_IN, TestPoint:TestPoint_Loop_D2.50mm_Drill1.0mm, B.Cu at (147.7, 128.0)
- added TP8: CV_OUT_1, TestPoint:TestPoint_Loop_D2.50mm_Drill1.0mm, B.Cu at (134.5, 111.8)
- added TP9: CV_OUT_2, TestPoint:TestPoint_Loop_D2.50mm_Drill1.0mm, B.Cu at (137.8, 95.2)
- added U11: DAC80502, Package_DIP:DIP-10_W7.62mm_LongPads, F.Cu at (174.0, 122.1)
- added XP1: Conn_01x08_Pin, Connector_PinHeader_2.54mm:PinHeader_1x08_P2.54mm_Vertical, B.Cu at (88.9, 128.0)
- added XP10: Conn_01x04_Pin, Connector_PinHeader_2.54mm:PinHeader_1x04_P2.54mm_Vertical, B.Cu at (83.8, 79.0)
- added XP11: Conn_01x04_Pin, Connector_PinHeader_2.54mm:PinHeader_1x04_P2.54mm_Vertical, B.Cu at (83.8, 101.0)
- added XP12: Conn_01x04_Socket, Connector_PinSocket_2.54mm:PinSocket_1x04_P2.54mm_Vertical, F.Cu at (163.8, 101.0)
- added XP13: Conn_01x04_Pin, Connector_PinHeader_2.54mm:PinHeader_1x04_P2.54mm_Vertical, B.Cu at (52.0, 72.0)
- added XP14: Conn_01x04_Socket, Connector_PinSocket_2.54mm:PinSocket_1x04_P2.54mm_Vertical, F.Cu at (132.0, 72.0)
- added XP15: Conn_01x04_Socket, Connector_PinSocket_2.54mm:PinSocket_1x04_P2.54mm_Vertical, F.Cu at (188.0, 72.0)
- added XP16: Conn_01x04_Pin, Connector_PinHeader_2.54mm:PinHeader_1x04_P2.54mm_Vertical, B.Cu at (108.0, 72.0)
- added XP2: Conn_01x08_Socket, Connector_PinSocket_2.54mm:PinSocket_1x08_P2.54mm_Vertical, F.Cu at (168.9, 128.0)
- added XP3: Conn_01x04_Socket, Connector_PinSocket_2.54mm:PinSocket_1x04_P2.54mm_Vertical, F.Cu at (188.0, 127.0)
- added XP4: Conn_01x04_Pin, Connector_PinHeader_2.54mm:PinHeader_1x04_P2.54mm_Vertical, B.Cu at (108.0, 127.0)
- added XP5: Conn_01x04_Pin, Connector_PinHeader_2.54mm:PinHeader_1x04_P2.54mm_Vertical, B.Cu at (52.0, 127.0)
- added XP6: Conn_01x04_Socket, Connector_PinSocket_2.54mm:PinSocket_1x04_P2.54mm_Vertical, F.Cu at (132.0, 127.0)
- added XP7: Conn_01x04_Pin, Connector_PinHeader_2.54mm:PinHeader_1x04_P2.54mm_Vertical, B.Cu at (83.8, 105.0)
- added XP8: Conn_01x04_Socket, Connector_PinSocket_2.54mm:PinSocket_1x04_P2.54mm_Vertical, F.Cu at (163.8, 105.0)
- added XP9: Conn_01x04_Socket, Connector_PinSocket_2.54mm:PinSocket_1x04_P2.54mm_Vertical, F.Cu at (163.8, 79.0)
- added Y1: 20MHZ, Crystal:Crystal_SMD_HC49-SD, B.Cu at (160.0, 90.0)
- C10: value 2.2uF -> 20pF
- C11: value 100nF -> 20pF
- C12: value 100nF -> 2.2uF
- C18: moved to B.Cu
- C21: value 47uF -> 100nF; footprint Capacitor_THT:CP_Radial_D6.3mm_P2.50mm -> Capacitor_SMD:C_0805_2012Metric_Pad1.18x1.45mm_HandSolder
- C22: value 100nF -> 47uF; footprint Capacitor_SMD:C_0805_2012Metric_Pad1.18x1.45mm_HandSolder -> Capacitor_THT:CP_Radial_D6.3mm_P2.50mm
- C23: value 470nF -> 100nF
- C24: value 100nF -> 470nF
- D5: value 1N4148WS -> 1N5817
- J1: value BOOT_RUN -> CV_INPUT; footprint Connector_PinHeader_2.54mm:PinHeader_1x03_P2.54mm_Vertical -> Synth:Jack_3.5mm_QingPu_WQP-PJ398SM_Vertical_CircularHoles; moved to F.Cu
- J2: value RX/TX -> CV_OUTPUT; footprint Connector_PinHeader_2.54mm:PinHeader_1x03_P2.54mm_Vertical -> Synth:Jack_3.5mm_QingPu_WQP-PJ398SM_Vertical_CircularHoles; moved to F.Cu
- J3: value Conn_01x04 -> CV_OUTPUT; footprint Connector_PinHeader_2.54mm:PinHeader_1x04_P2.54mm_Vertical -> Synth:Jack_3.5mm_QingPu_WQP-PJ398SM_Vertical_CircularHoles; moved to F.Cu
- J5: value CV_INPUT -> BOOT_RUN; footprint Synth:Jack_3.5mm_QingPu_WQP-PJ398SM_Vertical_CircularHoles -> Connector_PinHeader_2.54mm:PinHeader_1x03_P2.54mm_Vertical; moved to B.Cu
- J6: value CV_OUTPUT -> RX/TX; footprint Synth:Jack_3.5mm_QingPu_WQP-PJ398SM_Vertical_CircularHoles -> Connector_PinHeader_2.54mm:PinHeader_1x03_P2.54mm_Vertical; moved to B.Cu
- J7: value CV_INPUT -> Conn_01x04; footprint Synth:Jack_3.5mm_QingPu_WQP-PJ398SM_Vertical_CircularHoles -> Connector_PinHeader_2.54mm:PinHeader_1x04_P2.54mm_Vertical; moved to B.Cu
- J8: value CV_INPUT -> I2C1; footprint Synth:Jack_3.5mm_QingPu_WQP-PJ398SM_Vertical_CircularHoles -> Connector_PinHeader_2.54mm:PinHeader_1x03_P2.54mm_Vertical; moved to B.Cu
- J9: value CV_OUTPUT -> TRIG_INPUT
- R1, R2: value 10K -> 1K
- R10: value 470R -> 10K
- R11, R13, R15, R17, R19, R21, R23: value 100R -> 470R
- R12, R14, R16, R18, R20, R22, R24: value 100R -> 10K
- R25: value 10K -> 470R
- R27: value 100K -> 470R
- R28: value 22K -> 10K
- R29, R31: value 22K -> 470R
- R3, R32, R4: value 1K -> 10K
- R30: value 120K -> 10K
- R33: value 3K3 -> 470R
- R34: value 3K3 -> 10K
- R35: value 30K [0.1%] -> 10K
- R36: value 10K [0.1%] -> 100K
- R37: value 22K -> 40K [0.1%]
- R38: value 22K -> 10K [0.1%]
- R39: value 120K -> 10K [0.1%]
- R40: value 22K -> 22K [1%]
- R41: value 10K -> 10K [0.1%]
- R42: value 10K -> 18K [1%]
- R43: value 100K -> 30K [0.1%]
- R44: value 1K -> 10K [0.1%]
- R45: value 3K3 -> 30K [0.1%]
- R46: value 3K3 -> 10K [0.1%]
- R47: value 30K [0.1%] -> 40K [0.1%]
- R5: value 10R -> 100R
- R6: value 1K -> 10R
- R7: value 2K -> 1K
- R8: value 10R -> 2K
- R9: value 470R -> 10R
- SW2: value ENCODER -> CH_1_SW; footprint Synth:RotaryEncoder_Alps_EC11E-Switch_Vertical_H20mm_CircularMountingHoles -> Synth:ML6-H2T2GQA
- TP1, TP2, TP3: moved to F.Cu
- U10: value MCP47256 -> 74HC165; footprint Package_TO_SOT_SMD:SOT-23-6_Handsoldering -> Synth:SOIC-16
- U2: value 74HC595 -> LM1117DT-3.3; footprint Synth:SOIC-16 -> Package_TO_SOT_SMD:TO-252-3_TabPin2
- U3: value 74HC595 -> TL072; footprint Synth:SOIC-16 -> Synth:SOIC-8
- U4: value LM1117DT-3.3 -> OPA2277; footprint Package_TO_SOT_SMD:TO-252-3_TabPin2 -> Synth:SOIC-8; moved to B.Cu
- U5: value TL072 -> MCP6002
- U6: value OPA2277 -> LM4040DBZ-2.5; footprint Synth:SOIC-8 -> Package_TO_SOT_SMD:SOT-23
- U7: value MCP6002 -> 74HC165; footprint Synth:SOIC-8 -> Synth:SOIC-16
- U8: value LM4040DBZ-2.5 -> 74HC595; footprint Package_TO_SOT_SMD:SOT-23 -> Synth:SOIC-16
- U9: value dual_segment_display -> 74HC595; footprint Synth:7-segment-display_DA56 -> Synth:SOIC-16; moved to B.Cu
- moved C5 155.8 mm to (183.2, 87.5)
- moved C3 153.0 mm to (183.2, 89.6)
- moved C4 150.0 mm to (183.2, 102.5)
- moved C6 145.7 mm to (170.9, 84.1), turned to 0 degrees
- moved FB1 144.0 mm to (165.4, 86.4)
- moved C9 143.8 mm to (165.3, 84.4)
- moved C8 141.2 mm to (165.4, 88.4), turned to 0 degrees
- moved C7 141.1 mm to (168.2, 93.2), turned to 0 degrees
- moved C2 140.2 mm to (170.8, 89.6), turned to 0 degrees
- moved C1 135.6 mm to (170.8, 102.5), turned to 0 degrees
- moved U5 132.8 mm to (142.5, 102.3)
- moved C10 131.6 mm to (155.2, 94.8), turned to -90 degrees
- moved R37 130.6 mm to (153.5, 124.5), turned to -90 degrees
- moved R38 122.9 mm to (147.3, 111.5), turned to -90 degrees
- moved R40 116.3 mm to (140.5, 121.5), turned to 0 degrees
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Connections:
- C1 pad 1: GNDREF -> GND
- C1 pad 2: +3.3V -> +3.3VB
- C10 pad 1: /stm32F411/VCap -> Net-(C10-Pad1)
- C10 pad 2: GNDREF -> GND
- C11 pad 1: +3.3V -> Net-(U1-PH1)
- C11 pad 2: GNDREF -> GND
- C12 pad 1: +3.3V -> /stm32F411/VCap
- C12 pad 2: GNDREF -> GND
- C15 pad 1: +12V -> +12VB
- C15 pad 2: GNDREF -> GND
- C17 pad 1: +3.3V -> +3.3VB
- C17 pad 2: GNDREF -> GND
- C2 pad 1: GNDREF -> GND
- C2 pad 2: +3.3V -> +3.3VB
- C20 pad 1: GNDREF -> GND
- C20 pad 2: -12V -> -12VB
- C23 pad 1: VREF__2_5V -> GNDREF
- C23 pad 2: GNDREF -> -12V
- C24 pad 1: GNDREF -> VREF__2_5V
- C24 pad 2: +3.3V -> GND
- C25 pad 1: GNDREF -> +3.3V
- C25 pad 2: +3.3V -> GNDREF
- C3 pad 1: GNDREF -> GND
- C3 pad 2: +3.3V -> +3.3VB
- C4 pad 1: GNDREF -> GND
- C4 pad 2: +3.3V -> +3.3VB
- C5 pad 1: GNDREF -> GND
- C5 pad 2: +3.3V -> +3.3VB
- C6 pad 2: GNDREF -> GND
- C7 pad 1: GNDREF -> GND
- C8 pad 1: GNDREF -> GND
- C9 pad 1: GNDREF -> GND
- C9 pad 2: +3.3V -> +3.3VB
- D5 pad 1: Net-(D5-K) -> +3.3VB
- D5 pad 2: GNDREF -> Net-(D5-A)
- FB1 pad 2: +3.3V -> +3.3VB
- J4 pad T: Net-(J4-PadT) -> Net-(XP1H-Pin_8)
- J4 pad TN: Net-(J4-PadTN) -> Net-(J13-Pin_2)
- J9 pad TN: unconnected-(J9-PadTN) -> Net-(J9-PadTN)
- Q1 pad 1: Net-(Q1-B) -> Net-(D4-K)
- Q1 pad 3: /display/segment_display/K1 -> /trigger_input/TRIG_OUT
- Q2 pad 1: Net-(Q2-B) -> Net-(D9-K)
- Q2 pad 3: /display/segment_display/K2 -> /trigger_input1/TRIG_OUT
- Q3 pad 1: Net-(D4-K) -> /channel_a_trigger/TRIG_IN
- Q3 pad 3: /stm32F411/TRIG_1_IN -> Net-(Q3-C)
- Q4 pad 1: Net-(D5-K) -> /channel_b_trigger/TRIG_IN
- Q4 pad 3: /stm32F411/TRIG_2_IN -> Net-(Q4-C)
- R1 pad 1: /stm32F411/NRST -> /cv_output/OUT_A
- R1 pad 2: +3.3V -> Net-(J2-PadT)
- R10 pad 1: /controls/LED_2 -> GNDREF
- R10 pad 2: Net-(R10-Pad2) -> Net-(SW1-A)
- R11 pad 1: Net-(U9-A) -> Net-(U8-QB)
- R11 pad 2: /display/segment_display/A_12 -> Net-(R11-Pad2)
- R12 pad 1: Net-(U9-B) -> GNDREF
- R12 pad 2: /display/segment_display/B_10 -> Net-(SW2-A)
- R13 pad 1: Net-(U9-C) -> Net-(U8-QC)
- R13 pad 2: /display/segment_display/C_9 -> Net-(R13-Pad2)
- R14 pad 1: Net-(U9-D) -> GNDREF
- R14 pad 2: /display/segment_display/D_7 -> Net-(SW3-A)
- R15 pad 1: Net-(U9-E) -> Net-(U8-QD)
- R15 pad 2: /display/segment_display/E_1 -> Net-(R15-Pad2)
- R16 pad 1: Net-(U9-F) -> GNDREF
- R16 pad 2: /display/segment_display/F_18 -> Net-(SW4-A)
- R17 pad 1: Net-(U9-G) -> Net-(U8-QE)
- R17 pad 2: /display/segment_display/G_17 -> Net-(R17-Pad2)
- R18 pad 1: Net-(U9-H) -> GNDREF
- R18 pad 2: /display/segment_display/H_15 -> Net-(SW5-A)
- R19 pad 1: Net-(U9-J) -> Net-(U8-QF)
- R19 pad 2: /display/segment_display/J_14 -> Net-(R19-Pad2)
- R2 pad 1: /stm32F411/BOOT0 -> /cv_output/OUT_B
- R2 pad 2: /stm32F411/BOOT0_MCU -> Net-(J3-PadT)
- R20 pad 1: Net-(U9-K) -> GNDREF
- R20 pad 2: /display/segment_display/K_6 -> Net-(SW6-A)
- R21 pad 1: Net-(U9-L) -> Net-(U8-QG)
- R21 pad 2: /display/segment_display/L_5 -> Net-(R21-Pad2)
- R22 pad 1: Net-(U9-M) -> GNDREF
- R22 pad 2: /display/segment_display/M_4 -> Net-(SW7-A)
- R23 pad 1: Net-(U9-N) -> Net-(U9-QB)
- R23 pad 2: /display/segment_display/N_2 -> Net-(R23-Pad2)
- R24 pad 1: Net-(U9-P) -> GNDREF
- R24 pad 2: /display/segment_display/P_13 -> Net-(SW8-A)
- R25 pad 1: /stm32F411/TRIG_1_EN -> Net-(U9-QC)
- R25 pad 2: Net-(J4-PadTN) -> Net-(R25-Pad2)
- R26 pad 1: Net-(D4-K) -> GNDREF
- R26 pad 2: Net-(J4-PadT) -> Net-(SW9-A)
- R27 pad 1: Net-(D4-K) -> Net-(U9-QD)
- R27 pad 2: GNDREF -> Net-(R27-Pad2)
- R28 pad 1: Net-(R28-Pad1) -> GNDREF
- R28 pad 2: Net-(U5A-+) -> Net-(SW10-A)
- R29 pad 1: /cv_input/CV_OUT -> Net-(U9-QE)
- R29 pad 2: Net-(U7A--) -> Net-(R29-Pad2)
- R3 pad 1: Net-(Q1-B) -> /stm32F411/NRST
- R3 pad 2: /display/DISPLAY_CHAR_1 -> +3.3VB
- R30 pad 1: Net-(U5A-+) -> GNDREF
- R30 pad 2: Net-(J5-PadT) -> Net-(SW11-A)
- R31 pad 1: Net-(U7A--) -> Net-(U9-QF)
- R31 pad 2: Net-(R28-Pad1) -> Net-(R31-Pad2)
- R32 pad 1: Net-(R32-Pad1) -> GNDREF
- R32 pad 2: Net-(J6-PadT) -> Net-(SW12-A)
- R33 pad 1: /cv_output/SCL_IN -> Net-(U9-QG)
- R33 pad 2: +3.3V -> Net-(R33-Pad2)
- R34 pad 1: /cv_output/SDA_IN -> /trigger_input/TRIG_ENABLED
- R34 pad 2: +3.3V -> Net-(J9-PadTN)
- R35 pad 1: Net-(U6A--) -> Net-(D4-K)
- R35 pad 2: Net-(R32-Pad1) -> Net-(J9-PadT)
- R36 pad 1: GNDREF -> Net-(D4-K)
- R36 pad 2: Net-(U6A--) -> GNDREF
- R37 pad 1: Net-(R37-Pad1) -> Net-(U3A--)
- R37 pad 2: Net-(U5B-+) -> /cv_normalizer/CV_IN
- R38 pad 1: /cv_input1/CV_OUT -> Net-(D5-A)
- R38 pad 2: Net-(U7B--) -> Net-(U3A--)
- R39 pad 1: Net-(U5B-+) -> /cv_normalizer/CV_OUT
- R39 pad 2: Net-(J7-PadT) -> Net-(U5A--)
- R4 pad 1: Net-(Q2-B) -> /stm32F411/BOOT0
- R4 pad 2: /display/DISPLAY_CHAR_2 -> /stm32F411/BOOT0_MCU
- R40 pad 1: Net-(U7B--) -> +3.3VB
- R40 pad 2: Net-(R37-Pad1) -> Net-(U3A-+)
- R41 pad 1: /stm32F411/TRIG_2_EN -> Net-(U5A--)
- R41 pad 2: Net-(J8-PadTN) -> Net-(D5-A)
- R42 pad 1: Net-(D5-K) -> Net-(U3A-+)
- R42 pad 2: Net-(J8-PadT) -> GND
- R43 pad 1: Net-(D5-K) -> Net-(U4A--)
- R43 pad 2: GNDREF -> /cv_output/OUT_B
- R44 pad 1: Net-(R44-Pad1) -> GNDREF
- R44 pad 2: Net-(J9-PadT) -> Net-(U4A--)
- R45 pad 1: /cv_output1/SCL_IN -> Net-(U4B--)
- R45 pad 2: +3.3V -> /cv_output/OUT_A
- R46 pad 1: /cv_output1/SDA_IN -> GNDREF
- R46 pad 2: +3.3V -> Net-(U4B--)
- R47 pad 1: Net-(U6B--) -> Net-(U3B--)
- R47 pad 2: Net-(R44-Pad1) -> /cv_normalizer1/CV_IN
- R48 pad 1: GNDREF -> Net-(D7-A)
- R48 pad 2: Net-(U6B--) -> Net-(U3B--)
- R5 pad 1: Net-(D1-K) -> Net-(C10-Pad1)
- R5 pad 2: +12V -> Net-(U1-PH0)
- R6 pad 1: VREF__2_5V -> Net-(D1-K)
- R6 pad 2: +3.3V -> +12V
- R7 pad 1: GNDREF -> VREF__2_5V
- R7 pad 2: Net-(D2-K) -> +3.3VB
- R8 pad 1: Net-(D3-A) -> GNDREF
- R8 pad 2: -12V -> Net-(D2-K)
- R9 pad 1: /controls/LED_1 -> Net-(D3-A)
- R9 pad 2: Net-(R9-Pad2) -> -12V
- SW1 pad 1: /controls/LED_SW_1 -> +3.3V
- SW1 pad 2: /controls/LED_SW_1 -> +3.3V
- SW1 pad 3: GNDREF -> Net-(SW1-A)
- SW1 pad 4: GNDREF -> Net-(SW1-A)
- SW1 pad L1: Net-(R9-Pad2) -> Net-(R11-Pad2)
- SW3 pad 1: /controls/LED_SW_2 -> +3.3V
- SW3 pad 2: /controls/LED_SW_2 -> +3.3V
- SW3 pad 3: GNDREF -> Net-(SW3-A)
- SW3 pad 4: GNDREF -> Net-(SW3-A)
- SW3 pad L1: Net-(R10-Pad2) -> Net-(R15-Pad2)
- U1 pad 1: +3.3V -> +3.3VB
- U1 pad 10: unconnected-(U1-PC2-Pad10) -> /cv_normalizer/CV_OUT
- U1 pad 11: unconnected-(U1-PC3-Pad11) -> /cv_normalizer1/CV_OUT
- U1 pad 12: GNDREF -> GND
- U1 pad 14: /cv_input/CV_OUT -> unconnected-(U1-PA0-Pad14)
- U1 pad 15: /cv_input1/CV_OUT -> unconnected-(U1-PA1-Pad15)
- U1 pad 18: GNDREF -> GND
- U1 pad 19: +3.3V -> +3.3VB
- U1 pad 21: /controls/ENC_SW -> /stm32F411/ENC_SW
- U1 pad 22: /controls/ENC_CH_A -> /stm32F411/ENC_1
- U1 pad 23: /controls/ENC_CH_B -> /stm32F411/ENC_2
- U1 pad 24: unconnected-(U1-PC4-Pad24) -> /stm32F411/TRIG_A_IN
- U1 pad 25: unconnected-(U1-PC5-Pad25) -> /stm32F411/TRIG_B_IN
- U1 pad 26: unconnected-(U1-PB0-Pad26) -> /stm32F411/TRIG_A_OUT
- U1 pad 27: unconnected-(U1-PB1-Pad27) -> /stm32F411/TRIG_B_OUT
- U1 pad 29: /cv_output1/SCL_IN -> /stm32F411/SPI2_SW_SCK
- U1 pad 3: /stm32F411/TRIG_1_IN -> unconnected-(U1-PC14-Pad3)
- U1 pad 31: GNDREF -> GND
- U1 pad 32: +3.3V -> +3.3VB
- U1 pad 33: /controls/LED_1 -> unconnected-(U1-PB12-Pad33)
- U1 pad 34: /controls/LED_SW_1 -> /stm32F411/SPI2_SW_READ
- U1 pad 35: /controls/LED_2 -> /stm32F411/SPI2_SW_MISO
- U1 pad 36: /controls/LED_SW_2 -> unconnected-(U1-PB15-Pad36)
- U1 pad 38: unconnected-(U1-PC7-Pad38) -> /stm32F411/SW_A
- U1 pad 39: unconnected-(U1-PC8-Pad39) -> /stm32F411/SW_B
- U1 pad 4: /stm32F411/TRIG_2_IN -> unconnected-(U1-PC15-Pad4)
- U1 pad 44: /display/DISPLAY_CHAR_1 -> unconnected-(U1-PA11-Pad44)
- U1 pad 45: /display/DISPLAY_CHAR_2 -> unconnected-(U1-PA12-Pad45)
- U1 pad 47: GNDREF -> GND
- U1 pad 48: +3.3V -> +3.3VB
- U1 pad 5: unconnected-(U1-PH0-Pad5) -> Net-(U1-PH0)
- U1 pad 51: /display/DISPLAY_CLOCK -> /stm32F411/SPI3_LED_SCK
- U1 pad 52: /display/DISPLAY_ENABLE -> /stm32F411/SPI3_LED_WRITE
- U1 pad 53: /display/DISPLAY_DATA_IN -> /stm32F411/SPI3_LED_MOSI
- U1 pad 55: /cv_output1/SDA_IN -> /cv_output/SCLK
- U1 pad 56: unconnected-(U1-PB4-Pad56) -> /cv_output/_SYNC
- U1 pad 57: unconnected-(U1-PB5-Pad57) -> /cv_output/SDIN
- U1 pad 58: /cv_output/SCL_IN -> Net-(J8-Pin_2)
- U1 pad 59: /cv_output/SDA_IN -> Net-(J8-Pin_3)
- U1 pad 6: unconnected-(U1-PH1-Pad6) -> Net-(U1-PH1)
- U1 pad 63: GNDREF -> GND
- U1 pad 64: +3.3V -> +3.3VB
- U1 pad 8: /stm32F411/TRIG_1_EN -> /stm32F411/TRIG_A_EN
- U1 pad 9: /stm32F411/TRIG_2_EN -> /stm32F411/TRIG_B_EN
- U10 pad 1: Net-(U10-VOUT) -> /controls/SW_READ
- U10 pad 2: GNDREF -> /controls/SW_SCK
- U10 pad 3: +3.3V -> Net-(SW11-A)
- U10 pad 4: /cv_output/SDA_IN -> Net-(SW12-A)
- U10 pad 5: /cv_output/SCL_IN -> unconnected-(U10-D6-Pad5)
- U10 pad 6: VREF__2_5V -> unconnected-(U10-D7-Pad6)
- U2 pad 1: /display/segment_display/E_1 -> GNDREF
- U2 pad 2: /display/segment_display/N_2 -> +3.3V
- U2 pad 3: /display/segment_display/M_4 -> +12V
- U3 pad 1: /display/segment_display/B_10 -> Net-(D5-A)
- U3 pad 2: /display/segment_display/A_12 -> Net-(U3A--)
- U3 pad 3: /display/segment_display/P_13 -> Net-(U3A-+)
- U3 pad 4: /display/segment_display/J_14 -> -12VB
- U3 pad 5: /display/segment_display/H_15 -> Net-(U3B-+)
- U3 pad 6: /display/segment_display/G_17 -> Net-(U3B--)
- U3 pad 7: /display/segment_display/F_18 -> Net-(D7-A)
- U3 pad 8: GNDREF -> +12VB
- U4 pad 1: GNDREF -> /cv_output/OUT_B
- U4 pad 2: +3.3V -> Net-(U4A--)
- U4 pad 3: +12V -> Net-(U4A-+)
- U5 pad 1: Net-(R28-Pad1) -> /cv_normalizer/CV_OUT
- U5 pad 2: GNDREF -> Net-(U5A--)
- U5 pad 3: Net-(U5A-+) -> GND
- U5 pad 4: -12V -> GND
- U5 pad 5: Net-(U5B-+) -> GND
- U5 pad 6: GNDREF -> Net-(U5B--)
- U5 pad 7: Net-(R37-Pad1) -> /cv_normalizer1/CV_OUT
- U5 pad 8: +12V -> +3.3VB
- U6 pad 1: Net-(R32-Pad1) -> VREF__2_5V
- U6 pad 2: Net-(U6A--) -> GND
- U6 pad 3: Net-(U10-VOUT) -> unconnected-(U6-NC-Pad3)
- U7 pad 1: /cv_input/CV_OUT -> /controls/SW_READ
- U7 pad 2: Net-(U7A--) -> /controls/SW_SCK
- U7 pad 3: GNDREF -> Net-(SW5-A)
- U7 pad 4: GNDREF -> Net-(SW6-A)
- U7 pad 5: GNDREF -> unconnected-(U7-D6-Pad5)
- U7 pad 6: Net-(U7B--) -> unconnected-(U7-D7-Pad6)
- U7 pad 7: /cv_input1/CV_OUT -> unconnected-(U7-~{Q7}-Pad7)
- U7 pad 8: +3.3V -> GNDREF
- U8 pad 1: VREF__2_5V -> Net-(U8-QB)
- U8 pad 2: GNDREF -> Net-(U8-QC)
- U8 pad 3: unconnected-(U8-NC-Pad3) -> Net-(U8-QD)
- U9 pad 1: Net-(U9-E) -> Net-(U9-QB)
- U9 pad 10: Net-(U9-B) -> +3.3V
- U9 pad 11: /display/segment_display/K2 -> /controls/LED_SCK
- U9 pad 12: Net-(U9-A) -> /controls/LED_WRITE
- U9 pad 13: Net-(U9-P) -> GNDREF
- U9 pad 14: Net-(U9-J) -> Net-(U8-QH')
- U9 pad 15: Net-(U9-H) -> unconnected-(U9-QA-Pad15)
- U9 pad 16: /display/segment_display/K1 -> +3.3V
- U9 pad 2: Net-(U9-N) -> Net-(U9-QC)
- U9 pad 3: (no net) -> Net-(U9-QD)
- U9 pad 4: Net-(U9-M) -> Net-(U9-QE)
- U9 pad 5: Net-(U9-L) -> Net-(U9-QF)
- U9 pad 6: Net-(U9-K) -> Net-(U9-QG)
- U9 pad 7: Net-(U9-D) -> unconnected-(U9-QH-Pad7)
- U9 pad 8: unconnected-(U9-DP1-Pad8) -> GNDREF
- U9 pad 9: Net-(U9-C) -> /controls/unconnected-(U9-QH&amp;apos;-Pad9)
Routing:
- net +3.3V: track 0.00 -> 327.7 mm, vias 0 -> 2
- net +12V: track 0.00 -> 273.3 mm, vias 0 -> 2
- net +3.3VB: track 0.00 -> 243.5 mm, vias 0 -> 9
- net -12V: track 0.00 -> 164.5 mm, vias 0 -> 1
- net -12VB: track 0.00 -> 130.9 mm, vias 0 -> 1
- net /stm32F411/SW_A: track 0.00 -> 97.2 mm, vias 0 -> 2
- net /stm32F411/TRIG_B_EN: track 0.00 -> 53.3 mm, vias 0 -> 1
- net /stm32F411/TRIG_B_IN: track 0.00 -> 52.5 mm, vias 0 -> 1
- net /stm32F411/TRIG_A_EN: track 0.00 -> 51.8 mm, vias 0 -> 1
- net Net-(J13-Pin_1): track 0.00 -> 50.3 mm, vias 0 -> 1
- net Net-(J13-Pin_2): track 0.00 -> 50.0 mm
- net +12VB: track 0.00 -> 48.3 mm, vias 0 -> 1
- net /stm32F411/TRIG_A_IN: track 0.00 -> 46.8 mm, vias 0 -> 1
- net /stm32F411/TRIG_A_OUT: track 0.00 -> 45.7 mm, vias 0 -> 2
- net /cv_normalizer1/CV_OUT: track 0.00 -> 44.9 mm, vias 0 -> 1
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- added copper zone on B.Cu, net GND
- added copper zone on F.Cu, net GND
- added copper zone on In1.Cu, net GND
- added copper zone on In2.Cu, net GND
- added copper zone on B.Cu, net GNDREF
- added copper zone on F.Cu, net GNDREF
Other:
- board size 59 x 110 mm -> 140 x 110 mm
- board text added: "+3.3V"
- board text added: "BOOT"
- board text added: "Breakout for WSON-10 DAC80502"
- board text added: "CLK"
- board text added: "Calibration"
- board text added: "GND"
- board text added: "I2C"
- board text added: "IO"
- board text added: "LENIMAL PCB DESIGN - 05.25"
- board text added: "OFF"
- board text added: "ON"
- board text added: "Quantizzle & Sequentizzle Brain"
- board text added: "Quantizzle/Sequentizzle"
- board text added: "RUN"
- board text added: "RX"
- board text added: "TX"
- board text added: "This component has 2 modes, Quantizer or Sequencer. The front-plate is semetric and can be turned around for the alternative version."
- board text added: "github.com/lennartquerter/euro-rack-synth"
