File: modules/utility/2-quantizer/kiCad/segment_display.kicad_sch (KiCad schematic)
At the start: 15 parts, among them U8 dual_segment_display

Commit message: firmware for midas, quantizer updates
Parts:
- renumbered R21 to R11, R22 to R12, R23 to R13, R24 to R14, R25 to R15, R26 to R16, R27 to R17, R28 to R18, R29 to R19, R30 to R20, R31 to R21, R32 to R22, R33 to R23, R34 to R24, U8 to U9
