File: modules/utility/2-quantizer/kiCad/stm32F411.kicad_sch (KiCad schematic)
At the start: 17 parts, among them J5 BOOT_RUN, J6 RX/TX, J7 Conn_01x04, U6 STM32F411RETx

Commit message: firmware for midas, quantizer updates
Parts:
- renumbered C3 to C1, C14 to C10, C4 to C2, C5 to C3, C6 to C4, C7 to C5, C8 to C6, C9 to C7, C10 to C8, C11 to C9, J5 to J1, J6 to J2, J7 to J3, R19 to R1, R20 to R2, U6 to U1
Connections:
- net TRIG_1_IN: now reaches U1.3 (PC14)
- net TRIG_2_IN: now reaches U1.4 (PC15)
- net TRIG_1_EN: now reaches U1.8 (PC0)
- net TRIG_2_EN: now reaches U1.9 (PC1)
- no-connect marks 28 -> 24

Commit message: quantizers_stls
Parts:
- added C10, C11: 20pF, Capacitor_SMD:C_0805_2012Metric_Pad1.18x1.45mm_HandSolder, symbol Device:C
- added J8: I2C1, Connector_PinHeader_2.54mm:PinHeader_1x03_P2.54mm_Vertical, symbol Connector_Generic:Conn_01x03
- added R5: 100R, Resistor_SMD:R_0805_2012Metric_Pad1.20x1.40mm_HandSolder, symbol Device:R
- added Y1: 20MHZ, Crystal:Crystal_SMD_HC49-SD, symbol Device:Crystal
- renumbered C10 to C12, J1 to J5, J2 to J6, J3 to J7, R1 to R3, R2 to R4
Connections:
- net CV_A_IN: now reaches U1.10 (PC2)
- net CV_B_IN: now reaches U1.11 (PC3)
- net TRIG_A_IN: now reaches U1.24 (PC4)
- net TRIG_B_IN: now reaches U1.25 (PC5)
- net TRIG_A_OUT: now reaches U1.26 (PB0)
- net TRIG_B_OUT: now reaches U1.27 (PB1)
- net SW_A: now reaches U1.38 (PC7)
- net SW_B: now reaches U1.39 (PC8)
- net at U1.5 (PH0): now also R5.2
- net SPI1_DAC_SYNC: now reaches U1.56 (PB4)
- net SPI1_DAC_MOSI: now reaches U1.57 (PB5)
- net at U1.6 (PH1): now also C11.1, Y1.2
- net +3.3V renamed +3.3VB
- net +3.3VB: now also J8.1 (Pin_1)
- net ADC_1: no longer names the net of U1.14 (PA0)
- net ADC_2: no longer names the net of U1.15 (PA1)
- net DISPLAY_CHAR_1: no longer names the net of U1.44 (PA11)
- net DISPLAY_CHAR_2: no longer names the net of U1.45 (PA12)
- net DISPLAY_CLOCK renamed SPI3_LED_SCK
- net DISPLAY_DATA renamed SPI3_LED_MOSI
- net DISPLAY_ENABLE renamed SPI3_LED_WRITE
- net GNDREF renamed GND
- net GND: now also C10.2, C11.2
- net I2C1_SCL: no longer names the net of U1.58 (PB6)
- net I2C1_SCL: now also J8.2 (Pin_2)
- net I2C1_SDA: no longer names the net of U1.59 (PB7)
- net I2C1_SDA: now also J8.3 (Pin_3)
- net I2C2_SCL renamed SPI2_SW_SCK
- net I2C2_SDA renamed SPI1_DAC_SCK
- net LED_1: no longer names the net of U1.33 (PB12)
- net LED_2 renamed SPI2_SW_MISO
- net LED_SW_1 renamed SPI2_SW_READ
- net LED_SW_2: no longer names the net of U1.36 (PB15)
- net TRIG_1_EN renamed TRIG_A_EN
- net TRIG_1_IN: no longer names the net of U1.3 (PC14)
- net TRIG_2_EN renamed TRIG_B_EN
- net TRIG_2_IN: no longer names the net of U1.4 (PC15)
- new net: C10.1, R5.1, Y1.1
- no-connect marks 24 -> 20
Other:
- note added: "A - 0/1/2/3/4 -- ALT pins for ANALOG INPUT"
- note added: "TRIG_IN & TRIG_EN: Ensure the pins are pulled high on the MCU to register the EN"
- moved on the sheet: J5, J7
