File: modules/voltage-controlled-oscillators/3-lfo/kiCad/XOF.kicad_sch (KiCad schematic)
At the start: 54 parts, among them J1 SQUARE_OUT, J2 TRI_OUT, J3 SINE_OUT, Q3 2N3904, Q4 2N3904, SW1 SW_SPDT, U1 TL074, U2 TL074

Commit message: update XFO and 7555 ADSR, update status in readme
Parts:
- removed unit 1 of U2
- added D1: LED, Synth:LED_D5.0mm (center Aligned), symbol synth:LED (5mm)
- added D4: DUAL_LED, Synth:LED_D5.0mm (center Aligned), symbol Device:LED_Dual_Bidirectional
- added H10, H11, H12, H13, H14, H15, H8, H9: MountingHole, MountingHole:MountingHole_3.2mm_M3, symbol Mechanical:MountingHole
- added unit 1 of H4
- added unit 4 of H4
- added unit 4 of H5
- added unit 1 of H5
- added H6: PinSocket_01x04, Synth:PinSocket_1x04_P2.54mm_Vertical, symbol synth:PinSocket_01x04
- added H7: PinHeader_01x04, Synth:PinHeader_1x04_P2.54mm_Vertical, symbol synth:PinHeader_01x04
- added R20: 1K, Synth:R_Default (DIN0207), symbol synth:R_Default
- added R3: 500R, Synth:R_Default (DIN0207), symbol synth:R_Default
- added TP1: RATE_INPUT, Connector_Pin:Pin_D1.0mm_L10.0mm, symbol Connector:TestPoint
- added TP12: SQR_OUT, Connector_Pin:Pin_D1.0mm_L10.0mm, symbol Connector:TestPoint
- added TP13: +12V, Connector_Pin:Pin_D1.0mm_L10.0mm, symbol Connector:TestPoint
- added TP14: GND, Connector_Pin:Pin_D1.0mm_L10.0mm, symbol Connector:TestPoint
- added TP15: -12V, Connector_Pin:Pin_D1.0mm_L10.0mm, symbol Connector:TestPoint
- added TP2: TRI, Connector_Pin:Pin_D1.0mm_L10.0mm, symbol Connector:TestPoint
- added TP3: SQR, Connector_Pin:Pin_D1.0mm_L10.0mm, symbol Connector:TestPoint
- added TP4: TRI_IN, Connector_Pin:Pin_D1.0mm_L10.0mm, symbol Connector:TestPoint
- added TP6: TRI_OUT, Connector_Pin:Pin_D1.0mm_L10.0mm, symbol Connector:TestPoint
- added TP8: SQR_IN, Connector_Pin:Pin_D1.0mm_L10.0mm, symbol Connector:TestPoint
- added unit 3 of U1
- added unit 4 of U2
- added unit 3 of U2
- C2: footprint Synth:C_RECT_WIMA_0.1uF -> Synth:C_RECT_MKT_1uF
- Q1: renamed from Q3; footprint Package_TO_SOT_THT:TO-92L_HandSolder -> Package_TO_SOT_THT:TO-92_HandSolder
- Q2: renamed from Q4; footprint Package_TO_SOT_THT:TO-92L_HandSolder -> Package_TO_SOT_THT:TO-92_HandSolder
- U1: footprint (none) -> Package_DIP:DIP-14_W7.62mm_Socket_LongPads
- U2: renamed from U1; footprint (none) -> Package_DIP:DIP-14_W7.62mm_Socket_LongPads
- renumbered C8 to C10, C9 to C3, C10 to C4, C3 to C5, C4 to C6, C5 to C7, C6 to C8, C7 to C9, D1 to D2, D2 to D3, R7 to R10, R8 to R11, R16 to R12, RV2 to R13, R18 to R14, R20 to R15, R21 to R16, R22 to R17, R15 to R18, R23 to R19, R14 to R21, R3 to R4, R4 to R5, R5 to R6, R6 to R7, R10 to R8, R13 to R9, TIME_1 to RATE_1, R17 to RV2, J3 to SIN_OUT_1, J1 to SQR_OUT_1, TP4 to TP10, TP5 to TP11, TP1 to TP5, TP2 to TP7, TP3 to TP9, J2 to TRI_OUT_1, U2 to U1
Connections:
- net +12V: now also D1.2 (A), H4.4 (Pin_4), H6.4 (Pin_4), TP13.1
- net -12V: now also TP15.1
- net GNDREF: now also H1.8 (Pin_8), H2.8 (Pin_8), D4.1 (KA), H4.1 (Pin_1), H6.1 (Pin_1), H6.2 (Pin_2), H6.3 (Pin_3), R3.1, TP14.1, U2.10 (+), U2.12 (+); no longer H5.2 (Pin_2), H5.3 (Pin_3)
- net at R18.2: now also H7.1 (Pin_1); no longer H1.7 (Pin_7)
- net at H2.4 (Pin_4): now also U1.3 (+), TP8.1; no longer U1.12 (+)
- net at Q1.3 (C), R17.2, R9.1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: now also U1.6 (-); no longer U1.13 (-)
- net at Q2.3 (C), R14.1, R16.2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: now also U1.5 (+); no longer U1.12 (+)
- net at H2.1 (Pin_3), U2.2 (-): now also TP1.1
- net at H2.5 (Pin_5), R4.2, RV1.1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: now also H2.7 (Pin_7), TP2.1; no longer SW1.2 (B)
- net at H2.3 (Pin_3), R6.2, U2.7: now also TP3.1
- net at R21.2: now also H7.4 (Pin_4); no longer H1.8 (Pin_8)
- net at H2.6 (Pin_6): now also U1.12 (+), TP4.1; no longer U1.10 (+)
- new net: H5.1 (Pin_1), TP12.1, U1.1, U1.2 (-)
- new net: H5.2 (Pin_2), R17.1, U1.7
- new net: H1.7 (Pin_7), SW1.2 (B)
- new net: H7.2 (Pin_2), R19.2
- new net: U2.13 (-), U2.14
- new net: D1.1 (K), R3.2
- new net: H7.3 (Pin_3), R20.2
- new net: H5.4 (Pin_4), TP6.1, U1.10 (+), U1.13 (-), U1.14
- new net: H5.3 (Pin_3), U1.8, U1.9 (-)
- new net: D4.2 (AK), R20.1
- new net: U2.8, U2.9 (-)
Other:
- moved on the sheet: H1D, H1E, H1F, H2D, H2E, H2F, Q1, Q2, R12, R13, R14, R15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

Commit message: update components, PCB 3320 and design
Parts:
- added H16: PinHeader_01x02, Synth:PinHeader_1x02_P2.54mm_Vertical, symbol synth:PinHeader_01x02
- added H17: PinSocket_01x02, Synth:PinSocket_1x02_P2.54mm_Vertical, symbol synth:PinSocket_01x02
Connections:
- net at H1.1 (Pin_1), R2.1: no longer C1.1, C2.1
- net at H2.1 (Pin_3), TP1.1, U2.2 (-): now also C1.1, C2.1
- net at C1.2: now also H17.2 (Pin_2); no longer SW1.3 (C)
- net at SW1.1 (A): now also H16.1 (Pin_1); no longer C2.2
- new net: H16.2 (Pin_2), SW1.3 (C)
- new net: C2.2, H17.1 (Pin_1)
Other:
- moved on the sheet: C1, C2, R1, R2, RATE_1

Commit message: update component status, add IBOM for built modules
Parts:
- R10, R11: value 10 -> 10R
- R14, R16, R17, R9: value 10K, 1% -> 10K [1%]
- R15, R8: value 2.2K, 1% -> 2K2 [1%]
- R3: value 500R -> 470R
Changed lines of the file:
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@@
 	(wire
 		(pts
-			(xy 228.6 124.46) (xy 223.52 124.46)
+			(xy 228.6 120.65) (xy 223.52 120.65)
 		)
 		(stroke
@@
 	(wire
 		(pts
-			(xy 223.52 124.46) (xy 223.52 120.65)
-		)
-		(stroke
-			(width 0)
-			(type default)
-		)
-	)
-	(wire
-		(pts
 			(xy 304.8 219.71) (xy 304.8 212.09)
 		)
@@
 	(wire
 		(pts
-			(xy 228.6 125.73) (xy 228.6 124.46)
+			(xy 228.6 125.73) (xy 228.6 120.65)
 		)
 		(stroke
@@
 			)
 		)
-		(property "Value" "10"
+		(property "Value" "10R"
 			(at 198.12 276.86 90)
 			(effects
@@
 			)
 		)
-		(property "Value" "2.2K, 1%"
+		(property "Value" "2K2 [1%]"
 			(at 231.14 130.8099 0)
 			(effects
@@
 			)
 		)
-		(property "Value" "10K, 1%"
+		(property "Value" "10K [1%]"
 			(at 242.57 90.1699 0)
 			(effects
@@
 			)
 		)
-		(property "Value" "2.2K, 1%"
+		(property "Value" "2K2 [1%]"
 			(at 161.29 130.8099 0)
 			(effects
@@
 			)
 		)
-		(property "Value" "10"
+		(property "Value" "10R"
 			(at 198.12 248.92 90)
 			(effects
@@
 			)
 		)
-		(property "Value" "10K, 1%"
+		(property "Value" "10K [1%]"
 			(at 198.12 88.8999 0)
 			(effects
@@
 			)
 		)
-		(property "Value" "500R"
+		(property "Value" "470R"
 			(at 55.88 269.2399 0)
 			(effects
@@
 			)
 		)
-		(property "Value" "10K, 1%"
+		(property "Value" "10K [1%]"
 			(at 257.81 110.49 90)
 			(effects
@@
 			)
 		)
-		(property "Value" "10K, 1%"
+		(property "Value" "10K [1%]"
 			(at 218.44 88.8999 0)
 			(effects

Commit message: quantizers_stls
Parts:
- TP1, TP10, TP11, TP12, TP13, TP14, TP15, TP2, TP3, TP4, TP5, TP6, TP7, TP8, TP9: now left out of the parts list
Changed lines of the file:
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@@
 (kicad_sch
-	(version 20231120)
+	(version 20250114)
 	(generator "eeschema")
-	(generator_version "8.0")
+	(generator_version "9.0")
 	(paper "A3")
+	(rectangle
+		(start 149.86 241.3)
+		(end 248.92 281.94)
+		(stroke
+			(width 0.25)
+			(type dot)
+		)
+		(fill
+			(type none)
+		)
+	)
+	(rectangle
+		(start 250.19 241.3)
+		(end 297.18 281.94)
+		(stroke
+			(width 0.25)
+			(type dot)
+		)
+		(fill
+			(type none)
+		)
+	)
+	(rectangle
+		(start 63.5 241.3)
+		(end 104.14 281.94)
+		(stroke
+			(width 0.25)
+			(type dot)
+		)
+		(fill
+			(type none)
+		)
+	)
+	(rectangle
+		(start 107.95 241.3)
+		(end 148.59 281.94)
+		(stroke
+			(width 0.25)
+			(type dot)
+		)
+		(fill
+			(type none)
+		)
+	)
+	(text "SIN Symetry"
+		(exclude_from_sim no)
+		(at 214.122 152.4 0)
+		(effects
+			(font
+				(size 1.27 1.27)
+			)
+		)
+	)
+	(text "SIN_DISTORT"
+		(exclude_from_sim no)
+		(at 144.526 130.048 0)
+		(effects
+			(font
+				(size 1.27 1.27)
+			)
+		)
+	)
 	(junction
 		(at 207.01 262.89)
@@
 		)
 	)
-	(rectangle
-		(start 149.86 241.3)
-		(end 248.92 281.94)
-		(stroke
-			(width 0.25)
-			(type dot)
-		)
-		(fill
-			(type none)
-		)
-	)
-	(rectangle
-		(start 250.19 241.3)
-		(end 297.18 281.94)
-		(stroke
-			(width 0.25)
-			(type dot)
-		)
-		(fill
-			(type none)
-		)
-	)
-	(rectangle
-		(start 63.5 241.3)
-		(end 104.14 281.94)
-		(stroke
-			(width 0.25)
-			(type dot)
-		)
-		(fill
-			(type none)
-		)
-	)
-	(rectangle
-		(start 107.95 241.3)
-		(end 148.59 281.94)
-		(stroke
-			(width 0.25)
-			(type dot)
-		)
-		(fill
-			(type none)
-		)
-	)
-	(text "SIN Symetry"
-		(exclude_from_sim no)
-		(at 214.122 152.4 0)
-		(effects
-			(font
-				(size 1.27 1.27)
-			)
-		)
-	)
-	(text "SIN_DISTORT"
-		(exclude_from_sim no)
-		(at 144.526 130.048 0)
-		(effects
-			(font
-				(size 1.27 1.27)
-			)
-		)
-	)
 	(symbol
 		(lib_id "Mechanical:MountingHole")
@@
 		(unit 1)
 		(exclude_from_sim no)
-		(in_bom yes)
+		(in_bom no)
 		(on_board yes)
 		(dnp no)
@@
 		(unit 1)
 		(exclude_from_sim no)
-		(in_bom yes)
+		(in_bom no)
 		(on_board yes)
 		(dnp no)
@@
 		(unit 1)
 		(exclude_from_sim no)
-		(in_bom yes)
+		(in_bom no)
 		(on_board yes)
 		(dnp no)
@@
 		(unit 1)
 		(exclude_from_sim no)
-		(in_bom yes)
+		(in_bom no)
 		(on_board yes)
 		(dnp no)
@@
 		(unit 1)
 		(exclude_from_sim no)
-		(in_bom yes)
+		(in_bom no)
 		(on_board yes)
 		(dnp no)
@@
 		(unit 1)
 		(exclude_from_sim no)
-		(in_bom yes)
+		(in_bom no)
 		(on_board yes)
 		(dnp no)
@@
 		(unit 1)
 		(exclude_from_sim no)
-		(in_bom yes)
+		(in_bom no)
 		(on_board yes)
 		(dnp no)
@@
 		(unit 1)
 		(exclude_from_sim no)
-		(in_bom yes)
+		(in_bom no)
 		(on_board yes)
 		(dnp no)
@@
 		(unit 1)
 		(exclude_from_sim no)
-		(in_bom yes)
+		(in_bom no)
 		(on_board yes)
 		(dnp no)
@@
 		(unit 1)
 		(exclude_from_sim no)
-		(in_bom yes)
+		(in_bom no)
 		(on_board yes)
 		(dnp no)
@@
 		(unit 1)
 		(exclude_from_sim no)
-		(in_bom yes)
+		(in_bom no)
 		(on_board yes)
 		(dnp no)
@@
 		(unit 1)
 		(exclude_from_sim no)
-		(in_bom yes)
+		(in_bom no)
 		(on_board yes)
 		(dnp no)
@@
 		(unit 1)
 		(exclude_from_sim no)
-		(in_bom yes)
+		(in_bom no)
 		(on_board yes)
 		(dnp no)
@@
 		(unit 1)
 		(exclude_from_sim no)
-		(in_bom yes)
+		(in_bom no)
 		(on_board yes)
 		(dnp no)
@@
 		(unit 1)
 		(exclude_from_sim no)
-		(in_bom yes)
+		(in_bom no)
 		(on_board yes)
 		(dnp no)
@@
 		)
 	)
+	(embedded_fonts no)
 )
