File: modules/bus-board/KiCad/bus-board.kicad_pcb (KiCad board)
At the start: 2 copper layers, 300 x 40 mm, 51 parts, among them J1 PWR_16, J10 -12V, J11 GND, J12 +12V, J13 -12V, J14 +5V, J2 PWR_16, J3 PWR_16, J4 PWR_16, J5 PWR_16, J6 PWR_16, J7 +5V, J8 GND, J9 +12V

Commit message: Update files to newest version, add multiple boards and update v4_run (not ordered). Some AI generated files added.
Parts:
- added D4: LED, LED_SMD:LED_0805_2012Metric_Pad1.15x1.40mm_HandSolder, F.Cu at (200.5, 73.5)
- added D5: LED, LED_SMD:LED_0805_2012Metric_Pad1.15x1.40mm_HandSolder, F.Cu at (199.5, 81.5)
- added D6: LED, LED_SMD:LED_0805_2012Metric_Pad1.15x1.40mm_HandSolder, F.Cu at (199.0, 58.5)
- added G***: LOGO, synth-gfx:github-QR_lenimal_white, B.Cu at (190.0, 55.0)
- added R4: 1K, Resistor_SMD:R_0805_2012Metric_Pad1.20x1.40mm_HandSolder, F.Cu at (196.5, 73.5)
- added R5: 680R, Resistor_SMD:R_0805_2012Metric_Pad1.20x1.40mm_HandSolder, F.Cu at (195.5, 81.5)
- added R6: 1K, Resistor_SMD:R_0805_2012Metric_Pad1.20x1.40mm_HandSolder, F.Cu at (195.0, 58.5)
- moved H14 11.6 mm to (336.0, 54.0)
- moved H10 10.6 mm to (63.0, 54.0)
- moved H13 10.6 mm to (337.0, 86.0)
- moved H15 10.6 mm to (63.0, 86.0)
- moved H11 1.00 mm to (275.0, 86.0)
- moved H12 1.00 mm to (275.0, 54.0)
- moved H16 1.00 mm to (200.0, 54.0)
- moved H21 1.00 mm to (125.0, 86.0)
- moved H22 1.00 mm to (125.0, 54.0)
- moved H9 1.00 mm to (200.0, 86.0)
- moved J6 0.50 mm to (326.5, 65.0)
Routing:
- net -12V: track 309.6 -> 315.2 mm
- net +5V: track 310.3 -> 314.5 mm
- net Net-(D5-K): track 0.00 -> 2.00 mm
- net Net-(D6-A): track 0.00 -> 1.97 mm
- net Net-(J1-GATE-Pad15): track 263.2 -> 262.7 mm
- net Net-(J1-CV-Pad13): track 264.9 -> 264.4 mm
