File: modules/bus-board/KiCad/bus-board.kicad_sch (KiCad schematic)
At the start: 49 parts, among them J1 PWR_16, J10 -12V, J11 GND, J12 +12V, J13 -12V, J14 +5V, J2 PWR_16, J3 PWR_16, J4 PWR_16, J5 PWR_16, J6 PWR_16, J7 +5V, J8 GND, J9 +12V

Commit message: Update files to newest version, add multiple boards and update v4_run (not ordered). Some AI generated files added.
Parts:
- added D4, D5, D6: LED, LED_SMD:LED_0805_2012Metric_Pad1.15x1.40mm_HandSolder, symbol Device:LED
- added R4, R6: 1K, Resistor_SMD:R_0805_2012Metric_Pad1.20x1.40mm_HandSolder, symbol synth:R_Default
- added R5: 680R, Resistor_SMD:R_0805_2012Metric_Pad1.20x1.40mm_HandSolder, symbol synth:R_Default
Connections:
- net +12V: now also D4.2 (A)
- net +5V: now also D5.2 (A)
- net -12V: now also D6.1 (K)
- net GNDREF: now also R4.1, R5.1, R6.1
- new net: D4.1 (K), R4.2
- new net: D6.2 (A), R6.2
- new net: D5.1 (K), R5.2
Other:
- note added: "SMD"
- note added: "THT"
- moved on the sheet: C1, C2, C3
