File: modules/drums/1-kick/kiCad/kicks.kicad_sch (KiCad schematic)
At the start: 64 parts, among them J1 INPUT, J2 INPUT, J3 INPUT, J4 OUTPUT, Q1 BC858, Q2 BC848, Q3 BC858, Q4 BC848, Q5 BC848, U1 TL074

Commit message: Update files to newest version, add multiple boards and update v4_run (not ordered). Some AI generated files added.
Parts:
- R15: value 100K -> 47K
- R18: value 14K -> 10K
Other:
- note added: "Rev.1: Output is quite low, Replaced values R15 with 47K [100K] and R18 with 10K [14K]"
