File: modules/utility/7-compressor/kiCad/compressor.kicad_pcb (KiCad board)
At the start: 4 copper layers, 60 x 110 mm, 180 parts, among them J1 LEFT_OUT, J2 RIGHT_OUT, J3 STEREO_OUT, J4 INPUT, J5 INPUT, J6 SIDECHAIN_IN, J7 SIDECHAIN_IN, Q1 MMBT3904, Q10 MMBT3904, Q2 MMBT3904, Q3 MMBT3904, Q4 MMBT3904, Q5 MMBT3904, Q6 MMBT3904, Q7 MMBT3904, Q8 MMBT3904, Q9 MMBT3904, SW1 SW_SPDT, SW2 SW_SPDT, U1 TL072, U2 TL074, U3 TL074, U4 TL072, U5 TL072, U6 TL072

Commit message: Update files to newest version, add multiple boards and update v4_run (not ordered). Some AI generated files added.
Connections:
- RV12 pad 2: Net-(RV12-Pad2) -> GNDREF
- RV12 pad 3: Net-(RV12-Pad2) -> GNDREF
- RV8 pad 2: Net-(RV8-Pad2) -> GNDREF
- RV8 pad 3: Net-(RV8-Pad2) -> GNDREF
Routing:
- net GNDREF: track 31.2 -> 36.2 mm
- net Net-(RV8-Pad2): track 2.50 -> 0.00 mm
- net Net-(RV12-Pad2): track 2.50 -> 0.00 mm
