File: modules/utility/8-precision-adder/kiCad/precision-adder.kicad_pcb (KiCad board)
At the start: 2 copper layers, 30 x 110 mm, 57 parts, among them J1 OUT, J2 INPUT, J3 OUT, J4 INPUT, J5 OUT, J6 INPUT, J7 INV_OUT, J8 INPUT, SW1 ON_OFF_ON, SW2 ON_OFF_ON, SW3 ON_OFF_ON, SW4 ON_OFF_ON, U1 OPA4171, U2 OPA4171, U3 LM4040DBZ-2.0

Commit message: Update files to newest version, add multiple boards and update v4_run (not ordered). Some AI generated files added.
Parts:
- RV2: value R_Potentiometer -> B100K
- moved RV3 1.00 mm to (75.0, 59.0)
Connections:
- R2 pad 1: Net-(U2C-+) -> Net-(U2C--)
- R7 pad 2: Net-(U2C-+) -> Net-(U2C--)
- U2 pad 10: Net-(U2C-+) -> GNDREF
- U2 pad 9: GNDREF -> Net-(U2C--)
Routing:
- net Net-(U2C-+): track 9.70 -> 0.00 mm
- net Net-(U2C--): track 0.00 -> 8.09 mm
- net GNDREF: track 5.07 -> 7.70 mm
- net Net-(R18-Pad2): track 2.44 -> 3.39 mm
