File: modules/drums/2-clap/kiCad/body_osc.kicad_sch (KiCad schematic)
At the start: 25 parts, among them U2 TL074, U3 TL074

Commit message: remove test for claude skill
Parts:
- removed RV1: B250K, Potentiometer_THT:Potentiometer_Alpha_RD902F-40-00D_Dual_Vertical_CircularHoles, symbol Device:R_Potentiometer_Dual
- added RV14, RV16: A1M, Synth:Potentiometer_TT_P0915N, symbol synth:R_Potentiometer (P0915N)
Connections:
- net BODY_OUT: now also U3.8; no longer U3.1
- net GNDREF: now also R11.2, R12.2, U2.12 (+), U2.9 (-), U3.10 (+); no longer U2.10 (+), U2.13 (-), U3.3 (+)
- net OSC2: now also U2.14; no longer U2.8
- net at R17.2, R18.2, R19.1: now also U3.9 (-); no longer U3.2 (-)
- net at R24.2, TP7.1: now also U2.8; no longer U2.14
- net at R22.1, R24.1, R50.1: now also RV16.3
- net at R14.1, R15.1, R9.1: now also RV14.3
- net at R10.2: now also RV14.2
- net at R25.2: now also RV16.2
- net at R12.1: now also RV16.1
- net at C4.1, R25.1: now also U2.13 (-); no longer U2.9 (-)
- net at R16.1, R22.2: now also U2.10 (+); no longer U2.12 (+)
- net -12V: no longer names the net of R11.1
- net -12V: now also RV14.1; no longer R12.2
Other:
- note added: "If you want higher sounds, C3/C4 can be dropped to 4.7nF"
- note added: "Resistors could be higher, up to 4.7K/10K to offset some of the 'dead' zone"
- note added: "TUNE A"
- note added: "TUNE B"
- note removed: "Originally going to GND for both pots, but that would cause 'bleed'. Something to check on breadboard."
- moved on the sheet: C3, C4, R10, R12, R13, R14, R15, R16, R17, R18, R22, R24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
