File: modules/drums/2-clap/kiCad/lm13700_vca.kicad_sch (KiCad schematic)
At the start: 5 parts, among them U5 LM13700

Commit message: remove test for claude skill
Changed lines of the file:
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@@
+	(wire
+		(pts
+			(xy 129.54 60.96) (xy 140.97 60.96)
+		)
+		(stroke
+			(width 0)
+			(type default)
+		)
+	)
 	(wire
 		(pts
@@
 	(hierarchical_label "INPUT"
 		(shape input)
-		(at 140.97 60.96 180)
+		(at 129.54 60.96 180)
 		(effects
 			(font
