File: modules/drums/2-clap/kiCad/snare_env.kicad_sch (KiCad schematic)
At the start: 7 parts, among them U1 TL074

Commit message: remove test for claude skill
Parts:
- removed unit 4 of U1
- added J7: SHELL_DECAY_CV, Synth:Jack_3.5mm_QingPu_WQP-PJ398SM_Vertical_CircularHoles, symbol synth:AudioJack_Mono_3.5mm
- added J8: SNAP_DECAY_CV, Synth:Jack_3.5mm_QingPu_WQP-PJ398SM_Vertical_CircularHoles, symbol synth:AudioJack_Mono_3.5mm
- added R73, R79: 470K, Resistor_SMD:R_0805_2012Metric_Pad1.20x1.40mm_HandSolder, symbol Device:R
- added R74, R80: 100K, Resistor_SMD:R_0805_2012Metric_Pad1.20x1.40mm_HandSolder, symbol Device:R
- added R75, R81: 1K, Resistor_SMD:R_0805_2012Metric_Pad1.20x1.40mm_HandSolder, symbol Device:R
- added R76, R77, R82, R83: 47K, Resistor_SMD:R_0805_2012Metric_Pad1.20x1.40mm_HandSolder, symbol Device:R
- added R78, R84: 2K2, Resistor_SMD:R_0805_2012Metric_Pad1.20x1.40mm_HandSolder, symbol Device:R
- added RV10, RV13: 5K, Potentiometer_THT:Potentiometer_Runtron_RM-065_Vertical, symbol Device:R_Potentiometer_Trim
- added RV11, RV9: B10K, Synth:Potentiometer_TT_P0915N, symbol synth:R_Potentiometer (P0915N)
- added unit 2 of U10
- added U8: LM13700, Synth:SOIC-16, symbol Amplifier_Operational:LM13700
- D3, D4: footprint Synth:D_DO-35_SOD27_P7.62mm_Horizontal -> Diode_SMD:D_SOD-323_HandSoldering
- RV2, RV3: value B500K -> B10K
- U10: renamed from U1; value TL074 -> TL072; footprint Synth:SOIC-14 -> Synth:SOIC-8; symbol Amplifier_Operational:TL074 -> Amplifier_Operational:TL072
Connections:
- net GNDREF: now also J7.S, J7.TN, J8.S, J8.TN, R73.1, R75.2, R79.1, R81.2, RV11.1, RV9.1, U8.10, U8.14 (+), U8.3 (+), U8.7; no longer RV2.2, RV3.2
- net SHELL_CAP: now also U10.3 (+), R73.2, R74.2, U8.5; no longer RV2.1, U10.10 (+)
- net SHELL_ENV: now also U10.1, U10.2 (-); no longer U10.8, U10.9 (-)
- net SNAP_CAP: now also R79.2, R80.2, U10.5 (+), U8.12; no longer RV3.1
- net SNAP_ENV: now also U10.6 (-), U10.7
- new net: J7.T, RV9.3
- new net: R76.1, RV2.2
- new net: R83.1, RV3.2
- new net: R74.1, R75.1, U8.4 (-)
- new net: J8.T, RV11.3
- new net: R76.2, R77.2, R78.2, U8.1
- new net: R77.1, RV9.2
- new net: R78.1, RV10.1
- new net: R82.1, RV11.2
- new net: R80.1, R81.1, U8.13 (-)
- new net: R82.2, R83.2, R84.2, U8.16
- new net: R84.1, RV13.1
- new net +12V: RV2.1, RV3.1
- new net -12V: RV10.2, RV10.3, RV13.2, RV13.3
- no-connect marks 0 -> 4
Other:
- moved on the sheet: C5, C7, D3, D4, U10A
