File: modules/drums/2-clap/kiCad/trigger_input.kicad_sch (KiCad schematic)
At the start: 16 parts, among them J1 SNARE_TRIG, J2 CLAP_TRIG, J3 TRIG_NORM_JPR, U1 TL074

Commit message: remove test for claude skill
Parts:
- R2: value 39K -> 100K
- U1: value TL074 -> TL072; footprint Synth:SOIC-14 -> Synth:SOIC-8; symbol Amplifier_Operational:TL074 -> Amplifier_Operational:TL072
Changed lines of the file:
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@@
 	(wire
 		(pts
-			(xy 118.11 104.14) (xy 111.76 104.14)
+			(xy 151.13 104.14) (xy 111.76 104.14)
 		)
 		(stroke
@@
 	(wire
 		(pts
-			(xy 113.03 34.29) (xy 105.41 34.29)
+			(xy 153.67 34.29) (xy 105.41 34.29)
 		)
 		(stroke
@@
 	(hierarchical_label "CLAP_FIRE"
 		(shape input)
-		(at 118.11 104.14 0)
+		(at 151.13 104.14 0)
 		(effects
 			(font
@@
 	(hierarchical_label "SNARE_FIRE"
 		(shape input)
-		(at 113.03 34.29 0)
+		(at 153.67 34.29 0)
 		(effects
 			(font
@@
 			)
 		)
-		(property "Value" "39K"
+		(property "Value" "100K"
 			(at 69.85 40.6399 0)
 			(show_name no)
@@
 	)
 	(symbol
-		(lib_id "Amplifier_Operational:TL074")
+		(lib_id "Amplifier_Operational:TL072")
 		(at 104.14 104.14 0)
 		(unit 2)
@@
 			)
 		)
-		(property "Value" "TL074"
+		(property "Value" "TL072"
 			(at 104.14 96.52 0)
 			(show_name no)
@@
 			)
 		)
-		(property "Footprint" "Synth:SOIC-14"
-			(at 102.87 101.6 0)
+		(property "Footprint" "Synth:SOIC-8"
+			(at 104.14 104.14 0)
 			(hide yes)
 			(show_name no)
@@
 		)
 		(property "Datasheet" "http://www.ti.com/lit/ds/symlink/tl071.pdf"
-			(at 105.41 99.06 0)
-			(hide yes)
-			(show_name no)
-			(do_not_autoplace no)
-			(effects
-				(font
-					(size 1.27 1.27)
-				)
-			)
-		)
-		(property "Description" "Quad Low-Noise JFET-Input Operational Amplifiers, DIP-14/SOIC-14"
 			(at 104.14 104.14 0)
 			(hide yes)
@@
 			)
 		)
-		(pin "13"
-		)
-		(pin "11"
-		)
-		(pin "14"
+		(property "Description" "Dual Low-Noise JFET-Input Operational Amplifiers, DIP-8/SOIC-8"
+			(at 104.14 104.14 0)
+			(hide yes)
+			(show_name no)
+			(do_not_autoplace no)
+			(effects
+				(font
+					(size 1.27 1.27)
+				)
+			)
 		)
 		(pin "4"
-		)
-		(pin "12"
-		)
-		(pin "9"
-		)
-		(pin "10"
 		)
 		(pin "3"
@@
 	)
 	(symbol
-		(lib_id "Amplifier_Operational:TL074")
+		(lib_id "Amplifier_Operational:TL072")
 		(at 97.79 34.29 0)
 		(unit 1)
@@
 			)
 		)
-		(property "Value" "TL074"
+		(property "Value" "TL072"
 			(at 97.79 26.67 0)
 			(show_name no)
@@
 			)
 		)
-		(property "Footprint" "Synth:SOIC-14"
-			(at 96.52 31.75 0)
+		(property "Footprint" "Synth:SOIC-8"
+			(at 97.79 34.29 0)
 			(hide yes)
 			(show_name no)
@@
 		)
 		(property "Datasheet" "http://www.ti.com/lit/ds/symlink/tl071.pdf"
-			(at 99.06 29.21 0)
-			(hide yes)
-			(show_name no)
-			(do_not_autoplace no)
-			(effects
-				(font
-					(size 1.27 1.27)
-				)
-			)
-		)
-		(property "Description" "Quad Low-Noise JFET-Input Operational Amplifiers, DIP-14/SOIC-14"
 			(at 97.79 34.29 0)
 			(hide yes)
@@
 			)
 		)
-		(pin "13"
-		)
-		(pin "11"
-		)
-		(pin "14"
+		(property "Description" "Dual Low-Noise JFET-Input Operational Amplifiers, DIP-8/SOIC-8"
+			(at 97.79 34.29 0)
+			(hide yes)
+			(show_name no)
+			(do_not_autoplace no)
+			(effects
+				(font
+					(size 1.27 1.27)
+				)
+			)
 		)
 		(pin "4"
 		)
-		(pin "12"
-		)
-		(pin "9"
-		)
-		(pin "10"
-		)
 		(pin "3"
