File: modules/drums/3-hats/kiCad/mad-hatter.kicad_sch (KiCad schematic)
At the start: 19 parts, among them Q1 MMBT3904, U1 TL074, U2 TL074, U3 TL074, U4 40106, U5 LM13700, U6 LM13700

Commit message: remove test for claude skill
Parts:
- removed C21, C22: 47uF, Capacitor_THT:CP_Radial_D6.3mm_P2.50mm, symbol Device:C_Polarized
- removed C23, C24: 100nF, Capacitor_SMD:C_0805_2012Metric_Pad1.18x1.45mm_HandSolder, symbol Device:C
- removed D10, D11: 1N5819WS, Diode_SMD:D_SOD-323_HandSoldering, symbol Diode:1N5819WS
- removed H2: POWER_CONN, Synth:IDC-Header_2x05_P2.54mm_Vertical, symbol synth:Conn_02x05_EuroRack_Power
- removed R40, R41: 10R, Resistor_SMD:R_0805_2012Metric_Pad1.20x1.40mm_HandSolder, symbol Device:R
- removed TP12: GND, Connector_Pin:Pin_D1.0mm_L10.0mm, symbol Connector:TestPoint
- removed TP13: -12V, Connector_Pin:Pin_D1.0mm_L10.0mm, symbol Connector:TestPoint
- removed TP6: +12V, Connector_Pin:Pin_D1.0mm_L10.0mm, symbol Connector:TestPoint
- removed U1: TL074, Synth:SOIC-14, symbol Amplifier_Operational:TL074
- removed unit 5 of U2
- removed unit 1 of U2
- removed unit 5 of U3
- removed U4: 40106, symbol 4xxx:40106
- removed U5, U6: LM13700, Synth:SOIC-16, symbol Amplifier_Operational:LM13700
- added U6: LM13700, Synth:SOIC-16, symbol Amplifier_Operational:LM13700
- added U7: NOISE_BOARD, Synth:noise_board, symbol synth:noise_board
Connections:
- net +12V: now also U7.1 (+12V)
- net -12V: now also U7.3 (-12V)
- net GNDREF: now also U7.2 (GND)
- new net metalic_core/NOISE_IN: U7.4 (WHITE)
- no-connect marks 0 -> 1
Other:
- added sheet CH (untitled.kicad_sch)
- added sheet metalic_core (metalic_core.kicad_sch)
- added sheet power (power.kicad_sch)
- sheet 13700_vca ports: added CTRL_INPUT, OUTPUT, SIGNAL_INPUT; removed none
- sheet trigger ports: added CH_FIRE, CYM_FIRE, OH_FIRE; removed none
- moved on the sheet: U2B, U2C, U2D, U3A, U3B, U3C, U3D
