File: modules/drums/3-hats/kiCad/power.kicad_sch (KiCad schematic)
At the start: 27 parts, among them J9 CLAP_DECAY_CV, U6 LM13700, U7 40106

Commit message: remove test for claude skill
Parts:
- removed C10, C9: 100nF, Capacitor_SMD:C_0805_2012Metric_Pad1.18x1.45mm_HandSolder, symbol synth:C_sm (MKS)
- removed C11: 1uF, Capacitor_SMD:C_0805_2012Metric_Pad1.18x1.45mm_HandSolder, symbol synth:C_sm (MKS)
- removed C8: 470nF, Capacitor_SMD:C_0805_2012Metric_Pad1.18x1.45mm_HandSolder, symbol synth:C_sm (MKS)
- removed D5, D6, D7, D8, D9: 1N4148, Diode_SMD:D_SOD-323_HandSoldering, symbol synth:D_Signal (1N4148)
- removed J9: CLAP_DECAY_CV, Synth:Jack_3.5mm_QingPu_WQP-PJ398SM_Vertical_CircularHoles, symbol synth:AudioJack_Mono_3.5mm
- removed R37, R48, R49: 100K, Resistor_SMD:R_0805_2012Metric_Pad1.20x1.40mm_HandSolder, symbol synth:R_Default
- removed R38: 82K, Resistor_SMD:R_0805_2012Metric_Pad1.20x1.40mm_HandSolder, symbol synth:R_Default
- removed R39: 75K, Resistor_SMD:R_0805_2012Metric_Pad1.20x1.40mm_HandSolder, symbol synth:R_Default
- removed R46: 22K, Resistor_SMD:R_0805_2012Metric_Pad1.20x1.40mm_HandSolder, symbol synth:R_Default
- removed R85: 470K, Resistor_SMD:R_0805_2012Metric_Pad1.20x1.40mm_HandSolder, symbol Device:R
- removed R86: 100K, Resistor_SMD:R_0805_2012Metric_Pad1.20x1.40mm_HandSolder, symbol Device:R
- removed R87: 1K, Resistor_SMD:R_0805_2012Metric_Pad1.20x1.40mm_HandSolder, symbol Device:R
- removed R88, R89: 47K, Resistor_SMD:R_0805_2012Metric_Pad1.20x1.40mm_HandSolder, symbol Device:R
- removed R90: 2K2, Resistor_SMD:R_0805_2012Metric_Pad1.20x1.40mm_HandSolder, symbol Device:R
- removed RV12, RV8: B10K, Synth:Potentiometer_TT_P0915N, symbol synth:R_Potentiometer (P0915N)
- removed RV15: 5K, Potentiometer_THT:Potentiometer_Runtron_RM-065_Vertical, symbol Device:R_Potentiometer_Trim
- removed U6: LM13700, Synth:SOIC-16, symbol Amplifier_Operational:LM13700
- removed U7: 40106, Synth:SOIC-14, symbol 4xxx:40106
- added C21, C22: 47uF, Capacitor_THT:CP_Radial_D6.3mm_P2.50mm, symbol Device:C_Polarized
- added C23, C24, C29, C30, C31, C32, C33, C34, C35, C36, C37, C38, C39: 100nF, Capacitor_SMD:C_0805_2012Metric_Pad1.18x1.45mm_HandSolder, symbol Device:C
- added D10, D11: 1N5819WS, Diode_SMD:D_SOD-323_HandSoldering, symbol Diode:1N5819WS
- added H2: POWER_CONN, Synth:IDC-Header_2x05_P2.54mm_Vertical, symbol synth:Conn_02x05_EuroRack_Power
- added R40, R41: 10R, Resistor_SMD:R_0805_2012Metric_Pad1.20x1.40mm_HandSolder, symbol Device:R
- added TP12: GND, Connector_Pin:Pin_D1.0mm_L10.0mm, symbol Connector:TestPoint
- added TP13: -12V, Connector_Pin:Pin_D1.0mm_L10.0mm, symbol Connector:TestPoint
- added TP6: +12V, Connector_Pin:Pin_D1.0mm_L10.0mm, symbol Connector:TestPoint
- added U1: TL074, Synth:SOIC-14, symbol Amplifier_Operational:TL074
- added U2, U3: TL074, symbol Amplifier_Operational:TL074
- added U4: 40106, symbol 4xxx:40106
- added U5, U6: LM13700, Synth:SOIC-16, symbol Amplifier_Operational:LM13700
Connections:
- net +12V: now also C21.1, C23.1, C29.1, C31.1, C33.1, C35.1, C37.1, C39.1, R40.2, TP6.1, U1.4 (V+), U2.4 (V+), U3.4 (V+), U4.14 (VDD), U5.11 (V+), U6.11 (V+)
- net -12V: now also C22.2, C24.2, C30.2, C32.2, C34.2, C36.2, C38.2, R41.2, TP13.1, U1.11 (V-), U2.11 (V-), U3.11 (V-), U5.6 (V-), U6.6 (V-)
- net GNDREF: now also C21.2, C22.1, C23.2, C24.1, C29.2, C30.1, C31.2, C32.1, C33.2, C34.1, C35.2, C36.1, C37.2, C38.1, C39.2, H2.3 (Pin_3), H2.4 (Pin_4), H2.5 (Pin_5), H2.6 (Pin_6), H2.7 (Pin_7), H2.8 (Pin_8), TP12.1, U4.7 (VSS)
- new net: D11.1 (K), H2.1 (Pin_1), H2.2 (Pin_2)
- new net: D11.2 (A), R41.1
- new net: D10.1 (K), R40.1
- new net: D10.2 (A), H2.10 (Pin_10), H2.9 (Pin_9)
- no-connect marks 2 -> 0
Other:
- note removed: "CLAP DECAY"
